Commit message: Load hips and feet names by yaml file

File: descriptions/anymal_description/robots/anymal.urdf.xacro (robot description, xacro)
@@ -109,5 +109,5 @@
         </inertial>
     </link>
-    <link name="lf_hipassembly">
+    <link name="lf_hip">
         <visual>
             <origin rpy="0 0 0.0" xyz="0 0 0"/>
@@ -140,5 +140,5 @@
     <joint name="lf_haa_joint" type="revolute">
         <parent link="trunk"/>
-        <child link="lf_hipassembly"/>
+        <child link="lf_hip"/>
         <origin xyz="0.277 0.116 0.0"/>
         <axis xyz="1 0 0"/>
@@ -146,5 +146,5 @@
         <dynamics damping="0.0" friction="0.0"/>
     </joint>
-    <link name="LF_THIGH">
+    <link name="lf_thigh">
         <visual>
             <origin rpy="0 0 0.0" xyz="0 0 0"/>
@@ -183,6 +183,6 @@
     <!-- Thigh joint -->
     <joint name="lf_hfe_joint" type="revolute">
-        <parent link="lf_hipassembly"/>
-        <child link="LF_THIGH"/>
+        <parent link="lf_hip"/>
+        <child link="lf_thigh"/>
         <origin xyz="0.0635                    0.041                    0.0"/>
         <axis xyz="0 1 0"/>
@@ -190,5 +190,5 @@
         <dynamics damping="0.0" friction="0.0"/>
     </joint>
-    <link name="LF_SHANK">
+    <link name="lf_shank">
         <visual>
             <origin rpy="0 0 0.0" xyz="0 0 0"/>
@@ -212,6 +212,6 @@
     <!-- Shank joint -->
     <joint name="lf_kfe_joint" type="revolute">
-        <parent link="LF_THIGH"/>
-        <child link="LF_SHANK"/>
+        <parent link="lf_thigh"/>
+        <child link="lf_shank"/>
         <origin xyz="0.0 0.109 -0.25"/>
         <axis xyz="0 1 0"/>
@@ -220,11 +220,11 @@
     </joint>
     <!-- Shank to Adapter joint -->
-    <joint name="LF_SHANK_TO_ADAPTER" type="fixed">
-        <parent link="LF_SHANK"/>
-        <child link="LF_ADAPTER"/>
+    <joint name="lf_shank_to_adapter" type="fixed">
+        <parent link="lf_shank"/>
+        <child link="lf_adapter"/>
         <origin rpy="0.0 0.0 0.0" xyz="0.1 -0.02 0.0"/>
     </joint>
     <!-- Adapter link -->
-    <link name="LF_ADAPTER">
+    <link name="lf_adapter">
         <visual>
             <origin rpy="0 0 0.0" xyz="0 0 0.032"/>
@@ -248,6 +248,6 @@
     </link>
     <!-- Adapter to Foot joint -->
-    <joint name="LF_ADAPTER_TO_FOOT" type="fixed">
-        <parent link="LF_ADAPTER"/>
+    <joint name="lf_adapter_to_foot" type="fixed">
+        <parent link="lf_adapter"/>
         <child link="lf_foot"/>
         <origin rpy="0.0 0.0 0.0" xyz="0.0 0.0 -0.32125"/>
@@ -262,5 +262,5 @@
         </collision>
     </link>
-    <link name="rf_hipassembly">
+    <link name="rf_hip">
         <visual>
             <origin rpy="0 0 0.0" xyz="0 0 0"/>
@@ -293,5 +293,5 @@
     <joint name="rf_haa_joint" type="revolute">
         <parent link="trunk"/>
-        <child link="rf_hipassembly"/>
+        <child link="rf_hip"/>
         <origin xyz="0.277 -0.116 0.0"/>
         <axis xyz="1 0 0"/>
@@ -299,5 +299,5 @@
         <dynamics damping="0.0" friction="0.0"/>
     </joint>
-    <link name="RF_THIGH">
+    <link name="rf_tigh">
         <visual>
             <origin rpy="0 0 0.0" xyz="0 0 0"/>
@@ -336,6 +336,6 @@
     <!-- Thigh joint -->
     <joint name="rf_hfe_joint" type="revolute">
-        <parent link="rf_hipassembly"/>
-        <child link="RF_THIGH"/>
+        <parent link="rf_hip"/>
+        <child link="rf_tigh"/>
         <origin xyz="0.0635                    -0.041                    0.0"/>
         <axis xyz="0 1 0"/>
@@ -343,5 +343,5 @@
         <dynamics damping="0.0" friction="0.0"/>
     </joint>
-    <link name="RF_SHANK">
+    <link name="rf_shank">
         <visual>
             <origin rpy="0 0 0.0" xyz="0 0 0"/>
@@ -365,6 +365,6 @@
     <!-- Shank joint -->
     <joint name="rf_kfe_joint" type="revolute">
-        <parent link="RF_THIGH"/>
-        <child link="RF_SHANK"/>
+        <parent link="rf_tigh"/>
+        <child link="rf_shank"/>
         <origin xyz="0.0 -0.109 -0.25"/>
         <axis xyz="0 1 0"/>
@@ -373,11 +373,11 @@
     </joint>
     <!-- Shank to Adapter joint -->
-    <joint name="RF_SHANK_TO_ADAPTER" type="fixed">
-        <parent link="RF_SHANK"/>
-        <child link="RF_ADAPTER"/>
+    <joint name="rf_shank_to_adapter" type="fixed">
+        <parent link="rf_shank"/>
+        <child link="rf_adapter"/>
         <origin rpy="-0.0 0.0 -0.0" xyz="0.1 0.02 0.0"/>
     </joint>
     <!-- Adapter link -->
-    <link name="RF_ADAPTER">
+    <link name="rf_adapter">
         <visual>
             <origin rpy="0 0 0.0" xyz="0 0 0.032"/>
@@ -401,6 +401,6 @@
     </link>
     <!-- Adapter to Foot joint -->
-    <joint name="RF_ADAPTER_TO_FOOT" type="fixed">
-        <parent link="RF_ADAPTER"/>
+    <joint name="rf_adapter_to_foot" type="fixed">
+        <parent link="rf_adapter"/>
         <child link="rf_foot"/>
         <origin rpy="-0.0 0.0 -0.0" xyz="0.0 -0.0 -0.32125"/>
@@ -415,5 +415,5 @@
         </collision>
     </link>
-    <link name="lh_hipassembly">
+    <link name="lh_hip">
         <visual>
             <origin rpy="0 0 -3.14159265359" xyz="0 0 0"/>
@@ -446,5 +446,5 @@
     <joint name="lh_haa_joint" type="revolute">
         <parent link="trunk"/>
-        <child link="lh_hipassembly"/>
+        <child link="lh_hip"/>
         <origin xyz="-0.277 0.116 0.0"/>
         <axis xyz="1 0 0"/>
@@ -452,5 +452,5 @@
         <dynamics damping="0.0" friction="0.0"/>
     </joint>
-    <link name="LH_THIGH">
+    <link name="lh_thigh">
         <visual>
             <origin rpy="0 0 -3.14159265359" xyz="0 0 0"/>
@@ -489,6 +489,6 @@
     <!-- Thigh joint -->
     <joint name="lh_hfe_joint" type="revolute">
-        <parent link="lh_hipassembly"/>
-        <child link="LH_THIGH"/>
+        <parent link="lh_hip"/>
+        <child link="lh_thigh"/>
         <origin xyz="-0.0635                    0.041                    0.0"/>
         <axis xyz="0 1 0"/>
@@ -496,5 +496,5 @@
         <dynamics damping="0.0" friction="0.0"/>
     </joint>
-    <link name="LH_SHANK">
+    <link name="lh_shank">
         <visual>
             <origin rpy="0 0 -3.14159265359" xyz="0 0 0"/>
@@ -518,6 +518,6 @@
     <!-- Shank joint -->
     <joint name="lh_kfe_joint" type="revolute">
-        <parent link="LH_THIGH"/>
-        <child link="LH_SHANK"/>
+        <parent link="lh_thigh"/>
+        <child link="lh_shank"/>
         <origin xyz="-0.0 0.109 -0.25"/>
         <axis xyz="0 1 0"/>
@@ -526,11 +526,11 @@
     </joint>
     <!-- Shank to Adapter joint -->
-    <joint name="LH_SHANK_TO_ADAPTER" type="fixed">
-        <parent link="LH_SHANK"/>
-        <child link="LH_ADAPTER"/>
+    <joint name="lh_shank_to_adapter" type="fixed">
+        <parent link="lh_shank"/>
+        <child link="lh_adapter"/>
         <origin rpy="0.0 -0.0 -0.0" xyz="-0.1 -0.02 0.0"/>
     </joint>
     <!-- Adapter link -->
-    <link name="LH_ADAPTER">
+    <link name="lh_adapter">
         <visual>
             <origin rpy="0 0 -3.14159265359" xyz="0 0 0.032"/>
@@ -554,6 +554,6 @@
     </link>
     <!-- Adapter to Foot joint -->
-    <joint name="LH_ADAPTER_TO_FOOT" type="fixed">
-        <parent link="LH_ADAPTER"/>
+    <joint name="lh_adapter_to_foot" type="fixed">
+        <parent link="lh_adapter"/>
         <child link="lh_foot"/>
         <origin rpy="0.0 -0.0 -0.0" xyz="-0.0 0.0 -0.32125"/>
@@ -568,5 +568,5 @@
         </collision>
     </link>
-    <link name="rh_hipassembly">
+    <link name="rh_hip">
         <visual>
             <origin rpy="0 0 -3.14159265359" xyz="0 0 0"/>
@@ -599,5 +599,5 @@
     <joint name="rh_haa_joint" type="revolute">
         <parent link="trunk"/>
-        <child link="rh_hipassembly"/>
+        <child link="rh_hip"/>
         <origin xyz="-0.277 -0.116 0.0"/>
         <axis xyz="1 0 0"/>
@@ -605,5 +605,5 @@
         <dynamics damping="0.0" friction="0.0"/>
     </joint>
-    <link name="RH_THIGH">
+    <link name="rh_thigh">
         <visual>
             <origin rpy="0 0 -3.14159265359" xyz="0 0 0"/>
@@ -642,6 +642,6 @@
     <!-- Thigh joint -->
     <joint name="rh_hfe_joint" type="revolute">
-        <parent link="rh_hipassembly"/>
-        <child link="RH_THIGH"/>
+        <parent link="rh_hip"/>
+        <child link="rh_thigh"/>
         <origin xyz="-0.0635                    -0.041                    0.0"/>
         <axis xyz="0 1 0"/>
@@ -649,5 +649,5 @@
         <dynamics damping="0.0" friction="0.0"/>
     </joint>
-    <link name="RH_SHANK">
+    <link name="rh_shank">
         <visual>
             <origin rpy="0 0 -3.14159265359" xyz="0 0 0"/>
@@ -671,6 +671,6 @@
     <!-- Shank joint -->
     <joint name="rh_kfe_joint" type="revolute">
-        <parent link="RH_THIGH"/>
-        <child link="RH_SHANK"/>
+        <parent link="rh_thigh"/>
+        <child link="rh_shank"/>
         <origin xyz="-0.0 -0.109 -0.25"/>
         <axis xyz="0 1 0"/>
@@ -679,11 +679,11 @@
     </joint>
     <!-- Shank to Adapter joint -->
-    <joint name="RH_SHANK_TO_ADAPTER" type="fixed">
-        <parent link="RH_SHANK"/>
-        <child link="RH_ADAPTER"/>
+    <joint name="rh_shank_to_adapter" type="fixed">
+        <parent link="rh_shank"/>
+        <child link="rh_adapter"/>
         <origin rpy="-0.0 -0.0 0.0" xyz="-0.1 0.02 0.0"/>
     </joint>
     <!-- Adapter link -->
-    <link name="RH_ADAPTER">
+    <link name="rh_adapter">
         <visual>
             <origin rpy="0 0 -3.14159265359" xyz="0 0 0.032"/>
@@ -707,6 +707,6 @@
     </link>
     <!-- Adapter to Foot joint -->
-    <joint name="RH_ADAPTER_TO_FOOT" type="fixed">
-        <parent link="RH_ADAPTER"/>
+    <joint name="rh_adapter_to_foot" type="fixed">
+        <parent link="rh_adapter"/>
         <child link="rh_foot"/>
         <origin rpy="-0.0 -0.0 0.0" xyz="-0.0 -0.0 -0.32125"/>
@@ -737,9 +737,4 @@
                 imu_topic="trunk_imu_1/data"
                 update_rate="250">
-                <!-- old URDF -->
-                <!--origin xyz="0.290 0.000 0.0999214" rpy="0 ${-PI} 0"/ -->
-                <!-- new URDF with ideal values from CAD -->
-                <!--origin xyz="0.28525 0.000 0.0967678" rpy="0 0 0"/-->
-                <!-- new URDF, REAL values manually measured from the edge of the robot -->
                 <origin xyz="0.27025 0.000 0.0967678" rpy="0 0 0"/>
         </xacro:microstrain_3dmgx425_imu>
@@ -749,11 +744,4 @@
                 imu_topic="kvh_imu/data"
                 update_rate="250">
-            <!-- OLD URDF with manually created cylinder -->
-            <!--origin xyz="0.352845 0.0029 0.0503678" rpy="0 ${-PI} 0"/-->
-            <!-- NEW URDF with mesh, ideal values from CAD -->
-            <!--origin xyz="0.36347 0.00 0.0887678" rpy="0 ${PI} ${PI/4}"/-->
-                <!-- NEW URDF with mesh, REAL values measured from the edge of the robot -->
-                <!-- x = (500 - 153 - 61.77/2) / 1000	-->
-                <!-- y = from CAD -->
                 <origin xyz="0.316115 0.00 0.0887678" rpy="0 ${PI} ${PI/4}"/>
         </xacro:kvh_1775_imu>

Commit message: Params to make anymal work, pt2 fix the urdf

File: descriptions/anymal_description/robots/anymal.urdf.xacro (robot description, xacro)
@@ -105,5 +105,5 @@
         <inertial>
             <origin rpy="0 0 0" xyz="-0.001960558279 -0.001413217745 0.050207125344"/>
-            <mass value="16.793507758"/>
+            <mass value="40.793507758"/>
             <inertia ixx="0.217391101503" ixy="-0.00132873239126" ixz="-0.00228200226173" iyy="0.639432546734" iyz="-0.00138078263145" izz="0.62414077654"/>
         </inertial>
@@ -177,5 +177,5 @@
         <inertial>
             <origin rpy="0 0 0" xyz="-0.003897968082 0.054226618537 -0.214583373795"/>
-            <mass value="1.634976467"/>
+            <mass value="2.3"/>
             <inertia ixx="0.0120367944369" ixy="6.762065206e-05" ixz="0.000287806340448" iyy="0.0120643637939" iyz="-0.00140610131218" izz="0.00249422574881"/>
         </inertial>
@@ -330,5 +330,5 @@
         <inertial>
             <origin rpy="0 0 0" xyz="-0.003897968082 -0.054226618537 -0.214583373795"/>
-            <mass value="1.634976467"/>
+            <mass value="2.3"/>
             <inertia ixx="0.0120367944369" ixy="-6.762065206e-05" ixz="0.000287806340448" iyy="0.0120643637939" iyz="0.00140610131218" izz="0.00249422574881"/>
         </inertial>
@@ -483,5 +483,5 @@
         <inertial>
             <origin rpy="0 0 0" xyz="0.003897968082 0.054226618537 -0.214583373795"/>
-            <mass value="1.634976467"/>
+            <mass value="2.3"/>
             <inertia ixx="0.0120367944369" ixy="-6.762065206e-05" ixz="-0.000287806340448" iyy="0.0120643637939" iyz="-0.00140610131218" izz="0.00249422574881"/>
         </inertial>
@@ -636,5 +636,5 @@
         <inertial>
             <origin rpy="0 0 0" xyz="0.003897968082 -0.054226618537 -0.214583373795"/>
-            <mass value="1.634976467"/>
+            <mass value="2.3"/>
             <inertia ixx="0.0120367944369" ixy="6.762065206e-05" ixz="-0.000287806340448" iyy="0.0120643637939" iyz="0.00140610131218" izz="0.00249422574881"/>
         </inertial>

Commit message: Clean anymal launch and urdf

File: descriptions/anymal_description/robots/anymal.urdf.xacro (robot description, xacro)
@@ -730,20 +730,3 @@
     <xacro:leg_transmission name="lh"/>
     <xacro:leg_gazebo name="lh" load_force_sensors="$(arg load_force_sensors)"/>
-    <xacro:if value="$(arg sensors)">
-        <!-- IMU trunk -->
-        <xacro:microstrain_3dmgx425_imu
-                parent="base"
-                imu_name="trunk_imu"
-                imu_topic="trunk_imu_1/data"
-                update_rate="250">
-                <origin xyz="0.27025 0.000 0.0967678" rpy="0 0 0"/>
-        </xacro:microstrain_3dmgx425_imu>
-        <xacro:kvh_1775_imu
-                parent="base"
-                imu_name="kvh_imu"
-                imu_topic="kvh_imu/data"
-                update_rate="250">
-                <origin xyz="0.316115 0.00 0.0887678" rpy="0 ${PI} ${PI/4}"/>
-        </xacro:kvh_1775_imu>
-    </xacro:if>
 </robot>

Commit message: Working on anymal

File: descriptions/anymal_description/robots/anymal.urdf.xacro (robot description, xacro)
@@ -146,5 +146,5 @@
         <dynamics damping="0.0" friction="0.0"/>
     </joint>
-    <link name="lf_thigh">
+    <link name="lf_upperleg">
         <visual>
             <origin rpy="0 0 0.0" xyz="0 0 0"/>
@@ -155,5 +155,5 @@
         </visual>
         <collision>
-            <!-- thigh with heat fins -->
+            <!-- upperleg with heat fins -->
             <origin rpy="0.145 0 0" xyz="0 0.035 -0.125"/>
             <geometry>
@@ -181,8 +181,8 @@
         </inertial>
     </link>
-    <!-- Thigh joint -->
+    <!-- upperleg joint -->
     <joint name="lf_hfe_joint" type="revolute">
         <parent link="lf_hip"/>
-        <child link="lf_thigh"/>
+        <child link="lf_upperleg"/>
         <origin xyz="0.0635                    0.041                    0.0"/>
         <axis xyz="0 1 0"/>
@@ -190,5 +190,5 @@
         <dynamics damping="0.0" friction="0.0"/>
     </joint>
-    <link name="lf_shank">
+    <link name="lf_lowerleg">
         <visual>
             <origin rpy="0 0 0.0" xyz="0 0 0"/>
@@ -210,8 +210,8 @@
         </inertial>
     </link>
-    <!-- Shank joint -->
+    <!-- lowerleg joint -->
     <joint name="lf_kfe_joint" type="revolute">
-        <parent link="lf_thigh"/>
-        <child link="lf_shank"/>
+        <parent link="lf_upperleg"/>
+        <child link="lf_lowerleg"/>
         <origin xyz="0.0 0.109 -0.25"/>
         <axis xyz="0 1 0"/>
@@ -219,7 +219,7 @@
         <dynamics damping="0.0" friction="0.0"/>
     </joint>
-    <!-- Shank to Adapter joint -->
-    <joint name="lf_shank_to_adapter" type="fixed">
-        <parent link="lf_shank"/>
+    <!-- lowerleg to Adapter joint -->
+    <joint name="lf_lowerleg_to_adapter" type="fixed">
+        <parent link="lf_lowerleg"/>
         <child link="lf_adapter"/>
         <origin rpy="0.0 0.0 0.0" xyz="0.1 -0.02 0.0"/>
@@ -308,5 +308,5 @@
         </visual>
         <collision>
-            <!-- thigh with heat fins -->
+            <!-- upperleg with heat fins -->
             <origin rpy="-0.145 0 0" xyz="0 -0.035 -0.125"/>
             <geometry>
@@ -334,5 +334,5 @@
         </inertial>
     </link>
-    <!-- Thigh joint -->
+    <!-- upperleg joint -->
     <joint name="rf_hfe_joint" type="revolute">
         <parent link="rf_hip"/>
@@ -343,5 +343,5 @@
         <dynamics damping="0.0" friction="0.0"/>
     </joint>
-    <link name="rf_shank">
+    <link name="rf_lowerleg">
         <visual>
             <origin rpy="0 0 0.0" xyz="0 0 0"/>
@@ -363,8 +363,8 @@
         </inertial>
     </link>
-    <!-- Shank joint -->
+    <!-- lowerleg joint -->
     <joint name="rf_kfe_joint" type="revolute">
         <parent link="rf_tigh"/>
-        <child link="rf_shank"/>
+        <child link="rf_lowerleg"/>
         <origin xyz="0.0 -0.109 -0.25"/>
         <axis xyz="0 1 0"/>
@@ -372,7 +372,7 @@
         <dynamics damping="0.0" friction="0.0"/>
     </joint>
-    <!-- Shank to Adapter joint -->
-    <joint name="rf_shank_to_adapter" type="fixed">
-        <parent link="rf_shank"/>
+    <!-- lowerleg to Adapter joint -->
+    <joint name="rf_lowerleg_to_adapter" type="fixed">
+        <parent link="rf_lowerleg"/>
         <child link="rf_adapter"/>
         <origin rpy="-0.0 0.0 -0.0" xyz="0.1 0.02 0.0"/>
@@ -452,5 +452,5 @@
         <dynamics damping="0.0" friction="0.0"/>
     </joint>
-    <link name="lh_thigh">
+    <link name="lh_upperleg">
         <visual>
             <origin rpy="0 0 -3.14159265359" xyz="0 0 0"/>
@@ -461,5 +461,5 @@
         </visual>
         <collision>
-            <!-- thigh with heat fins -->
+            <!-- upperleg with heat fins -->
             <origin rpy="0.145 0 0" xyz="0 0.035 -0.125"/>
             <geometry>
@@ -487,8 +487,8 @@
         </inertial>
     </link>
-    <!-- Thigh joint -->
+    <!-- upperleg joint -->
     <joint name="lh_hfe_joint" type="revolute">
         <parent link="lh_hip"/>
-        <child link="lh_thigh"/>
+        <child link="lh_upperleg"/>
         <origin xyz="-0.0635                    0.041                    0.0"/>
         <axis xyz="0 1 0"/>
@@ -496,5 +496,5 @@
         <dynamics damping="0.0" friction="0.0"/>
     </joint>
-    <link name="lh_shank">
+    <link name="lh_lowerleg">
         <visual>
             <origin rpy="0 0 -3.14159265359" xyz="0 0 0"/>
@@ -516,8 +516,8 @@
         </inertial>
     </link>
-    <!-- Shank joint -->
+    <!-- lowerleg joint -->
     <joint name="lh_kfe_joint" type="revolute">
-        <parent link="lh_thigh"/>
-        <child link="lh_shank"/>
+        <parent link="lh_upperleg"/>
+        <child link="lh_lowerleg"/>
         <origin xyz="-0.0 0.109 -0.25"/>
         <axis xyz="0 1 0"/>
@@ -525,7 +525,7 @@
         <dynamics damping="0.0" friction="0.0"/>
     </joint>
-    <!-- Shank to Adapter joint -->
-    <joint name="lh_shank_to_adapter" type="fixed">
-        <parent link="lh_shank"/>
+    <!-- lowerleg to Adapter joint -->
+    <joint name="lh_lowerleg_to_adapter" type="fixed">
+        <parent link="lh_lowerleg"/>
         <child link="lh_adapter"/>
         <origin rpy="0.0 -0.0 -0.0" xyz="-0.1 -0.02 0.0"/>
@@ -605,5 +605,5 @@
         <dynamics damping="0.0" friction="0.0"/>
     </joint>
-    <link name="rh_thigh">
+    <link name="rh_upperleg">
         <visual>
             <origin rpy="0 0 -3.14159265359" xyz="0 0 0"/>
@@ -614,5 +614,5 @@
         </visual>
         <collision>
-            <!-- thigh with heat fins -->
+            <!-- upperleg with heat fins -->
             <origin rpy="-0.145 0 0" xyz="0 -0.035 -0.125"/>
             <geometry>
@@ -640,8 +640,8 @@
         </inertial>
     </link>
-    <!-- Thigh joint -->
+    <!-- upperleg joint -->
     <joint name="rh_hfe_joint" type="revolute">
         <parent link="rh_hip"/>
-        <child link="rh_thigh"/>
+        <child link="rh_upperleg"/>
         <origin xyz="-0.0635                    -0.041                    0.0"/>
         <axis xyz="0 1 0"/>
@@ -649,5 +649,5 @@
         <dynamics damping="0.0" friction="0.0"/>
     </joint>
-    <link name="rh_shank">
+    <link name="rh_lowerleg">
         <visual>
             <origin rpy="0 0 -3.14159265359" xyz="0 0 0"/>
@@ -669,8 +669,8 @@
         </inertial>
     </link>
-    <!-- Shank joint -->
+    <!-- lowerleg joint -->
     <joint name="rh_kfe_joint" type="revolute">
-        <parent link="rh_thigh"/>
-        <child link="rh_shank"/>
+        <parent link="rh_upperleg"/>
+        <child link="rh_lowerleg"/>
         <origin xyz="-0.0 -0.109 -0.25"/>
         <axis xyz="0 1 0"/>
@@ -678,7 +678,7 @@
         <dynamics damping="0.0" friction="0.0"/>
     </joint>
-    <!-- Shank to Adapter joint -->
-    <joint name="rh_shank_to_adapter" type="fixed">
-        <parent link="rh_shank"/>
+    <!-- lowerleg to Adapter joint -->
+    <joint name="rh_lowerleg_to_adapter" type="fixed">
+        <parent link="rh_lowerleg"/>
         <child link="rh_adapter"/>
         <origin rpy="-0.0 -0.0 0.0" xyz="-0.1 0.02 0.0"/>

Commit message: Fix names in anymal

File: descriptions/anymal_description/robots/anymal.urdf.xacro (robot description, xacro)
@@ -299,5 +299,5 @@
         <dynamics damping="0.0" friction="0.0"/>
     </joint>
-    <link name="rf_tigh">
+    <link name="rf_upperleg">
         <visual>
             <origin rpy="0 0 0.0" xyz="0 0 0"/>
@@ -337,5 +337,5 @@
     <joint name="rf_hfe_joint" type="revolute">
         <parent link="rf_hip"/>
-        <child link="rf_tigh"/>
+        <child link="rf_upperleg"/>
         <origin xyz="0.0635                    -0.041                    0.0"/>
         <axis xyz="0 1 0"/>
@@ -365,5 +365,5 @@
     <!-- lowerleg joint -->
     <joint name="rf_kfe_joint" type="revolute">
-        <parent link="rf_tigh"/>
+        <parent link="rf_upperleg"/>
         <child link="rf_lowerleg"/>
         <origin xyz="0.0 -0.109 -0.25"/>

Commit message: ported anymal to 20.04. Looks not tuned properly

File: descriptions/anymal_description/robots/anymal.urdf.xacro (robot description, xacro)
@@ -8,4 +8,5 @@
     <xacro:arg name="load_force_sensors" default="false"/>
     <xacro:arg name="task_period" default="0.004"/>
+    <xacro:arg name="floating_base_link" default="true"/>
     <!-- generic simulator_gazebo plugins for starting mechanism control, ros time -->
     <xacro:include filename="$(find anymal_description)/gazebo/gazebo.urdf.xacro">
@@ -83,10 +84,12 @@
     </link>
     <!-- Floating-base Joint -->
-    <link name="world"/>
-    <joint name="floating_base_joint" type="floating">
-      <origin rpy="0 0 0" xyz="0 0 0"/>
-      <parent link="world"/>
-      <child link="base_link"/>
-    </joint>
+    <xacro:if value="$(arg floating_base_link)">
+	    <link name="world"/>
+	    <joint name="floating_base_joint" type="floating">
+	      <origin rpy="0 0 0" xyz="0 0 0"/>
+	      <parent link="world"/>
+	      <child link="base_link"/>
+	    </joint>
+    </xacro:if>
     <joint name="floating_base" type="fixed">
       <origin rpy="0 0 0" xyz="0 0 0"/>
