Commit message: Remove damping from the urdf

File: descriptions/hyq_description/urdfs/leg/leg.urdf.xacro (robot description, xacro)
@@ -15,5 +15,5 @@
 			<axis xyz="0 0 1"/>
 			<limit effort="${haa_limit}" velocity="12.0" lower="${haa_min*PI/180}" upper="${haa_max*PI/180}" />
-			<dynamics damping="0.1" friction="0" />
+                        <dynamics damping="0.0" friction="0" />
 			<safety_controller k_position="50" k_velocity="10"
 							   soft_lower_limit="${haa_min*PI/180}" soft_upper_limit="${haa_max*PI/180}" />
@@ -28,5 +28,5 @@
                   lower="${(1-knee_bent_backward)*(hfe_min)*PI/180 + (knee_bent_backward)*(-hfe_max)*PI/180}"
                   upper="${(1-knee_bent_backward)*(hfe_max)*PI/180 + (knee_bent_backward)*(-hfe_min)*PI/180}"/>
-			<dynamics damping="0.1" friction="0" />
+                        <dynamics damping="0.0" friction="0" />
 			<safety_controller k_position="50" k_velocity="10"
                   soft_lower_limit="${(1-knee_bent_backward)*(hfe_min)*PI/180 + (knee_bent_backward)*(-hfe_max)*PI/180}"
@@ -42,5 +42,5 @@
                   lower="${(1-knee_bent_backward)*(kfe_min)*PI/180 + (knee_bent_backward)*(-kfe_max)*PI/180}"
                   upper="${(1-knee_bent_backward)*(kfe_max)*PI/180 + (knee_bent_backward)*(-kfe_min)*PI/180}"/>
-			<dynamics damping="0.1" friction="0" />
+                        <dynamics damping="0.0" friction="0" />
 			<safety_controller k_position="50" k_velocity="10"
                   soft_lower_limit="${(1-knee_bent_backward)*(kfe_min)*PI/180 + (knee_bent_backward)*(-kfe_max)*PI/180}"
