Commit message: Fix teleop_urdf -> teleop_description

File: descriptions/teleop_description/urdf/parts/arm.urdf.xacro (robot description, xacro)
@@ -24,5 +24,5 @@
       <origin xyz="0 0 0" rpy="${PI_2} 0 0"/>
       <geometry name="teleop_link0_visual">
-        <mesh filename="package://teleop_urdf/meshes/_teleop_link0.stl" scale="0.001 0.001 0.001" />
+        <mesh filename="package://teleop_description/meshes/_teleop_link0.stl" scale="0.001 0.001 0.001" />
       </geometry>
       <material name="red"/>
@@ -31,5 +31,5 @@
       <origin xyz="0 0 0" rpy="${PI_2} 0 0"/>
       <geometry name="teleop_link0_collision">
-        <mesh filename="package://teleop_urdf/meshes/simple/_teleop_link0.stl" scale="0.001 0.001 0.001" />
+        <mesh filename="package://teleop_description/meshes/simple/_teleop_link0.stl" scale="0.001 0.001 0.001" />
       </geometry>
     </collision>
@@ -44,5 +44,5 @@
       <origin xyz="0 0 0" rpy="${PI_2} 0 ${-PI_2}"/>
       <geometry name="teleop_link1_visual">
-        <mesh filename="package://teleop_urdf/meshes/_teleop_link1.stl" scale="0.001 0.001 0.001" />
+        <mesh filename="package://teleop_description/meshes/_teleop_link1.stl" scale="0.001 0.001 0.001" />
       </geometry>
       <material name="red"/>
@@ -51,5 +51,5 @@
       <origin xyz="0 0 0" rpy="${PI_2} 0 ${-PI_2}"/>
       <geometry name="teleop_link1_collision">
-        <mesh filename="package://teleop_urdf/meshes/simple/_teleop_link1.stl" scale="0.001 0.001 0.001" />
+        <mesh filename="package://teleop_description/meshes/simple/_teleop_link1.stl" scale="0.001 0.001 0.001" />
       </geometry>
     </collision>
@@ -64,5 +64,5 @@
       <origin xyz="0 0 0" rpy="${PI_2} 0 0"/>
       <geometry name="teleop_link2_visual">
-        <mesh filename="package://teleop_urdf/meshes/_teleop_link2.stl" scale="0.001 0.001 0.001" />
+        <mesh filename="package://teleop_description/meshes/_teleop_link2.stl" scale="0.001 0.001 0.001" />
       </geometry>
       <material name="red"/>
@@ -71,5 +71,5 @@
       <origin xyz="0 0 0" rpy="${PI_2} 0 0"/>
       <geometry name="teleop_link2_collision">
-        <mesh filename="package://teleop_urdf/meshes/simple/_teleop_link2.stl" scale="0.001 0.001 0.001" />
+        <mesh filename="package://teleop_description/meshes/simple/_teleop_link2.stl" scale="0.001 0.001 0.001" />
       </geometry>
     </collision>
@@ -84,5 +84,5 @@
       <origin xyz="0 0 0" rpy="${PI_2} 0 0"/>
       <geometry name="teleop_link3_visual">
-        <mesh filename="package://teleop_urdf/meshes/_teleop_link3.stl" scale="0.001 0.001 0.001" />
+        <mesh filename="package://teleop_description/meshes/_teleop_link3.stl" scale="0.001 0.001 0.001" />
       </geometry>
       <material name="red"/>
@@ -91,5 +91,5 @@
       <origin xyz="0 0 0" rpy="${PI_2} 0 0"/>
       <geometry name="teleop_link3_collision">
-        <mesh filename="package://teleop_urdf/meshes/simple/_teleop_link3.stl" scale="0.001 0.001 0.001" />
+        <mesh filename="package://teleop_description/meshes/simple/_teleop_link3.stl" scale="0.001 0.001 0.001" />
       </geometry>
     </collision>
@@ -104,5 +104,5 @@
       <origin xyz="0 0 0" rpy="${PI_2} 0 0"/>
       <geometry name="teleop_link4_visual">
-        <mesh filename="package://teleop_urdf/meshes/_teleop_link4.stl" scale="0.001 0.001 0.001" />
+        <mesh filename="package://teleop_description/meshes/_teleop_link4.stl" scale="0.001 0.001 0.001" />
       </geometry>
       <material name="red"/>
@@ -111,5 +111,5 @@
       <origin xyz="0 0 0" rpy="${PI_2} 0 0"/>
       <geometry name="teleop_link4_collision">
-        <mesh filename="package://teleop_urdf/meshes/simple/_teleop_link4.stl" scale="0.001 0.001 0.001" />
+        <mesh filename="package://teleop_description/meshes/simple/_teleop_link4.stl" scale="0.001 0.001 0.001" />
       </geometry>
     </collision>
@@ -125,5 +125,5 @@
       <origin xyz="0 0 0" rpy="${PI_2} 0 ${PI}"/>
       <geometry name="teleop_link5_visual">
-        <mesh filename="package://teleop_urdf/meshes/_teleop_link5.stl" scale="0.001 0.001 0.001" />
+        <mesh filename="package://teleop_description/meshes/_teleop_link5.stl" scale="0.001 0.001 0.001" />
       </geometry>
       <material name="red"/>
@@ -132,5 +132,5 @@
       <origin xyz="0 0 0" rpy="${PI_2} 0 ${PI}"/>
       <geometry name="teleop_link5_collision">
-        <mesh filename="package://teleop_urdf/meshes/simple/_teleop_link5.stl" scale="0.001 0.001 0.001" />
+        <mesh filename="package://teleop_description/meshes/simple/_teleop_link5.stl" scale="0.001 0.001 0.001" />
       </geometry>
     </collision>
@@ -146,5 +146,5 @@
       <origin xyz="0 0 0" rpy="${PI_2} 0 ${PI}"/>
       <geometry name="teleop_link5_visual">
-        <mesh filename="package://teleop_urdf/meshes/_teleop_link5.stl" scale="0.001 0.001 0.001" />
+        <mesh filename="package://teleop_description/meshes/_teleop_link5.stl" scale="0.001 0.001 0.001" />
       </geometry>
       <material name="red"/>
@@ -153,5 +153,5 @@
       <origin xyz="0 0 0" rpy="${PI_2} 0 ${PI}"/>
       <geometry name="teleop_link5_collision">
-        <mesh filename="package://teleop_urdf/meshes/simple/_teleop_link5.stl" scale="0.001 0.001 0.001" />
+        <mesh filename="package://teleop_description/meshes/simple/_teleop_link5.stl" scale="0.001 0.001 0.001" />
       </geometry>
     </collision>

File: descriptions/teleop_description/urdf/teleop.urdf.xacro (robot description, xacro)
@@ -8,7 +8,7 @@
 -->
 <!-- ************ MODEL CONFIGURATION ************ -->
-<xacro:include filename="$(find teleop_urdf)/urdf/teleop_config.urdf.xacro" />
+<xacro:include filename="$(find teleop_description)/urdf/teleop_config.urdf.xacro" />
 <!-- ************ TELEOP BASE ************** -->
-<xacro:include filename="$(find teleop_urdf)/urdf/teleop_base.urdf.xacro"/>
+<xacro:include filename="$(find teleop_description)/urdf/teleop_base.urdf.xacro"/>
 <xacro:if value="${TELEOP_FLOATING_BASE}" >
 	<link name="world"/>

File: descriptions/teleop_description/urdf/teleop_base.urdf.xacro (robot description, xacro)
@@ -24,4 +24,4 @@
 </xacro:if>
 <!-- SELECTION OF KINEMATICS CHAINS IS HANDLED INSIDE THE FILES -->
-<xacro:include filename="$(find teleop_urdf)/urdf/parts/arm.urdf.xacro" />
+<xacro:include filename="$(find teleop_description)/urdf/parts/arm.urdf.xacro" />
 </robot>

File: descriptions/teleop_description/urdf/teleop_robot.urdf.xacro (robot description, xacro)
@@ -6,8 +6,8 @@
   This file groups files to use COGIMON in GAZEBO
   -->
-  <xacro:include filename="$(find teleop_urdf)/urdf/teleop.urdf.xacro" />
-  <xacro:include filename="$(find teleop_urdf)/urdf/gazebo/teleop.gazebo.xacro" />
-  <xacro:include filename="$(find teleop_urdf)/urdf/gazebo/teleop_materials.gazebo.xacro" />
+  <xacro:include filename="$(find teleop_description)/urdf/teleop.urdf.xacro" />
+  <xacro:include filename="$(find teleop_description)/urdf/gazebo/teleop.gazebo.xacro" />
+  <xacro:include filename="$(find teleop_description)/urdf/gazebo/teleop_materials.gazebo.xacro" />
   <!--xacro:include filename="$(find cogimon_urdf)/urdf/gazebo/force_torque.gazebo.xacro" /-->
-  <xacro:include filename="$(find teleop_urdf)/urdf/gazebo/xbot_control.gazebo.xacro" />
+  <xacro:include filename="$(find teleop_description)/urdf/gazebo/xbot_control.gazebo.xacro" />
 </robot>
