Commit message: Initial position for kinova arm

File: descriptions/hyq_description/robots/hyq_kinova.srdf.xacro (robot description, xacro)
@@ -41,7 +41,7 @@
     <joint name="rh_kfe_joint" value="1.5"/>
     <joint name="kinova_joint_1" value="0.0"/>
-    <joint name="kinova_joint_2" value="0.0"/>
-    <joint name="kinova_joint_3" value="0.0"/>
-    <joint name="kinova_joint_4" value="0.0"/>
+    <joint name="kinova_joint_2" value="1.80"/>
+    <joint name="kinova_joint_3" value="4.0"/>
+    <joint name="kinova_joint_4" value="-1.5"/>
   </group_state>
 </robot>

Commit message: Work in progress to adapt to the new robot model

File: descriptions/hyq_description/robots/hyq_kinova.srdf.xacro (robot description, xacro)
@@ -19,4 +19,16 @@
   <group name="rh_leg">
     <chain base_link="trunk" tip_link="rh_foot"/>
+  </group>
+  <group name="feet">
+    <link name="lf_foot"/>
+    <link name="rf_foot"/>
+    <link name="lh_foot"/>
+    <link name="rh_foot"/>
+  </group>
+  <group name="hips">
+    <link name="lf_hipassembly"/>
+    <link name="rf_hipassembly"/>
+    <link name="lh_hipassembly"/>
+    <link name="rh_hipassembly"/>
   </group>
   <group name="legs">

File: descriptions/hyq_description/robots/hyq_teleop.srdf.xacro (robot description, xacro)
@@ -5,25 +5,46 @@
     <link name="teleop_link0"/>
   </group>
-  <group name="arm">
-       <chain base_link="teleop_link0" tip_link="TCP"/>
+  <group name="teleop_arm">
+    <chain base_link="teleop_link0" tip_link="TCP"/>
   </group>
-  <group name="lf">
+  <group name="lf_leg">
     <chain base_link="trunk" tip_link="lf_foot"/>
   </group>
-  <group name="rf">
+  <group name="rf_leg">
     <chain base_link="trunk" tip_link="rf_foot"/>
   </group>
-  <group name="lh">
+  <group name="lh_leg">
     <chain base_link="trunk" tip_link="lh_foot"/>
   </group>
-  <group name="rh">
+  <group name="rh_leg">
     <chain base_link="trunk" tip_link="rh_foot"/>
   </group>
+  <group name="lf_hip">
+    <chain base_link="trunk" tip_link="lf_hipassembly"/>
+  </group>
+  <group name="rf_hip">
+    <chain base_link="trunk" tip_link="rf_hipassembly"/>
+  </group>
+  <group name="lh_hip">
+    <chain base_link="trunk" tip_link="lh_hipassembly"/>
+  </group>
+  <group name="rh_hip">
+    <chain base_link="trunk" tip_link="rh_hipassembly"/>
+  </group>
+  <group name="legs">
+    <group name="lf_leg"/>
+    <group name="rf_leg"/>
+    <group name="lh_leg"/>
+    <group name="rh_leg"/>
+  </group>
+  <group name="arms">
+    <group name="teleop_arm"/>
+  </group>
   <group name="chains">
-    <group name="lf"/>
-    <group name="rf"/>
-    <group name="lh"/>
-    <group name="rh"/>
-    <group name="arm"/>
+    <group name="lf_leg"/>
+    <group name="rf_leg"/>
+    <group name="lh_leg"/>
+    <group name="rh_leg"/>
+    <group name="teleop_arm"/>
   </group>
   <group_state group="chains" name="home">
