Commit message: Fix homing position for hyq

File: descriptions/hyq_description/robots/hyq.srdf.xacro (robot description, xacro)
@@ -30,9 +30,9 @@
     <joint name="rf_kfe_joint" value="-1.5"/>
     <joint name="lh_haa_joint" value="-0.2"/>
-    <joint name="lh_hfe_joint" value="0.75"/>
-    <joint name="lh_kfe_joint" value="-1.5"/>
+    <joint name="lh_hfe_joint" value="-0.75"/>
+    <joint name="lh_kfe_joint" value="1.5"/>
     <joint name="rh_haa_joint" value="-0.2"/>
-    <joint name="rh_hfe_joint" value="0.75"/>
-    <joint name="rh_kfe_joint" value="-1.5"/>
+    <joint name="rh_hfe_joint" value="-0.75"/>
+    <joint name="rh_kfe_joint" value="1.5"/>
   </group_state>
 </robot>

Commit message: Working on quadruped robot class

File: descriptions/hyq_description/robots/hyq.srdf.xacro (robot description, xacro)
@@ -4,21 +4,39 @@
     <link name="base_link"/>
   </group>
-  <group name="lf">
+  <group name="lf_leg">
     <chain base_link="trunk" tip_link="lf_foot"/>
   </group>
-  <group name="rf">
+  <group name="rf_leg">
     <chain base_link="trunk" tip_link="rf_foot"/>
   </group>
-  <group name="lh">
+  <group name="lh_leg">
     <chain base_link="trunk" tip_link="lh_foot"/>
   </group>
-  <group name="rh">
+  <group name="rh_leg">
     <chain base_link="trunk" tip_link="rh_foot"/>
   </group>
+  <group name="lf_hip">
+    <chain base_link="trunk" tip_link="lf_hipassembly"/>
+  </group>
+  <group name="rf_hip">
+    <chain base_link="trunk" tip_link="rf_hipassembly"/>
+  </group>
+  <group name="lh_hip">
+    <chain base_link="trunk" tip_link="lh_hipassembly"/>
+  </group>
+  <group name="rh_hip">
+    <chain base_link="trunk" tip_link="rh_hipassembly"/>
+  </group>
+  <group name="legs">
+    <group name="lf_leg"/>
+    <group name="rf_leg"/>
+    <group name="lh_leg"/>
+    <group name="rh_leg"/>
+  </group>
   <group name="chains">
-    <group name="lf"/>
-    <group name="rf"/>
-    <group name="lh"/>
-    <group name="rh"/>
+    <group name="lf_leg"/>
+    <group name="rf_leg"/>
+    <group name="lh_leg"/>
+    <group name="rh_leg"/>
   </group>
   <group_state group="chains" name="home">

File: descriptions/hyq_description/robots/hyq_kinova.srdf.xacro (robot description, xacro)
@@ -20,15 +20,15 @@
     <chain base_link="trunk" tip_link="rh_foot"/>
   </group>
-  <group name="feet">
-    <link name="lf_foot"/>
-    <link name="rf_foot"/>
-    <link name="lh_foot"/>
-    <link name="rh_foot"/>
+  <group name="lf_hip">
+    <chain base_link="trunk" tip_link="lf_hipassembly"/>
   </group>
-  <group name="hips">
-    <link name="lf_hipassembly"/>
-    <link name="rf_hipassembly"/>
-    <link name="lh_hipassembly"/>
-    <link name="rh_hipassembly"/>
+  <group name="rf_hip">
+    <chain base_link="trunk" tip_link="rf_hipassembly"/>
+  </group>
+  <group name="lh_hip">
+    <chain base_link="trunk" tip_link="lh_hipassembly"/>
+  </group>
+  <group name="rh_hip">
+    <chain base_link="trunk" tip_link="rh_hipassembly"/>
   </group>
   <group name="legs">

Commit message: Update xacros

File: descriptions/hyq_description/robots/hyq.srdf.xacro (robot description, xacro)
@@ -6,13 +6,25 @@
   <group name="lf_leg">
     <chain base_link="trunk" tip_link="lf_foot"/>
+    <joint name="lf_haa_joint"/>
+    <joint name="lf_hfe_joint"/>
+    <joint name="lf_kfe_joint"/>
   </group>
   <group name="rf_leg">
     <chain base_link="trunk" tip_link="rf_foot"/>
+    <joint name="rf_haa_joint"/>
+    <joint name="rf_hfe_joint"/>
+    <joint name="rf_kfe_joint"/>
   </group>
   <group name="lh_leg">
     <chain base_link="trunk" tip_link="lh_foot"/>
+    <joint name="lh_haa_joint"/>
+    <joint name="lh_hfe_joint"/>
+    <joint name="lh_kfe_joint"/>
   </group>
   <group name="rh_leg">
     <chain base_link="trunk" tip_link="rh_foot"/>
+    <joint name="rh_haa_joint"/>
+    <joint name="rh_hfe_joint"/>
+    <joint name="rh_kfe_joint"/>
   </group>
   <group name="lf_hip">

File: descriptions/hyq_description/robots/hyq_kinova.srdf.xacro (robot description, xacro)
@@ -1,22 +1,38 @@
 <?xml version="1.0" ?>
 <robot name="hyq" xmlns:xacro="http://ros.org/wiki/xacro">
-  <group name="base">
-    <link name="base_link"/>
-    <link name="kinova_link_base"/>
-  </group>
+ <group name="bases">
+   <link name="base_link"/>
+   <link name="kinova_link_base"/>
+ </group>
   <group name="kinova_arm">
     <chain base_link="kinova_link_base" tip_link="kinova_end_effector"/>
+    <joint name="kinova_joint_1"/>
+    <joint name="kinova_joint_2"/>
+    <joint name="kinova_joint_3"/>
+    <joint name="kinova_joint_4"/>
   </group>
   <group name="lf_leg">
     <chain base_link="trunk" tip_link="lf_foot"/>
+    <joint name="lf_haa_joint"/>
+    <joint name="lf_hfe_joint"/>
+    <joint name="lf_kfe_joint"/>
   </group>
   <group name="rf_leg">
     <chain base_link="trunk" tip_link="rf_foot"/>
+    <joint name="rf_haa_joint"/>
+    <joint name="rf_hfe_joint"/>
+    <joint name="rf_kfe_joint"/>
   </group>
   <group name="lh_leg">
     <chain base_link="trunk" tip_link="lh_foot"/>
+    <joint name="lh_haa_joint"/>
+    <joint name="lh_hfe_joint"/>
+    <joint name="lh_kfe_joint"/>
   </group>
   <group name="rh_leg">
     <chain base_link="trunk" tip_link="rh_foot"/>
+    <joint name="rh_haa_joint"/>
+    <joint name="rh_hfe_joint"/>
+    <joint name="rh_kfe_joint"/>
   </group>
   <group name="lf_hip">

File: descriptions/hyq_description/robots/hyq_teleop.srdf.xacro (robot description, xacro)
@@ -1,5 +1,5 @@
 <?xml version="1.0" ?>
 <robot name="hyq" xmlns:xacro="http://ros.org/wiki/xacro">
-  <group name="base">
+  <group name="bases">
     <link name="base_link"/>
     <link name="teleop_link0"/>
@@ -7,16 +7,33 @@
   <group name="teleop_arm">
     <chain base_link="teleop_link0" tip_link="TCP"/>
+    <joint name="joint1"/>
+    <joint name="joint2"/>
+    <joint name="joint3"/>
+    <joint name="joint4"/>
+    <joint name="joint5"/>
   </group>
   <group name="lf_leg">
     <chain base_link="trunk" tip_link="lf_foot"/>
+    <joint name="lf_haa_joint"/>
+    <joint name="lf_hfe_joint"/>
+    <joint name="lf_kfe_joint"/>
   </group>
   <group name="rf_leg">
     <chain base_link="trunk" tip_link="rf_foot"/>
+    <joint name="rf_haa_joint"/>
+    <joint name="rf_hfe_joint"/>
+    <joint name="rf_kfe_joint"/>
   </group>
   <group name="lh_leg">
     <chain base_link="trunk" tip_link="lh_foot"/>
+    <joint name="lh_haa_joint"/>
+    <joint name="lh_hfe_joint"/>
+    <joint name="lh_kfe_joint"/>
   </group>
   <group name="rh_leg">
     <chain base_link="trunk" tip_link="rh_foot"/>
+    <joint name="rh_haa_joint"/>
+    <joint name="rh_hfe_joint"/>
+    <joint name="rh_kfe_joint"/>
   </group>
   <group name="lf_hip">
