Commit message: teleop and full distro

File: descriptions/hyq_description/robots/hyq.urdf.xacro (robot description, xacro)
@@ -1,5 +1,7 @@
 <?xml version="1.0"?>
 <robot name="hyq" xmlns:xacro="http://ros.org/wiki/xacro">
-<xacro:arg name="task_period" default="0.004"/>
+	<xacro:arg name="task_period" default="0.004"/>
+	<xacro:arg name="sensors" default="true"/>
+	<xacro:arg name="arm" default="false"/>
 	<!-- This argument allows us to load joint sensors that measure the internal wrenches -->
 	<xacro:arg name="load_force_sensors" default="false"/>
@@ -81,4 +83,19 @@
 		<origin xyz="${-d_fh/2} ${-d_lr/2} 0" rpy="0 ${PI/2} 0"/>
 	</xacro:hyq_leg>
+<xacro:if value="$(arg arm)">
+	<joint name="joint_base_robots" type="fixed">
+	    	<parent link="base_link"/>
+	    	<child link="teleop_link0"/>
+   	 	<origin xyz="0.59 0 0" rpy="0 0 0"/>
+    	</joint>
+	<!-- SELECTION OF KINEMATICS CHAINS IS HANDLED INSIDE THE FILES -->
+	<xacro:include filename="$(find teleop_urdf)/urdf/teleop.urdf.xacro" />
+        <xacro:include filename="$(find hyq_description)/urdfs/arm/arm.transmission.xacro"/>
+        <xacro:arm_transmission name="joint1"/>
+        <xacro:arm_transmission name="joint2"/>
+        <xacro:arm_transmission name="joint3"/>
+        <xacro:arm_transmission name="joint4"/>
+        <xacro:arm_transmission name="joint5"/>
+</xacro:if>
 <xacro:if value="$(arg sensors)">
 	<!-- IMU trunk -->

Commit message: Remove sensors description

File: descriptions/hyq_description/robots/hyq.urdf.xacro (robot description, xacro)
@@ -2,5 +2,4 @@
 <robot name="hyq" xmlns:xacro="http://ros.org/wiki/xacro">
 	<xacro:arg name="task_period" default="0.004"/>
-	<xacro:arg name="sensors" default="true"/>
         <xacro:arg name="arm_enabled" default="false"/>
         <xacro:arg name="arm_name" default="teleop"/>
@@ -14,13 +13,4 @@
 	<!-- HyQ legs -->
 	<xacro:include filename="$(find hyq_description)/urdfs/leg/leg.urdf.xacro"/>
-	<!-- HyQ sensors -->
-        <xacro:if value="$(arg sensors)">
-            <xacro:include filename="$(find sensors_description)/urdfs/sensors/microstrain_3dmgx425_imu.urdf.xacro"/>
-            <xacro:include filename="$(find sensors_description)/urdfs/sensors/kvh_1775_imu.urdf.xacro"/>
-            <xacro:include filename="$(find sensors_description)/urdfs/sensors/asus_xtion.urdf.xacro"/>
-            <!-- we may mount the hokuyo again in the future -->
-            <!--xacro:include filename="$(find sensors_description)/urdfs/sensors/hokuyo_laser.urdf.xacro"/-->
-            <xacro:include filename="$(find sensors_description)/urdfs/sensors/multisense_sl.urdf.xacro"/>
-        </xacro:if>
 	<!-- generic simulator_gazebo plugins for starting mechanism control, ros time -->
         <xacro:include filename="$(find hyq_description)/gazebo/gazebo.urdf.xacro">
@@ -87,55 +77,3 @@
                <xacro:include filename="$(find hyq_description)/urdfs/arm/$(arg arm_name)_adapter.urdf.xacro" /> -->
         </xacro:if>
-<xacro:if value="$(arg sensors)">
-	<!-- IMU trunk -->
-        <xacro:microstrain_3dmgx425_imu
-		parent="trunk"
-		imu_name="trunk_imu"
-		imu_topic="trunk_imu_1/data"
-		update_rate="250">
-		<!-- old URDF -->
-		<!--origin xyz="0.290 0.000 0.0999214" rpy="0 ${-PI} 0"/ -->
-		<!-- new URDF with ideal values from CAD -->
-                <!--origin xyz="0.28525 0.000 0.0967678" rpy="0 0 0"/-->
-		<!-- new URDF, REAL values manually measured from the edge of the robot -->
-                <origin xyz="0.27025 0.000 0.0967678" rpy="0 0 0"/>
-        </xacro:microstrain_3dmgx425_imu>
-        <!-- IMU trunk -->
-        <!-- TODO We have to substitute the microstrain IMU with this one. Note that the imu_name has to be
-                  trunk_imu because the DLS HW interfaces hardcoded that name -->
-    	<xacro:kvh_1775_imu
-                parent="trunk"
-                imu_name="kvh_imu"
-                imu_topic="kvh_imu/data"
-                update_rate="250">
-	    <!-- OLD URDF with manually created cylinder -->
-            <!--origin xyz="0.352845 0.0029 0.0503678" rpy="0 ${-PI} 0"/-->
-            <!-- NEW URDF with mesh, ideal values from CAD -->
-            <!--origin xyz="0.36347 0.00 0.0887678" rpy="0 ${PI} ${PI/4}"/-->
-	    	<!-- NEW URDF with mesh, REAL values measured from the edge of the robot -->
-		<!-- x = (500 - 153 - 61.77/2) / 1000	-->
-		<!-- y = from CAD -->
-		<origin xyz="0.316115 0.00 0.0887678" rpy="0 ${PI} ${PI/4}"/>
-        </xacro:kvh_1775_imu>
-	<!-- Hokuyo -->
-	<!--xacro:hokuyo_laser
-		name="laser"
-		parent="trunk"
-		ros_topic="scan"
-		update_rate="10"
-		min_angle="-5"
-		max_angle="5"
-		range="4.0">
-            <origin xyz="0.475 0.0 -0.08823" rpy="${PI} 0.0 0"/>
-	</xacro:hokuyo_laser-->
-        <xacro:multisense_sl parent="trunk" prefix="multisense">
-		<!-- taken from head calibration (with vicon) -->
-		<!--origin xyz="0.761 -0.013 0.127" rpy="-0.002799508 0.514994302 -0.013000958" /-->
-		<origin xyz="0.775883 0.000304069 0.147268" rpy="-0.0145379 0.52898 0.0107014"/>
-        </xacro:multisense_sl>
-	<!-- Asus Xtion Pro -->
-	<xacro:asus_xtion_camera name="asus" parent="trunk">
-		<origin xyz="0.660678 -0.00571526 0.0705706" rpy="0.0364271 1.00115 0.0827391"/>
-	</xacro:asus_xtion_camera>
-    </xacro:if>
 </robot>

File: descriptions/hyq_description/urdfs/common.xacro (robot description, xacro)
@@ -2,15 +2,15 @@
 <robot xmlns:xacro="http://ros.org/wiki/xacro">
 	<xacro:property name="PI" value="3.1415926535897931"/>
-    <!-- kin limits (sign ref is RH leg)-->
-    <xacro:property name="haa_max" value="25"/>
-    <xacro:property name="haa_min" value="-70"/>
-    <xacro:property name="hfe_max" value="50"/>
-    <xacro:property name="hfe_min" value="-70"/>
-    <xacro:property name="kfe_max" value="140"/>
-    <xacro:property name="kfe_min" value="20"/>
-    <!-- torque limits 120-->
-    <xacro:property name="haa_limit" value="150"/>
-    <xacro:property name="hfe_limit" value="150"/>
-    <xacro:property name="kfe_limit" value="150"/>
+        <!-- kin limits (sign ref is RH leg)-->
+        <xacro:property name="haa_max" value="25"/>
+        <xacro:property name="haa_min" value="-70"/>
+        <xacro:property name="hfe_max" value="50"/>
+        <xacro:property name="hfe_min" value="-70"/>
+        <xacro:property name="kfe_max" value="140"/>
+        <xacro:property name="kfe_min" value="20"/>
+        <!-- torque limits 120-->
+        <xacro:property name="haa_limit" value="150"/>
+        <xacro:property name="hfe_limit" value="150"/>
+        <xacro:property name="kfe_limit" value="150"/>
 	<!-- standard distances -->
 	<xacro:property name="d_lr" value="0.414"/>
