Commit message: Add spot!

File: descriptions/spot_description/gazebo/gazebo.urdf.xacro (robot description, xacro)
@@ -10,5 +10,5 @@
 		<plugin filename="libgazebo_ros_p3d.so" name="gazebo_ros_p3d">
                         <robotNamespace>/spot</robotNamespace>
-                        <bodyName>body</bodyName>
+                        <bodyName>base_link</bodyName>
 			<topicName>ground_truth</topicName>
 			<frameName>world</frameName>

File: descriptions/spot_description/robots/spot.srdf.xacro (robot description, xacro)
@@ -6,26 +6,26 @@
     </group>
     <group name="lf_leg">
-      <chain base_link="body" tip_link="lf_foot"/>
+      <chain base_link="base_link" tip_link="lf_foot"/>
     </group>
     <group name="rf_leg">
-      <chain base_link="body" tip_link="rf_foot"/>
+      <chain base_link="base_link" tip_link="rf_foot"/>
     </group>
     <group name="lh_leg">
-      <chain base_link="body" tip_link="lh_foot"/>
+      <chain base_link="base_link" tip_link="lh_foot"/>
     </group>
     <group name="rh_leg">
-      <chain base_link="body" tip_link="rh_foot"/>
+      <chain base_link="base_link" tip_link="rh_foot"/>
     </group>
     <group name="lf_hip">
-      <chain base_link="body" tip_link="lf_hip"/>
+      <chain base_link="base_link" tip_link="lf_hip"/>
     </group>
     <group name="rf_hip">
-      <chain base_link="body" tip_link="rf_hip"/>
+      <chain base_link="base_link" tip_link="rf_hip"/>
     </group>
     <group name="lh_hip">
-      <chain base_link="body" tip_link="lh_hip"/>
+      <chain base_link="base_link" tip_link="lh_hip"/>
     </group>
     <group name="rh_hip">
-      <chain base_link="body" tip_link="rh_hip"/>
+      <chain base_link="base_link" tip_link="rh_hip"/>
     </group>
     <group name="legs">

File: descriptions/spot_description/robots/spot.urdf.xacro (robot description, xacro)
@@ -60,4 +60,5 @@
     <!-- foot -->
     <xacro:property name="foot_mass" value="0.06"/>
+    <xacro:property name="foot_radius" value="0.034"/>
     <!-- Floating-base Joint -->
     <link name="world"/>
@@ -65,7 +66,7 @@
       <origin rpy="0 0 0" xyz="0 0 0"/>
       <parent link="world"/>
-      <child link="body"/>
-    </joint>
-    <link name="body">
+      <child link="base_link"/>
+    </joint>
+    <link name="base_link">
         <visual>
             <geometry>
@@ -87,14 +88,8 @@
         </inertial>
     </link>
-    <link name="base_link"/>
-    <joint name="base_link_joint" type="fixed">
-        <origin xyz="0 0 0" rpy="0 0 0" />
-        <parent link="body" />
-        <child link="base_link" />
-    </joint>
     <link name="front_rail"/>
     <joint name="front_rail_joint" type="fixed">
         <origin xyz="0.223 0 0.0805" rpy="0 0 0" />
-        <parent link="body" />
+        <parent link="base_link" />
         <child link="front_rail" />
     </joint>
@@ -102,5 +97,5 @@
     <joint name="rear_rail_joint" type="fixed">
         <origin xyz="-0.223 0 0.0805" rpy="0 0 0" />
-        <parent link="body" />
+        <parent link="base_link" />
         <child link="rear_rail" />
     </joint>
@@ -128,5 +123,5 @@
         <origin xyz="0.29785 0.05500 0.00000" rpy="0 0 0" />
         <axis xyz="1 0 0" />
-        <parent link="body" />
+        <parent link="base_link" />
         <child link="lf_hip" />
         <limit effort="1000" velocity="1000.00" lower="-0.78539816339744827899" upper="0.78539816339744827899" />
@@ -171,10 +166,10 @@
         </collision>
         <inertial>
-            <origin rpy="0 0 0" xyz="${upperleg_com_x} ${upperleg_com_y*1} ${upperleg_com_z}"/>
-            <mass value="${upperleg_mass}"/>
-            <inertia
-                ixx="${upperleg_ixx}" ixy="${upperleg_ixy*1}" ixz="${upperleg_ixz}"
-                iyy="${upperleg_iyy}" iyz="${upperleg_iyz*1}"
-                izz="${upperleg_izz}"/>
+            <origin rpy="0 0 0" xyz="${lowerleg_com_x} ${lowerleg_com_y*1} ${lowerleg_com_z}"/>
+            <mass value="${lowerleg_mass}"/>
+            <inertia
+                ixx="${lowerleg_ixx}" ixy="${lowerleg_ixy*1}" ixz="${lowerleg_ixz}"
+                iyy="${lowerleg_iyy}" iyz="${lowerleg_iyz*1}"
+                izz="${lowerleg_izz}"/>
         </inertial>
     </link>
@@ -192,4 +187,24 @@
     </joint>
     <link name="lf_foot">
+    <visual>
+        <origin rpy="0 0 0" xyz="0 0 0"/>
+        <geometry>
+            <sphere radius="${foot_radius-0.01}"/>
+        </geometry>
+        <material name="green"/>
+    </visual>
+    <collision>
+        <origin rpy="0 0 0" xyz="0 0 0"/>
+        <geometry>
+            <sphere radius="${foot_radius}"/>
+        </geometry>
+    </collision>
+    <inertial>
+        <mass value="${foot_mass}"/>
+        <inertia
+            ixx="${(2*foot_mass)/5.0*(foot_radius*foot_radius)}" ixy="0.0" ixz="0.0"
+            iyy="${(2*foot_mass)/5.0*(foot_radius*foot_radius)}" iyz="0.0"
+            izz="${(2*foot_mass)/5.0*(foot_radius*foot_radius)}"/>
+    </inertial>
     </link>
     <link name="rf_hip">
@@ -216,5 +231,5 @@
         <origin xyz="0.29785 -0.05500 0.00000" rpy="0 0 0" />
         <axis xyz="1 0 0" />
-        <parent link="body" />
+        <parent link="base_link" />
         <child link="rf_hip" />
         <limit effort="1000" velocity="1000.00" lower="-0.78539816339744827899" upper="0.78539816339744827899" />
@@ -259,10 +274,10 @@
         </collision>
         <inertial>
-            <origin rpy="0 0 0" xyz="${upperleg_com_x} ${upperleg_com_y*-1} ${upperleg_com_z}"/>
-            <mass value="${upperleg_mass}"/>
-            <inertia
-                ixx="${upperleg_ixx}" ixy="${upperleg_ixy*-1}" ixz="${upperleg_ixz}"
-                iyy="${upperleg_iyy}" iyz="${upperleg_iyz*-1}"
-                izz="${upperleg_izz}"/>
+            <origin rpy="0 0 0" xyz="${lowerleg_com_x} ${lowerleg_com_y*-1} ${lowerleg_com_z}"/>
+            <mass value="${lowerleg_mass}"/>
+            <inertia
+                ixx="${lowerleg_ixx}" ixy="${lowerleg_ixy*-1}" ixz="${lowerleg_ixz}"
+                iyy="${lowerleg_iyy}" iyz="${lowerleg_iyz*-1}"
+                izz="${lowerleg_izz}"/>
         </inertial>
     </link>
@@ -280,4 +295,24 @@
     </joint>
     <link name="rf_foot">
+    <visual>
+        <origin rpy="0 0 0" xyz="0 0 0"/>
+        <geometry>
+            <sphere radius="${foot_radius-0.01}"/>
+        </geometry>
+        <material name="green"/>
+    </visual>
+    <collision>
+        <origin rpy="0 0 0" xyz="0 0 0"/>
+        <geometry>
+            <sphere radius="${foot_radius}"/>
+        </geometry>
+    </collision>
+    <inertial>
+        <mass value="${foot_mass}"/>
+        <inertia
+            ixx="${(2*foot_mass)/5.0*(foot_radius*foot_radius)}" ixy="0.0" ixz="0.0"
+            iyy="${(2*foot_mass)/5.0*(foot_radius*foot_radius)}" iyz="0.0"
+            izz="${(2*foot_mass)/5.0*(foot_radius*foot_radius)}"/>
+    </inertial>
     </link>
     <link name="lh_hip">
@@ -304,5 +339,5 @@
         <origin xyz="-0.29785 0.05500 0.00000" rpy="0 0 0" />
         <axis xyz="1 0 0" />
-        <parent link="body" />
+        <parent link="base_link" />
         <child link="lh_hip" />
         <limit effort="1000" velocity="1000.00" lower="-0.78539816339744827899" upper="0.78539816339744827899" />
@@ -347,10 +382,10 @@
         </collision>
         <inertial>
-            <origin rpy="0 0 0" xyz="${upperleg_com_x} ${upperleg_com_y*1} ${upperleg_com_z}"/>
-            <mass value="${upperleg_mass}"/>
-            <inertia
-                ixx="${upperleg_ixx}" ixy="${upperleg_ixy*1}" ixz="${upperleg_ixz}"
-                iyy="${upperleg_iyy}" iyz="${upperleg_iyz*1}"
-                izz="${upperleg_izz}"/>
+            <origin rpy="0 0 0" xyz="${lowerleg_com_x} ${lowerleg_com_y*1} ${lowerleg_com_z}"/>
+            <mass value="${lowerleg_mass}"/>
+            <inertia
+                ixx="${lowerleg_ixx}" ixy="${lowerleg_ixy*1}" ixz="${lowerleg_ixz}"
+                iyy="${lowerleg_iyy}" iyz="${lowerleg_iyz*1}"
+                izz="${lowerleg_izz}"/>
         </inertial>
     </link>
@@ -368,4 +403,24 @@
     </joint>
     <link name="lh_foot">
+    <visual>
+        <origin rpy="0 0 0" xyz="0 0 0"/>
+        <geometry>
+            <sphere radius="${foot_radius-0.01}"/>
+        </geometry>
+        <material name="green"/>
+    </visual>
+    <collision>
+        <origin rpy="0 0 0" xyz="0 0 0"/>
+        <geometry>
+            <sphere radius="${foot_radius}"/>
+        </geometry>
+    </collision>
+    <inertial>
+        <mass value="${foot_mass}"/>
+        <inertia
+            ixx="${(2*foot_mass)/5.0*(foot_radius*foot_radius)}" ixy="0.0" ixz="0.0"
+            iyy="${(2*foot_mass)/5.0*(foot_radius*foot_radius)}" iyz="0.0"
+            izz="${(2*foot_mass)/5.0*(foot_radius*foot_radius)}"/>
+    </inertial>
     </link>
     <link name="rh_hip">
@@ -392,5 +447,5 @@
         <origin xyz="-0.29785 -0.05500 0.00000" rpy="0 0 0" />
         <axis xyz="1 0 0" />
-        <parent link="body" />
+        <parent link="base_link" />
         <child link="rh_hip" />
         <limit effort="1000" velocity="1000.00" lower="-0.78539816339744827899" upper="0.78539816339744827899" />
@@ -435,10 +490,10 @@
         </collision>
         <inertial>
-            <origin rpy="0 0 0" xyz="${upperleg_com_x} ${upperleg_com_y*-1} ${upperleg_com_z}"/>
-            <mass value="${upperleg_mass}"/>
-            <inertia
-                ixx="${upperleg_ixx}" ixy="${upperleg_ixy*-1}" ixz="${upperleg_ixz}"
-                iyy="${upperleg_iyy}" iyz="${upperleg_iyz*-1}"
-                izz="${upperleg_izz}"/>
+            <origin rpy="0 0 0" xyz="${lowerleg_com_x} ${lowerleg_com_y*-1} ${lowerleg_com_z}"/>
+            <mass value="${lowerleg_mass}"/>
+            <inertia
+                ixx="${lowerleg_ixx}" ixy="${lowerleg_ixy*-1}" ixz="${lowerleg_ixz}"
+                iyy="${lowerleg_iyy}" iyz="${lowerleg_iyz*-1}"
+                izz="${lowerleg_izz}"/>
         </inertial>
     </link>
@@ -456,4 +511,24 @@
     </joint>
     <link name="rh_foot">
+    <visual>
+        <origin rpy="0 0 0" xyz="0 0 0"/>
+        <geometry>
+            <sphere radius="${foot_radius-0.01}"/>
+        </geometry>
+        <material name="green"/>
+    </visual>
+    <collision>
+        <origin rpy="0 0 0" xyz="0 0 0"/>
+        <geometry>
+            <sphere radius="${foot_radius}"/>
+        </geometry>
+    </collision>
+    <inertial>
+        <mass value="${foot_mass}"/>
+        <inertia
+            ixx="${(2*foot_mass)/5.0*(foot_radius*foot_radius)}" ixy="0.0" ixz="0.0"
+            iyy="${(2*foot_mass)/5.0*(foot_radius*foot_radius)}" iyz="0.0"
+            izz="${(2*foot_mass)/5.0*(foot_radius*foot_radius)}"/>
+    </inertial>
     </link>
     <!-- Standard accessories. -->

File: descriptions/spot_description/urdfs/leg.gazebo.xacro (robot description, xacro)
@@ -81,5 +81,5 @@
 				<update_rate>250.0</update_rate>
 				<contact>
-					<collision>${name}_lowerleg_fixed_joint_lump__${name}_foot_collision_1</collision>
+                                        <collision>${name}_lowerleg_fixed_joint_lump__${name}_foot_collision_1</collision>
 				</contact>
                                 <!-- the sensor readings in terms of force torques are expressed in the lowerleg frame
