Commit message: Update solo description to make it compliant with the new wb version

File: descriptions/solo_description/gazebo/gazebo.urdf.xacro (robot description, xacro)
@@ -5,5 +5,5 @@
 		<plugin name="gazebo_ros_controller_manager" filename="libgazebo_ros_control.so">
 			<robotNamespace>/solo</robotNamespace>
-			<robotSimType>dls_gazebo_interface/DlsRobotHwSim</robotSimType>
+			<robotSimType>wb_gazebo_interface/WbRobotHwSim</robotSimType>
             		<controlPeriod>$(arg task_period)</controlPeriod>
 		</plugin>

File: descriptions/solo_description/robots/solo.srdf.xacro (robot description, xacro)
@@ -1,24 +1,44 @@
+<?xml version="1.0" ?>
 <robot name="solo" xmlns:xacro="http://ros.org/wiki/xacro">
-  <group name="base">
-    <link name="base_link"/>
-  </group>
-  <group name="lf">
-    <chain base_link="trunk" tip_link="lf_foot"/>
-  </group>
-  <group name="rf">
-    <chain base_link="trunk" tip_link="rf_foot"/>
-  </group>
-  <group name="lh">
-    <chain base_link="trunk" tip_link="lh_foot"/>
-  </group>
-  <group name="rh">
-    <chain base_link="trunk" tip_link="rh_foot"/>
-  </group>
-  <group name="chains">
-    <group name="lf"/>
-    <group name="rf"/>
-    <group name="lh"/>
-    <group name="rh"/>
-  </group>
+<xacro:arg name="arm" default="false"/>
+    <group name="base">
+      <link name="base_link"/>
+    </group>
+    <group name="lf_leg">
+      <chain base_link="base_link" tip_link="lf_foot"/>
+    </group>
+    <group name="rf_leg">
+      <chain base_link="base_link" tip_link="rf_foot"/>
+    </group>
+    <group name="lh_leg">
+      <chain base_link="base_link" tip_link="lh_foot"/>
+    </group>
+    <group name="rh_leg">
+      <chain base_link="base_link" tip_link="rh_foot"/>
+    </group>
+    <group name="lf_hip">
+      <chain base_link="base_link" tip_link="lf_hip_assembly"/>
+    </group>
+    <group name="rf_hip">
+      <chain base_link="base_link" tip_link="rf_hip_assembly"/>
+    </group>
+    <group name="lh_hip">
+      <chain base_link="base_link" tip_link="lh_hip_assembly"/>
+    </group>
+    <group name="rh_hip">
+      <chain base_link="base_link" tip_link="rh_hip_assembly"/>
+    </group>
+    <group name="legs">
+      <group name="lf_leg"/>
+      <group name="rf_leg"/>
+      <group name="lh_leg"/>
+      <group name="rh_leg"/>
+    </group>
+    <group name="chains">
+      <group name="lf_leg"/>
+      <group name="rf_leg"/>
+      <group name="lh_leg"/>
+      <group name="rh_leg"/>
+    </group>
   <group_state group="chains" name="home">
     <joint name="lf_haa_joint" value="0.0"/>
