Commit message: Move kinova in front of hyq

File: descriptions/hyq_description/urdfs/arm/kinova_adapter.urdf.xacro (robot description, xacro)
@@ -5,7 +5,7 @@
        <parent link="base_link"/>
        <child link="kinova_adapter_link"/>
-       <origin xyz="0.0 0.0 0.0" rpy="0 0 0"/>
+       <origin xyz="0.5 0.0 0.0" rpy="0 1.57 0"/>
 </joint>
-<xacro:include filename="$(find kinova_description)/urdf/j2n4s300.xacro"/>
-<xacro:j2n4s300  base_parent="kinova_adapter_link" prefix="kinova"/>
+<xacro:include filename="$(find kinova_description)/urdf/m1n4s200.xacro"/>
+<xacro:m1n4s200  base_parent="kinova_adapter_link" prefix="kinova"/>
 </robot>
