Commit message: Make fingers fixed in kinova

File: descriptions/kinova_description/urdf/kinova_common.xacro (robot description, xacro)
@@ -91,5 +91,5 @@
     <xacro:macro name="kinova_finger" params="prefix finger_number hand finger_origin_xyz finger_origin_rpy">
         <xacro:kinova_armlink link_name="${prefix}link_finger_${finger_number}" link_mesh="finger_proximal" mesh_no="57"/>
-        <joint name="${prefix}joint_finger_${finger_number}" type="revolute">
+        <joint name="${prefix}joint_finger_${finger_number}" type="fixed">
             <parent link="${hand}"/>
             <child link="${prefix}link_finger_${finger_number}"/>
@@ -98,5 +98,5 @@
             <limit lower="0" upper="1.51" effort="2" velocity="1"/>
         </joint>
-		    <transmission name="${prefix}joint_finger_${finger_number}_trans">
+        <!--	    <transmission name="${prefix}joint_finger_${finger_number}_trans">
 					<type>transmission_interface/SimpleTransmission</type>
 					<joint name="${prefix}joint_finger_${finger_number}">
@@ -107,7 +107,7 @@
 					<mechanicalReduction>1</mechanicalReduction>
 					</actuator>
-		    </transmission>
+                    </transmission> -->
         <xacro:kinova_armlink link_name="${prefix}link_finger_tip_${finger_number}" link_mesh="finger_distal" mesh_no="58"/>
-        <joint name="${prefix}joint_finger_tip_${finger_number}" type="revolute">
+        <joint name="${prefix}joint_finger_tip_${finger_number}" type="fixed">
             <parent link="${prefix}link_finger_${finger_number}"/>
             <child link="${prefix}link_finger_tip_${finger_number}"/>
@@ -116,5 +116,5 @@
             <limit lower="0" upper="2" effort="2" velocity="1"/>
         </joint>
-        <transmission name="${prefix}joint_finger_tip_${finger_number}_trans">
+        <!-- <transmission name="${prefix}joint_finger_tip_${finger_number}_trans">
 					<type>transmission_interface/SimpleTransmission</type>
 					<joint name="${prefix}joint_finger_tip_${finger_number}">
@@ -125,5 +125,5 @@
 					<mechanicalReduction>1</mechanicalReduction>
 					</actuator>
-        </transmission>
+        </transmission> -->
     </xacro:macro>
 </root>

Commit message: Add a little friction in the kinova joints

File: descriptions/kinova_description/urdf/kinova_common.xacro (robot description, xacro)
@@ -51,5 +51,5 @@
         <limit effort="${joint_torque_limit}" velocity="${joint_velocity_limit}" lower="${joint_lower_limit}" upper="${joint_upper_limit}"/>
         <origin xyz="${joint_origin_xyz}" rpy="${joint_origin_rpy}"/>
-        <dynamics damping="0.0" friction="0.0"/>
+        <dynamics damping="0.0" friction="0.03"/>
      </joint>
    <xacro:unless value="${fixed}">
