Commit message: Make aliengo compliant with kinova, to debug

File: descriptions/aliengo_description/robots/aliengo_kinova.srdf.xacro (robot description, xacro)
@@ -19,4 +19,16 @@
   <group name="rh_leg">
     <chain base_link="trunk" tip_link="rh_foot"/>
+  </group>
+  <group name="lf_hip">
+    <chain base_link="trunk" tip_link="lf_hip"/>
+  </group>
+  <group name="rf_hip">
+    <chain base_link="trunk" tip_link="rf_hip"/>
+  </group>
+  <group name="lh_hip">
+    <chain base_link="trunk" tip_link="lh_hip"/>
+  </group>
+  <group name="rh_hip">
+    <chain base_link="trunk" tip_link="rh_hip"/>
   </group>
   <group name="legs">
@@ -50,7 +62,7 @@
     <joint name="rh_kfe_joint" value="-1.3"/>
     <joint name="kinova_joint_1" value="0.0"/>
-    <joint name="kinova_joint_2" value="0.0"/>
-    <joint name="kinova_joint_3" value="0.0"/>
-    <joint name="kinova_joint_4" value="0.0"/>
+    <joint name="kinova_joint_2" value="1.80"/>
+    <joint name="kinova_joint_3" value="4.0"/>
+    <joint name="kinova_joint_4" value="-1.5"/>
   </group_state>
 </robot>

Commit message: Update aliengo with kinova

File: descriptions/aliengo_description/robots/aliengo_kinova.srdf.xacro (robot description, xacro)
@@ -78,7 +78,7 @@
     <joint name="rh_kfe_joint" value="-1.3"/>
     <joint name="kinova_joint_1" value="0.0"/>
-    <joint name="kinova_joint_2" value="1.80"/>
-    <joint name="kinova_joint_3" value="4.0"/>
-    <joint name="kinova_joint_4" value="-1.5"/>
+    <joint name="kinova_joint_2" value="4.0"/>
+    <joint name="kinova_joint_3" value="5.6"/>
+    <joint name="kinova_joint_4" value="3.14"/>
   </group_state>
 </robot>

File: descriptions/aliengo_description/urdfs/arm/kinova_adapter.urdf.xacro (robot description, xacro)
@@ -5,7 +5,7 @@
        <parent link="base_link"/>
        <child link="kinova_adapter_link"/>
-       <origin xyz="0.0 0.0 0.0" rpy="0 0 0"/>
+       <origin xyz="0.35 0.0 -0.08" rpy="0 0 0"/>
 </joint>
-<xacro:include filename="$(find kinova_description)/urdf/j2n4s300.xacro"/>
-<xacro:j2n4s300  base_parent="kinova_adapter_link" prefix="kinova"/>
+<xacro:include filename="$(find kinova_description)/urdf/m1n4s200.xacro"/>
+<xacro:m1n4s200  base_parent="kinova_adapter_link" prefix="kinova"/>
 </robot>
