Commit message: Ugly as fuck

File: descriptions/aliengo_description/robots/aliengo.srdf.xacro (robot description, xacro)
@@ -1,38 +1,88 @@
 <?xml version="1.0" ?>
 <robot name="aliengo" xmlns:xacro="http://ros.org/wiki/xacro">
-  <group name="base">
-    <link name="base_link"/>
-  </group>
-  <group name="lf">
-    <chain base_link="trunk" tip_link="lf_foot"/>
-  </group>
-  <group name="rf">
-    <chain base_link="trunk" tip_link="rf_foot"/>
-  </group>
-  <group name="lh">
-    <chain base_link="trunk" tip_link="lh_foot"/>
-  </group>
-  <group name="rh">
-    <chain base_link="trunk" tip_link="rh_foot"/>
-  </group>
-  <group name="chains">
-    <group name="lf"/>
-    <group name="rf"/>
-    <group name="lh"/>
-    <group name="rh"/>
-  </group>
-  <group_state group="chains" name="home">
-      <joint name="lf_haa_joint" value="0.0"/>
-      <joint name="lf_hfe_joint" value="0.67"/>
-      <joint name="lf_kfe_joint" value="-1.3"/>
-      <joint name="rf_haa_joint" value="0.0"/>
-      <joint name="rf_hfe_joint" value="0.67"/>
-      <joint name="rf_kfe_joint" value="-1.3"/>
-      <joint name="lh_haa_joint" value="0.0"/>
-      <joint name="lh_hfe_joint" value="0.67"/>
-      <joint name="lh_kfe_joint" value="-1.3"/>
-      <joint name="rh_haa_joint" value="0.0"/>
-      <joint name="rh_hfe_joint" value="0.67"/>
-      <joint name="rh_kfe_joint" value="-1.3"/>
-  </group_state>
+<xacro:arg name="arm" default="false"/>
+<xacro:if value="$(arg arm)">
+    <group name="base">
+      <link name="base_link"/>
+    </group>
+    <group name="arm">
+         <chain base_link="base_arm" tip_link="TCP"/>
+    </group>
+    <group name="lf">
+      <chain base_link="trunk" tip_link="lf_foot"/>
+    </group>
+    <group name="rf">
+      <chain base_link="trunk" tip_link="rf_foot"/>
+    </group>
+    <group name="lh">
+      <chain base_link="trunk" tip_link="lh_foot"/>
+    </group>
+    <group name="rh">
+      <chain base_link="trunk" tip_link="rh_foot"/>
+    </group>
+    <group name="chains">
+      <group name="lf"/>
+      <group name="rf"/>
+      <group name="lh"/>
+      <group name="rh"/>
+      <group name="arm"/>
+    </group>
+    <group_state group="chains" name="home">
+        <joint name="lf_haa_joint" value="0.0"/>
+        <joint name="lf_hfe_joint" value="0.67"/>
+        <joint name="lf_kfe_joint" value="-1.3"/>
+        <joint name="rf_haa_joint" value="0.0"/>
+        <joint name="rf_hfe_joint" value="0.67"/>
+        <joint name="rf_kfe_joint" value="-1.3"/>
+        <joint name="lh_haa_joint" value="0.0"/>
+        <joint name="lh_hfe_joint" value="0.67"/>
+        <joint name="lh_kfe_joint" value="-1.3"/>
+        <joint name="rh_haa_joint" value="0.0"/>
+        <joint name="rh_hfe_joint" value="0.67"/>
+        <joint name="rh_kfe_joint" value="-1.3"/>
+        <joint name="z_joint_1" value="0.0"/>
+        <joint name="z_joint_2" value="0.0"/>
+        <joint name="z_joint_3" value="0.0"/>
+        <joint name="z_joint_4" value="0.0"/>
+        <joint name="z_joint_5" value="0.0"/>
+        <joint name="z_joint_6" value="0.0"/>
+    </group_state>
+</xacro:if>
+<xacro:unless value="$(arg arm)">
+    <group name="base">
+      <link name="base_link"/>
+    </group>
+    <group name="lf">
+      <chain base_link="trunk" tip_link="lf_foot"/>
+    </group>
+    <group name="rf">
+      <chain base_link="trunk" tip_link="rf_foot"/>
+    </group>
+    <group name="lh">
+      <chain base_link="trunk" tip_link="lh_foot"/>
+    </group>
+    <group name="rh">
+      <chain base_link="trunk" tip_link="rh_foot"/>
+    </group>
+    <group name="chains">
+      <group name="lf"/>
+      <group name="rf"/>
+      <group name="lh"/>
+      <group name="rh"/>
+    </group>
+    <group_state group="chains" name="home">
+        <joint name="lf_haa_joint" value="0.0"/>
+        <joint name="lf_hfe_joint" value="0.67"/>
+        <joint name="lf_kfe_joint" value="-1.3"/>
+        <joint name="rf_haa_joint" value="0.0"/>
+        <joint name="rf_hfe_joint" value="0.67"/>
+        <joint name="rf_kfe_joint" value="-1.3"/>
+        <joint name="lh_haa_joint" value="0.0"/>
+        <joint name="lh_hfe_joint" value="0.67"/>
+        <joint name="lh_kfe_joint" value="-1.3"/>
+        <joint name="rh_haa_joint" value="0.0"/>
+        <joint name="rh_hfe_joint" value="0.67"/>
+        <joint name="rh_kfe_joint" value="-1.3"/>
+    </group_state>
+</xacro:unless>
 </robot>

File: descriptions/aliengo_description/robots/aliengo.urdf.xacro (robot description, xacro)
@@ -4,4 +4,5 @@
     <xacro:arg name="load_force_sensors" default="false"/>
     <xacro:arg name="task_period" default="0.004"/>
+    <xacro:arg name="arm" default="false"/>
     <xacro:include filename="$(find aliengo_description)/urdfs/const.xacro"/>
     <xacro:include filename="$(find aliengo_description)/urdfs/materials.xacro"/>
@@ -150,3 +151,18 @@
     <xacro:leg_transmission name="lh"/>
     <xacro:leg_gazebo name="lh" load_force_sensors="$(arg load_force_sensors)"/>
+    <xacro:if value="$(arg arm)">
+        <joint name="joint_base_robots" type="fixed">
+                <parent link="base_link"/>
+                <child link="base_arm"/>
+                <origin xyz="0 0 0" rpy="0 0 0"/>
+                </joint>
+            <xacro:include filename="$(find kinova_description)/urdf/arm.urdf.xacro" />
+            <xacro:include filename="$(find kinova_description)/urdf/arm.transmission.xacro"/>
+            <xacro:arm_transmission name="z_joint_1"/>
+            <xacro:arm_transmission name="z_joint_2"/>
+            <xacro:arm_transmission name="z_joint_3"/>
+            <xacro:arm_transmission name="z_joint_4"/>
+            <xacro:arm_transmission name="z_joint_5"/>
+            <xacro:arm_transmission name="z_joint_6"/>
+    </xacro:if>
 </robot>

Commit message: Add kinova descriptions and robot adapters

File: descriptions/aliengo_description/robots/aliengo.srdf.xacro (robot description, xacro)
@@ -2,52 +2,4 @@
 <robot name="aliengo" xmlns:xacro="http://ros.org/wiki/xacro">
 <xacro:arg name="arm" default="false"/>
-<xacro:if value="$(arg arm)">
-    <group name="base">
-      <link name="base_link"/>
-    </group>
-    <group name="arm">
-         <chain base_link="base_arm" tip_link="TCP"/>
-    </group>
-    <group name="lf">
-      <chain base_link="trunk" tip_link="lf_foot"/>
-    </group>
-    <group name="rf">
-      <chain base_link="trunk" tip_link="rf_foot"/>
-    </group>
-    <group name="lh">
-      <chain base_link="trunk" tip_link="lh_foot"/>
-    </group>
-    <group name="rh">
-      <chain base_link="trunk" tip_link="rh_foot"/>
-    </group>
-    <group name="chains">
-      <group name="lf"/>
-      <group name="rf"/>
-      <group name="lh"/>
-      <group name="rh"/>
-      <group name="arm"/>
-    </group>
-    <group_state group="chains" name="home">
-        <joint name="lf_haa_joint" value="0.0"/>
-        <joint name="lf_hfe_joint" value="0.67"/>
-        <joint name="lf_kfe_joint" value="-1.3"/>
-        <joint name="rf_haa_joint" value="0.0"/>
-        <joint name="rf_hfe_joint" value="0.67"/>
-        <joint name="rf_kfe_joint" value="-1.3"/>
-        <joint name="lh_haa_joint" value="0.0"/>
-        <joint name="lh_hfe_joint" value="0.67"/>
-        <joint name="lh_kfe_joint" value="-1.3"/>
-        <joint name="rh_haa_joint" value="0.0"/>
-        <joint name="rh_hfe_joint" value="0.67"/>
-        <joint name="rh_kfe_joint" value="-1.3"/>
-        <joint name="z_joint_1" value="0.0"/>
-        <joint name="z_joint_2" value="0.0"/>
-        <joint name="z_joint_3" value="0.0"/>
-        <joint name="z_joint_4" value="0.0"/>
-        <joint name="z_joint_5" value="0.0"/>
-        <joint name="z_joint_6" value="0.0"/>
-    </group_state>
-</xacro:if>
-<xacro:unless value="$(arg arm)">
     <group name="base">
       <link name="base_link"/>
@@ -85,4 +37,3 @@
         <joint name="rh_kfe_joint" value="-1.3"/>
     </group_state>
-</xacro:unless>
 </robot>

File: descriptions/aliengo_description/robots/aliengo.urdf.xacro (robot description, xacro)
@@ -4,5 +4,6 @@
     <xacro:arg name="load_force_sensors" default="false"/>
     <xacro:arg name="task_period" default="0.004"/>
-    <xacro:arg name="arm" default="false"/>
+    <xacro:arg name="arm_enabled" default="false"/>
+    <xacro:arg name="arm_name" default="kinova"/>
     <xacro:include filename="$(find aliengo_description)/urdfs/const.xacro"/>
     <xacro:include filename="$(find aliengo_description)/urdfs/materials.xacro"/>
@@ -151,18 +152,6 @@
     <xacro:leg_transmission name="lh"/>
     <xacro:leg_gazebo name="lh" load_force_sensors="$(arg load_force_sensors)"/>
-    <xacro:if value="$(arg arm)">
-        <joint name="joint_base_robots" type="fixed">
-                <parent link="base_link"/>
-                <child link="base_arm"/>
-                <origin xyz="0 0 0" rpy="0 0 0"/>
-                </joint>
-            <xacro:include filename="$(find kinova_description)/urdf/arm.urdf.xacro" />
-            <xacro:include filename="$(find kinova_description)/urdf/arm.transmission.xacro"/>
-            <xacro:arm_transmission name="z_joint_1"/>
-            <xacro:arm_transmission name="z_joint_2"/>
-            <xacro:arm_transmission name="z_joint_3"/>
-            <xacro:arm_transmission name="z_joint_4"/>
-            <xacro:arm_transmission name="z_joint_5"/>
-            <xacro:arm_transmission name="z_joint_6"/>
+    <xacro:if value="$(arg arm_enabled)">
+           <xacro:include filename="$(find aliengo_description)/urdfs/arm/$(arg arm_name)_adapter.urdf.xacro" /> -->
     </xacro:if>
 </robot>

File: descriptions/anymal_description/robots/anymal.urdf.xacro (robot description, xacro)
@@ -730,20 +730,3 @@
     <xacro:leg_transmission name="lh"/>
     <xacro:leg_gazebo name="lh" load_force_sensors="$(arg load_force_sensors)"/>
-    <xacro:if value="$(arg sensors)">
-        <!-- IMU trunk -->
-        <xacro:microstrain_3dmgx425_imu
-                parent="base"
-                imu_name="trunk_imu"
-                imu_topic="trunk_imu_1/data"
-                update_rate="250">
-                <origin xyz="0.27025 0.000 0.0967678" rpy="0 0 0"/>
-        </xacro:microstrain_3dmgx425_imu>
-        <xacro:kvh_1775_imu
-                parent="base"
-                imu_name="kvh_imu"
-                imu_topic="kvh_imu/data"
-                update_rate="250">
-                <origin xyz="0.316115 0.00 0.0887678" rpy="0 ${PI} ${PI/4}"/>
-        </xacro:kvh_1775_imu>
-    </xacro:if>
 </robot>

File: descriptions/hyq_description/robots/hyq.srdf.xacro (robot description, xacro)
@@ -1,53 +1,4 @@
 <?xml version="1.0" ?>
 <robot name="hyq" xmlns:xacro="http://ros.org/wiki/xacro">
-<xacro:arg name="arm" default="false"/>
-<xacro:if value="$(arg arm)">
-  <group name="base">
-    <link name="base_link"/>
-    <link name="teleop_link0"/>
-  </group>
-  <group name="arm">
-       <chain base_link="teleop_link0" tip_link="TCP"/>
-  </group>
-  <group name="lf">
-    <chain base_link="trunk" tip_link="lf_foot"/>
-  </group>
-  <group name="rf">
-    <chain base_link="trunk" tip_link="rf_foot"/>
-  </group>
-  <group name="lh">
-    <chain base_link="trunk" tip_link="lh_foot"/>
-  </group>
-  <group name="rh">
-    <chain base_link="trunk" tip_link="rh_foot"/>
-  </group>
-  <group name="chains">
-    <group name="lf"/>
-    <group name="rf"/>
-    <group name="lh"/>
-    <group name="rh"/>
-    <group name="arm"/>
-  </group>
-  <group_state group="chains" name="home">
-    <joint name="lf_haa_joint" value="-0.2"/>
-    <joint name="lf_hfe_joint" value="0.75"/>
-    <joint name="lf_kfe_joint" value="-1.5"/>
-    <joint name="rf_haa_joint" value="-0.2"/>
-    <joint name="rf_hfe_joint" value="0.75"/>
-    <joint name="rf_kfe_joint" value="-1.5"/>
-    <joint name="lh_haa_joint" value="-0.2"/>
-    <joint name="lh_hfe_joint" value="-0.75"/>
-    <joint name="lh_kfe_joint" value="1.5"/>
-    <joint name="rh_haa_joint" value="-0.2"/>
-    <joint name="rh_hfe_joint" value="-0.75"/>
-    <joint name="rh_kfe_joint" value="1.5"/>
-    <joint name="joint1" value="0.0"/>
-    <joint name="joint2" value="1.0"/>
-    <joint name="joint3" value="1.0"/>
-    <joint name="joint4" value="0.0"/>
-    <joint name="joint5" value="0.0"/>
-  </group_state>
-</xacro:if>
-<xacro:unless value="$(arg arm)">
   <group name="base">
     <link name="base_link"/>
@@ -85,4 +36,3 @@
     <joint name="rh_kfe_joint" value="1.5"/>
   </group_state>
-</xacro:unless>
 </robot>

Commit message: Change the haa starting position for aliengo

File: descriptions/aliengo_description/robots/aliengo.srdf.xacro (robot description, xacro)
@@ -42,14 +42,14 @@
     </group>
     <group_state group="chains" name="home">
-        <joint name="lf_haa_joint" value="0.0"/>
+        <joint name="lf_haa_joint" value="0.1"/>
         <joint name="lf_hfe_joint" value="0.67"/>
         <joint name="lf_kfe_joint" value="-1.3"/>
-        <joint name="rf_haa_joint" value="0.0"/>
+        <joint name="rf_haa_joint" value="-0.1"/>
         <joint name="rf_hfe_joint" value="0.67"/>
         <joint name="rf_kfe_joint" value="-1.3"/>
-        <joint name="lh_haa_joint" value="0.0"/>
+        <joint name="lh_haa_joint" value="0.1"/>
         <joint name="lh_hfe_joint" value="0.67"/>
         <joint name="lh_kfe_joint" value="-1.3"/>
-        <joint name="rh_haa_joint" value="0.0"/>
+        <joint name="rh_haa_joint" value="-0.1"/>
         <joint name="rh_hfe_joint" value="0.67"/>
         <joint name="rh_kfe_joint" value="-1.3"/>

Commit message: Update the srdfs

File: descriptions/aliengo_description/robots/aliengo.srdf.xacro (robot description, xacro)
@@ -2,18 +2,30 @@
 <robot name="aliengo" xmlns:xacro="http://ros.org/wiki/xacro">
 <xacro:arg name="arm" default="false"/>
-    <group name="base">
+    <group name="bases">
       <link name="base_link"/>
     </group>
     <group name="lf_leg">
-      <chain base_link="trunk" tip_link="lf_foot"/>
+      <chain base_link="base_link" tip_link="lf_foot"/>
+      <joint name="lf_haa_joint"/>
+      <joint name="lf_hfe_joint"/>
+      <joint name="lf_kfe_joint"/>
     </group>
     <group name="rf_leg">
-      <chain base_link="trunk" tip_link="rf_foot"/>
+      <chain base_link="base_link" tip_link="rf_foot"/>
+      <joint name="rf_haa_joint"/>
+      <joint name="rf_hfe_joint"/>
+      <joint name="rf_kfe_joint"/>
     </group>
     <group name="lh_leg">
-      <chain base_link="trunk" tip_link="lh_foot"/>
+      <chain base_link="base_link" tip_link="lh_foot"/>
+      <joint name="lh_haa_joint"/>
+      <joint name="lh_hfe_joint"/>
+      <joint name="lh_kfe_joint"/>
     </group>
     <group name="rh_leg">
-      <chain base_link="trunk" tip_link="rh_foot"/>
+      <chain base_link="base_link" tip_link="rh_foot"/>
+      <joint name="rh_haa_joint"/>
+      <joint name="rh_hfe_joint"/>
+      <joint name="rh_kfe_joint"/>
     </group>
     <group name="lf_hip">

File: descriptions/aliengo_description/robots/aliengo_kinova.srdf.xacro (robot description, xacro)
@@ -1,22 +1,38 @@
 <?xml version="1.0" ?>
 <robot name="aliengo" xmlns:xacro="http://ros.org/wiki/xacro">
-  <group name="base">
+  <group name="bases">
     <link name="base_link"/>
     <link name="kinova_link_base"/>
   </group>
   <group name="kinova_arm">
-       <chain base_link="kinova_link_base" tip_link="kinova_end_effector"/>
+    <chain base_link="kinova_link_base" tip_link="kinova_end_effector"/>
+    <joint name="kinova_joint_1"/>
+    <joint name="kinova_joint_2"/>
+    <joint name="kinova_joint_3"/>
+    <joint name="kinova_joint_4"/>
   </group>
   <group name="lf_leg">
-    <chain base_link="trunk" tip_link="lf_foot"/>
+    <chain base_link="base_link" tip_link="lf_foot"/>
+    <joint name="lf_haa_joint"/>
+    <joint name="lf_hfe_joint"/>
+    <joint name="lf_kfe_joint"/>
   </group>
   <group name="rf_leg">
-    <chain base_link="trunk" tip_link="rf_foot"/>
+    <chain base_link="base_link" tip_link="rf_foot"/>
+    <joint name="rf_haa_joint"/>
+    <joint name="rf_hfe_joint"/>
+    <joint name="rf_kfe_joint"/>
   </group>
   <group name="lh_leg">
-    <chain base_link="trunk" tip_link="lh_foot"/>
+    <chain base_link="base_link" tip_link="lh_foot"/>
+    <joint name="lh_haa_joint"/>
+    <joint name="lh_hfe_joint"/>
+    <joint name="lh_kfe_joint"/>
   </group>
   <group name="rh_leg">
-    <chain base_link="trunk" tip_link="rh_foot"/>
+    <chain base_link="base_link" tip_link="rh_foot"/>
+    <joint name="rh_haa_joint"/>
+    <joint name="rh_hfe_joint"/>
+    <joint name="rh_kfe_joint"/>
   </group>
   <group name="lf_hip">

File: descriptions/aliengo_description/robots/aliengo_teleop.srdf.xacro (robot description, xacro)
@@ -2,5 +2,5 @@
 <robot name="aliengo" xmlns:xacro="http://ros.org/wiki/xacro">
 <xacro:arg name="arm" default="false"/>
-    <group name="base">
+    <group name="bases">
       <link name="base_link"/>
     </group>
@@ -8,15 +8,27 @@
          <chain base_link="base_arm" tip_link="TCP"/>
     </group>
-    <group name="lf">
-      <chain base_link="trunk" tip_link="lf_foot"/>
+    <group name="lf_leg">
+      <chain base_link="base_link" tip_link="lf_foot"/>
+      <joint name="lf_haa_joint"/>
+      <joint name="lf_hfe_joint"/>
+      <joint name="lf_kfe_joint"/>
     </group>
-    <group name="rf">
-      <chain base_link="trunk" tip_link="rf_foot"/>
+    <group name="rf_leg">
+      <chain base_link="base_link" tip_link="rf_foot"/>
+      <joint name="rf_haa_joint"/>
+      <joint name="rf_hfe_joint"/>
+      <joint name="rf_kfe_joint"/>
     </group>
-    <group name="lh">
-      <chain base_link="trunk" tip_link="lh_foot"/>
+    <group name="lh_leg">
+      <chain base_link="base_link" tip_link="lh_foot"/>
+      <joint name="lh_haa_joint"/>
+      <joint name="lh_hfe_joint"/>
+      <joint name="lh_kfe_joint"/>
     </group>
-    <group name="rh">
-      <chain base_link="trunk" tip_link="rh_foot"/>
+    <group name="rh_leg">
+      <chain base_link="base_link" tip_link="rh_foot"/>
+      <joint name="rh_haa_joint"/>
+      <joint name="rh_hfe_joint"/>
+      <joint name="rh_kfe_joint"/>
     </group>
     <group name="chains">

File: descriptions/anymal_description/robots/anymal.srdf.xacro (robot description, xacro)
@@ -1,18 +1,30 @@
 <?xml version="1.0" ?>
 <robot name="anymal" xmlns:xacro="http://ros.org/wiki/xacro">
-  <group name="base">
+  <group name="bases">
     <link name="base_link"/>
   </group>
   <group name="lf_leg">
-    <chain base_link="trunk" tip_link="lf_foot"/>
+    <chain base_link="base_link" tip_link="lf_foot"/>
+    <joint name="lf_haa_joint"/>
+    <joint name="lf_hfe_joint"/>
+    <joint name="lf_kfe_joint"/>
   </group>
   <group name="rf_leg">
-    <chain base_link="trunk" tip_link="rf_foot"/>
+    <chain base_link="base_link" tip_link="rf_foot"/>
+    <joint name="rf_haa_joint"/>
+    <joint name="rf_hfe_joint"/>
+    <joint name="rf_kfe_joint"/>
   </group>
   <group name="lh_leg">
-    <chain base_link="trunk" tip_link="lh_foot"/>
+    <chain base_link="base_link" tip_link="lh_foot"/>
+    <joint name="lh_haa_joint"/>
+    <joint name="lh_hfe_joint"/>
+    <joint name="lh_kfe_joint"/>
   </group>
   <group name="rh_leg">
-    <chain base_link="trunk" tip_link="rh_foot"/>
+    <chain base_link="base_link" tip_link="rh_foot"/>
+    <joint name="rh_haa_joint"/>
+    <joint name="rh_hfe_joint"/>
+    <joint name="rh_kfe_joint"/>
   </group>
   <group name="lf_hip">

File: descriptions/spot_description/robots/spot.srdf.xacro (robot description, xacro)
@@ -7,13 +7,25 @@
     <group name="lf_leg">
       <chain base_link="base_link" tip_link="lf_foot"/>
+      <joint name="lf_haa_joint"/>
+      <joint name="lf_hfe_joint"/>
+      <joint name="lf_kfe_joint"/>
     </group>
     <group name="rf_leg">
       <chain base_link="base_link" tip_link="rf_foot"/>
+      <joint name="rf_haa_joint"/>
+      <joint name="rf_hfe_joint"/>
+      <joint name="rf_kfe_joint"/>
     </group>
     <group name="lh_leg">
       <chain base_link="base_link" tip_link="lh_foot"/>
+      <joint name="lh_haa_joint"/>
+      <joint name="lh_hfe_joint"/>
+      <joint name="lh_kfe_joint"/>
     </group>
     <group name="rh_leg">
       <chain base_link="base_link" tip_link="rh_foot"/>
+      <joint name="rh_haa_joint"/>
+      <joint name="rh_hfe_joint"/>
+      <joint name="rh_kfe_joint"/>
     </group>
     <group name="lf_hip">
