Commit message: Remove bases

File: descriptions/aliengo_description/robots/aliengo.srdf.xacro (robot description, xacro)
@@ -1,8 +1,4 @@
 <?xml version="1.0" ?>
 <robot name="aliengo" xmlns:xacro="http://ros.org/wiki/xacro">
-<xacro:arg name="arm" default="false"/>
-    <group name="bases">
-      <link name="base_link"/>
-    </group>
     <group name="lf_leg">
       <chain base_link="base_link" tip_link="lf_foot"/>

File: descriptions/aliengo_description/robots/aliengo_kinova.srdf.xacro (robot description, xacro)
@@ -1,8 +1,4 @@
 <?xml version="1.0" ?>
 <robot name="aliengo" xmlns:xacro="http://ros.org/wiki/xacro">
-  <group name="bases">
-    <link name="base_link"/>
-    <link name="kinova_link_base"/>
-  </group>
   <group name="kinova_arm">
     <chain base_link="kinova_link_base" tip_link="kinova_end_effector"/>

File: descriptions/anymal_description/robots/anymal.srdf.xacro (robot description, xacro)
@@ -1,7 +1,4 @@
 <?xml version="1.0" ?>
 <robot name="anymal" xmlns:xacro="http://ros.org/wiki/xacro">
-  <group name="bases">
-    <link name="base_link"/>
-  </group>
   <group name="lf_leg">
     <chain base_link="base_link" tip_link="lf_foot"/>

File: descriptions/hyq_description/robots/hyq.srdf.xacro (robot description, xacro)
@@ -1,7 +1,4 @@
 <?xml version="1.0" ?>
 <robot name="hyq" xmlns:xacro="http://ros.org/wiki/xacro">
-  <group name="base">
-    <link name="base_link"/>
-  </group>
   <group name="lf_leg">
     <chain base_link="trunk" tip_link="lf_foot"/>

File: descriptions/hyq_description/robots/hyq_kinova.srdf.xacro (robot description, xacro)
@@ -1,8 +1,4 @@
 <?xml version="1.0" ?>
 <robot name="hyq" xmlns:xacro="http://ros.org/wiki/xacro">
- <group name="bases">
-   <link name="base_link"/>
-   <link name="kinova_link_base"/>
- </group>
   <group name="kinova_arm">
     <chain base_link="kinova_link_base" tip_link="kinova_end_effector"/>

File: descriptions/hyq_description/robots/hyq_teleop.srdf.xacro (robot description, xacro)
@@ -1,8 +1,4 @@
 <?xml version="1.0" ?>
 <robot name="hyq" xmlns:xacro="http://ros.org/wiki/xacro">
-  <group name="bases">
-    <link name="base_link"/>
-    <link name="teleop_link0"/>
-  </group>
   <group name="teleop_arm">
     <chain base_link="teleop_link0" tip_link="TCP"/>

File: descriptions/solo_description/robots/solo.srdf.xacro (robot description, xacro)
@@ -1,8 +1,4 @@
 <?xml version="1.0" ?>
 <robot name="solo" xmlns:xacro="http://ros.org/wiki/xacro">
-<xacro:arg name="arm" default="false"/>
-    <group name="bases">
-      <link name="base_link"/>
-    </group>
     <group name="lf_leg">
         <joint name="lf_haa_joint" />

File: descriptions/spot_description/robots/spot.srdf.xacro (robot description, xacro)
@@ -1,8 +1,4 @@
 <?xml version="1.0" ?>
 <robot name="spot" xmlns:xacro="http://ros.org/wiki/xacro">
-<xacro:arg name="arm" default="false"/>
-    <group name="base">
-      <link name="base_link"/>
-    </group>
     <group name="lf_leg">
       <chain base_link="base_link" tip_link="lf_foot"/>

File: descriptions/spot_description/robots/spot_kinova.srdf.xacro (robot description, xacro)
@@ -1,8 +1,4 @@
 <?xml version="1.0" ?>
 <robot name="spot" xmlns:xacro="http://ros.org/wiki/xacro">
-    <group name="bases">
-      <link name="base_link"/>
-      <link name="kinova_link_base"/>
-    </group>
     <group name="kinova_arm">
       <chain base_link="kinova_link_base" tip_link="kinova_end_effector"/>

Commit message: Add base to the robot descriptions

File: descriptions/aliengo_description/robots/aliengo.srdf.xacro (robot description, xacro)
@@ -1,4 +1,7 @@
 <?xml version="1.0" ?>
 <robot name="aliengo" xmlns:xacro="http://ros.org/wiki/xacro">
+    <group name="base">
+      <link name="base_link"/>
+    </group>
     <group name="lf_leg">
       <chain base_link="base_link" tip_link="lf_foot"/>

File: descriptions/aliengo_description/robots/aliengo_kinova.srdf.xacro (robot description, xacro)
@@ -1,4 +1,7 @@
 <?xml version="1.0" ?>
 <robot name="aliengo" xmlns:xacro="http://ros.org/wiki/xacro">
+  <group name="base">
+    <link name="base_link"/>
+  </group>
   <group name="kinova_arm">
     <chain base_link="kinova_link_base" tip_link="kinova_end_effector"/>

File: descriptions/anymal_description/robots/anymal.srdf.xacro (robot description, xacro)
@@ -1,4 +1,7 @@
 <?xml version="1.0" ?>
 <robot name="anymal" xmlns:xacro="http://ros.org/wiki/xacro">
+  <group name="base">
+    <link name="base_link"/>
+  </group>
   <group name="lf_leg">
     <chain base_link="base_link" tip_link="lf_foot"/>

File: descriptions/hyq_description/robots/hyq.srdf.xacro (robot description, xacro)
@@ -1,4 +1,7 @@
 <?xml version="1.0" ?>
 <robot name="hyq" xmlns:xacro="http://ros.org/wiki/xacro">
+  <group name="base">
+    <link name="base_link"/>
+  </group>
   <group name="lf_leg">
     <chain base_link="trunk" tip_link="lf_foot"/>

File: descriptions/hyq_description/robots/hyq_kinova.srdf.xacro (robot description, xacro)
@@ -1,4 +1,7 @@
 <?xml version="1.0" ?>
 <robot name="hyq" xmlns:xacro="http://ros.org/wiki/xacro">
+ <group name="base">
+   <link name="base_link"/>
+ </group>
   <group name="kinova_arm">
     <chain base_link="kinova_link_base" tip_link="kinova_end_effector"/>

File: descriptions/hyq_description/robots/hyq_teleop.srdf.xacro (robot description, xacro)
@@ -1,4 +1,7 @@
 <?xml version="1.0" ?>
 <robot name="hyq" xmlns:xacro="http://ros.org/wiki/xacro">
+  <group name="base">
+    <link name="base_link"/>
+  </group>
   <group name="teleop_arm">
     <chain base_link="teleop_link0" tip_link="TCP"/>

File: descriptions/solo_description/robots/solo.srdf.xacro (robot description, xacro)
@@ -1,4 +1,7 @@
 <?xml version="1.0" ?>
 <robot name="solo" xmlns:xacro="http://ros.org/wiki/xacro">
+    <group name="base">
+      <link name="base_link"/>
+    </group>
     <group name="lf_leg">
         <joint name="lf_haa_joint" />

File: descriptions/spot_description/robots/spot.srdf.xacro (robot description, xacro)
@@ -1,4 +1,7 @@
 <?xml version="1.0" ?>
 <robot name="spot" xmlns:xacro="http://ros.org/wiki/xacro">
+    <group name="base">
+      <link name="base_link"/>
+    </group>
     <group name="lf_leg">
       <chain base_link="base_link" tip_link="lf_foot"/>

Commit message: Add bellydown

File: descriptions/aliengo_description/robots/aliengo.srdf.xacro (robot description, xacro)
@@ -60,3 +60,17 @@
         <joint name="rh_kfe_joint" value="-1.3"/>
     </group_state>
+    <group_state group="chains" name="bellydown">
+        <joint name="lf_haa_joint" value="0.60"/>
+        <joint name="lf_hfe_joint" value="1.70"/>
+        <joint name="lf_kfe_joint" value="-2.78"/>
+        <joint name="rf_haa_joint" value="-0.60"/>
+        <joint name="rf_hfe_joint" value="1.70"/>
+        <joint name="rf_kfe_joint" value="-2.78"/>
+        <joint name="lh_haa_joint" value="0.60"/>
+        <joint name="lh_hfe_joint" value="1.52"/>
+        <joint name="lh_kfe_joint" value="-2.78"/>
+        <joint name="rh_haa_joint" value="-0.60"/>
+        <joint name="rh_hfe_joint" value="1.52"/>
+        <joint name="rh_kfe_joint" value="-2.78"/>
+    </group_state>
 </robot>

File: descriptions/anymalc_description/robots/anymalc.srdf.xacro (robot description, xacro)
@@ -60,3 +60,17 @@
     <joint name="rh_kfe_joint" value="1.0"/>
   </group_state>
+  <group_state group="chains" name="bellydown">
+    <joint name="lf_haa_joint" value="0.0"/>
+    <joint name="lf_hfe_joint" value="1.60"/>
+    <joint name="lf_kfe_joint" value="-2.60"/>
+    <joint name="rf_haa_joint" value="0.0"/>
+    <joint name="rf_hfe_joint" value="1.60"/>
+    <joint name="rf_kfe_joint" value="-2.60"/>
+    <joint name="lh_haa_joint" value="0.0"/>
+    <joint name="lh_hfe_joint" value="-1.60"/>
+    <joint name="lh_kfe_joint" value="2.60"/>
+    <joint name="rh_haa_joint" value="0.0"/>
+    <joint name="rh_hfe_joint" value="-1.60"/>
+    <joint name="rh_kfe_joint" value="2.60"/>
+  </group_state>
 </robot>

File: descriptions/spot_description/robots/spot.srdf.xacro (robot description, xacro)
@@ -49,14 +49,28 @@
         <joint name="lf_haa_joint" value="0.20"/>
         <joint name="lf_hfe_joint" value="0.70"/>
-        <joint name="lf_kfe_joint"  value="-1.35"/>
+        <joint name="lf_kfe_joint" value="-1.35"/>
         <joint name="rf_haa_joint" value="-0.20"/>
         <joint name="rf_hfe_joint" value="0.70"/>
-        <joint name="rf_kfe_joint"  value="-1.35"/>
+        <joint name="rf_kfe_joint" value="-1.35"/>
         <joint name="lh_haa_joint" value="0.20"/>
         <joint name="lh_hfe_joint" value="0.70"/>
-        <joint name="lh_kfe_joint"  value="-1.35"/>
+        <joint name="lh_kfe_joint" value="-1.35"/>
         <joint name="rh_haa_joint" value="-0.20"/>
         <joint name="rh_hfe_joint" value="0.70"/>
-        <joint name="rh_kfe_joint"  value="-1.35"/>
+        <joint name="rh_kfe_joint" value="-1.35"/>
+    </group_state>
+    <group_state group="chains" name="bellydown">
+        <joint name="lf_haa_joint" value="0.5"/>
+        <joint name="lf_hfe_joint" value="1.75"/>
+        <joint name="lf_kfe_joint" value="-2.8"/>
+        <joint name="rf_haa_joint" value="0.5"/>
+        <joint name="rf_hfe_joint" value="1.75"/>
+        <joint name="rf_kfe_joint" value="-2.8"/>
+        <joint name="lh_haa_joint" value="-0.75"/>
+        <joint name="lh_hfe_joint" value="1.60"/>
+        <joint name="lh_kfe_joint" value="-2.6"/>
+        <joint name="rh_haa_joint" value="-0.75"/>
+        <joint name="rh_hfe_joint" value="1.60"/>
+        <joint name="rh_kfe_joint" value="-2.6"/>
     </group_state>
 </robot>

Commit message: Fix joint limits violation in aliengo and spot standown

File: descriptions/aliengo_description/robots/aliengo.srdf.xacro (robot description, xacro)
@@ -63,14 +63,14 @@
         <joint name="lf_haa_joint" value="0.60"/>
         <joint name="lf_hfe_joint" value="1.70"/>
-        <joint name="lf_kfe_joint" value="-2.78"/>
+        <joint name="lf_kfe_joint" value="-2.77"/>
         <joint name="rf_haa_joint" value="-0.60"/>
         <joint name="rf_hfe_joint" value="1.70"/>
-        <joint name="rf_kfe_joint" value="-2.78"/>
+        <joint name="rf_kfe_joint" value="-2.77"/>
         <joint name="lh_haa_joint" value="0.60"/>
         <joint name="lh_hfe_joint" value="1.52"/>
-        <joint name="lh_kfe_joint" value="-2.78"/>
+        <joint name="lh_kfe_joint" value="-2.77"/>
         <joint name="rh_haa_joint" value="-0.60"/>
         <joint name="rh_hfe_joint" value="1.52"/>
-        <joint name="rh_kfe_joint" value="-2.78"/>
+        <joint name="rh_kfe_joint" value="-2.77"/>
     </group_state>
 </robot>

File: descriptions/spot_description/robots/spot.srdf.xacro (robot description, xacro)
@@ -63,8 +63,8 @@
         <joint name="lf_haa_joint" value="0.5"/>
         <joint name="lf_hfe_joint" value="1.75"/>
-        <joint name="lf_kfe_joint" value="-2.8"/>
+        <joint name="lf_kfe_joint" value="-2.79"/>
         <joint name="rf_haa_joint" value="0.5"/>
         <joint name="rf_hfe_joint" value="1.75"/>
-        <joint name="rf_kfe_joint" value="-2.8"/>
+        <joint name="rf_kfe_joint" value="-2.79"/>
         <joint name="lh_haa_joint" value="-0.75"/>
         <joint name="lh_hfe_joint" value="1.60"/>
