Commit message: Remove unecessary xacro lines from aliengo

File: descriptions/aliengo_description/robots/aliengo.urdf.xacro (robot description, xacro)
@@ -150,20 +150,3 @@
     <xacro:leg_transmission name="lh"/>
     <xacro:leg_gazebo name="lh" load_force_sensors="$(arg load_force_sensors)"/>
-    <xacro:if value="$(arg sensors)">
-        <!-- IMU trunk -->
-        <xacro:microstrain_3dmgx425_imu
-                parent="base_link"
-                imu_name="trunk_imu"
-                imu_topic="trunk_imu_1/data"
-                update_rate="250">
-                <origin xyz="0.27025 0.000 0.0967678" rpy="0 0 0"/>
-        </xacro:microstrain_3dmgx425_imu>
-        <xacro:kvh_1775_imu
-                parent="base_link"
-                imu_name="kvh_imu"
-                imu_topic="kvh_imu/data"
-                update_rate="250">
-                <origin xyz="0.316115 0.00 0.0887678" rpy="0 ${PI} ${PI/4}"/>
-        </xacro:kvh_1775_imu>
-    </xacro:if>
 </robot>

Commit message: Add imu to aliengo

File: descriptions/aliengo_description/robots/aliengo.urdf.xacro (robot description, xacro)
@@ -6,4 +6,5 @@
     <xacro:arg name="arm_enabled" default="false"/>
     <xacro:arg name="arm_name" default="kinova"/>
+    <xacro:arg name="sensors" default="false"/>
     <xacro:include filename="$(find aliengo_description)/urdfs/const.xacro"/>
     <xacro:include filename="$(find aliengo_description)/urdfs/materials.xacro"/>
@@ -16,4 +17,8 @@
          <xacro:arg name="task_period" value="$(arg task_period)"/>
     </xacro:include>
+    <!-- sensors -->
+    <xacro:if value="$(arg sensors)">
+        <xacro:include filename="$(find sensors_description)/urdfs/sensors/imu.gazebo.xacro"/>
+    </xacro:if>
     <!-- Rollover Protection mode will add an additional stick on the top, use "true" or "false" to switch it. -->
     <xacro:property name="rolloverProtection" value="false"/>
@@ -107,8 +112,8 @@
     <joint name="imu_joint" type="fixed">
         <parent link="trunk"/>
-        <child link="imu_link"/>
+        <child link="trunk_imu"/>
         <origin rpy="0 0 0" xyz="0 0 0"/>
     </joint>
-    <link name="imu_link">
+    <link name="trunk_imu">
         <inertial>
             <mass value="0.001"/>
@@ -155,3 +160,18 @@
            <xacro:include filename="$(find aliengo_description)/urdfs/arm/$(arg arm_name)_adapter.urdf.xacro" /> -->
     </xacro:if>
+    <xacro:if value="$(arg sensors)">
+            <xacro:imu_sensor
+                imu_name="trunk_imu"
+                imu_topic="trunk_imu/data"
+                update_rate="250"
+                rate_mean="0"
+                rate_stddev="0"
+                rate_bias_mean="0"
+                rate_bias_stddev="0"
+                accel_mean="0"
+                accel_stddev="0"
+                accel_bias_mean="0"
+                accel_bias_stddev="0">
+            </xacro:imu_sensor>
+    </xacro:if>
 </robot>

Commit message: Ported aliengo to 20.04

File: descriptions/aliengo_description/robots/aliengo.urdf.xacro (robot description, xacro)
@@ -6,4 +6,5 @@
     <xacro:arg name="arm_enabled" default="false"/>
     <xacro:arg name="arm_name" default="kinova"/>
+    <xacro:arg name="floating_base_link" default="true"/>
     <xacro:include filename="$(find aliengo_description)/urdfs/const.xacro"/>
     <xacro:include filename="$(find aliengo_description)/urdfs/materials.xacro"/>
@@ -36,10 +37,12 @@
     </link>
     <!-- Floating-base Joint -->
-    <link name="world"/>
-    <joint name="floating_base_joint" type="floating">
-      <origin rpy="0 0 0" xyz="0 0 0"/>
-      <parent link="world"/>
-      <child link="base_link"/>
-    </joint>
+    <xacro:if value="$(arg floating_base_link)">
+	    <link name="world"/>
+	    <joint name="floating_base_joint" type="floating">
+	      <origin rpy="0 0 0" xyz="0 0 0"/>
+	      <parent link="world"/>
+	      <child link="base_link"/>
+	    </joint>
+    </xacro:if>
     <joint name="floating_base" type="fixed">
       <origin rpy="0 0 0" xyz="0 0 0"/>

Commit message: Use trunk instead of base_link in aliengo, fix missing ifxacro floating_base

File: descriptions/aliengo_description/robots/aliengo.urdf.xacro (robot description, xacro)
@@ -7,4 +7,5 @@
     <xacro:arg name="arm_name" default="kinova"/>
     <xacro:arg name="sensors" default="false"/>
+    <xacro:arg name="floating_base_link" default="true"/>
     <xacro:include filename="$(find aliengo_description)/urdfs/const.xacro"/>
     <xacro:include filename="$(find aliengo_description)/urdfs/materials.xacro"/>
@@ -32,24 +33,13 @@
         </joint>
     </xacro:if>  -->
-    <link name="base_link">
-        <visual>
-            <origin rpy="0 0 0" xyz="0 0 0"/>
-            <geometry>
-                <box size="0.001 0.001 0.001"/>
-            </geometry>
-        </visual>
-    </link>
     <!-- Floating-base Joint -->
-    <link name="world"/>
-    <joint name="floating_base_joint" type="floating">
-      <origin rpy="0 0 0" xyz="0 0 0"/>
-      <parent link="world"/>
-      <child link="base_link"/>
-    </joint>
-    <joint name="floating_base" type="fixed">
-      <origin rpy="0 0 0" xyz="0 0 0"/>
-      <parent link="base_link"/>
-      <child link="trunk"/>
-    </joint>
+    <xacro:if value="$(arg floating_base_link)">
+            <link name="world"/>
+            <joint name="floating_base_joint" type="floating">
+              <origin rpy="0 0 0" xyz="0 0 0"/>
+              <parent link="world"/>
+              <child link="trunk"/>
+            </joint>
+    </xacro:if>
     <link name="trunk">
         <visual>
