Commit message: Fix hardcoded aliengo in wolf_description_utils leg xacros

File: descriptions/aliengo_description/robots/aliengo.urdf.xacro (robot description, xacro)
@@ -140,12 +140,12 @@
     <!-- <xacro:stairs stairs="15" xpos="0" ypos="2.0" zpos="0" /> -->
     <!-- Extensions -->
-    <xacro:leg_transmission name="rf"/>
-    <xacro:leg_gazebo name="rf" load_force_sensors="$(arg load_force_sensors)"/>
-    <xacro:leg_transmission name="lf"/>
-    <xacro:leg_gazebo name="lf" load_force_sensors="$(arg load_force_sensors)"/>
-    <xacro:leg_transmission name="rh"/>
-    <xacro:leg_gazebo name="rh" load_force_sensors="$(arg load_force_sensors)"/>
-    <xacro:leg_transmission name="lh"/>
-    <xacro:leg_gazebo name="lh" load_force_sensors="$(arg load_force_sensors)"/>
+    <xacro:leg_transmission prefix="rf"/>
+    <xacro:leg_gazebo prefix="rf" robot_name="$(arg robot_name)" load_force_sensors="$(arg load_force_sensors)"/>
+    <xacro:leg_transmission prefix="lf"/>
+    <xacro:leg_gazebo prefix="lf" robot_name="$(arg robot_name)" load_force_sensors="$(arg load_force_sensors)"/>
+    <xacro:leg_transmission prefix="rh"/>
+    <xacro:leg_gazebo prefix="rh" robot_name="$(arg robot_name)" load_force_sensors="$(arg load_force_sensors)"/>
+    <xacro:leg_transmission prefix="lh"/>
+    <xacro:leg_gazebo prefix="lh" robot_name="$(arg robot_name)" load_force_sensors="$(arg load_force_sensors)"/>
     <xacro:if value="$(arg arm_enabled)">
            <xacro:include filename="$(find aliengo_description)/urdfs/arm/$(arg arm_name)_adapter.urdf.xacro" /> -->

File: descriptions/anymal_description/robots/anymal.urdf.xacro (robot description, xacro)
@@ -727,11 +727,11 @@
     </link>
     <!-- Extensions -->
-    <xacro:leg_transmission name="rf"/>
-    <xacro:leg_gazebo name="rf" load_force_sensors="$(arg load_force_sensors)"/>
-    <xacro:leg_transmission name="lf"/>
-    <xacro:leg_gazebo name="lf" load_force_sensors="$(arg load_force_sensors)"/>
-    <xacro:leg_transmission name="rh"/>
-    <xacro:leg_gazebo name="rh" load_force_sensors="$(arg load_force_sensors)"/>
-    <xacro:leg_transmission name="lh"/>
-    <xacro:leg_gazebo name="lh" load_force_sensors="$(arg load_force_sensors)"/>
+    <xacro:leg_transmission prefix="rf"/>
+    <xacro:leg_gazebo prefix="rf" robot_name="$(arg robot_name)" load_force_sensors="$(arg load_force_sensors)"/>
+    <xacro:leg_transmission prefix="lf"/>
+    <xacro:leg_gazebo prefix="lf" robot_name="$(arg robot_name)" load_force_sensors="$(arg load_force_sensors)"/>
+    <xacro:leg_transmission prefix="rh"/>
+    <xacro:leg_gazebo prefix="rh" robot_name="$(arg robot_name)" load_force_sensors="$(arg load_force_sensors)"/>
+    <xacro:leg_transmission prefix="lh"/>
+    <xacro:leg_gazebo prefix="lh" robot_name="$(arg robot_name)" load_force_sensors="$(arg load_force_sensors)"/>
 </robot>

File: descriptions/anymalc_description/robots/anymalc.urdf.xacro (robot description, xacro)
@@ -1620,11 +1620,11 @@
     </link>
     <!-- Extensions -->
-    <xacro:leg_transmission name="rf"/>
-    <xacro:leg_gazebo name="rf" load_force_sensors="$(arg load_force_sensors)"/>
-    <xacro:leg_transmission name="lf"/>
-    <xacro:leg_gazebo name="lf" load_force_sensors="$(arg load_force_sensors)"/>
-    <xacro:leg_transmission name="rh"/>
-    <xacro:leg_gazebo name="rh" load_force_sensors="$(arg load_force_sensors)"/>
-    <xacro:leg_transmission name="lh"/>
-    <xacro:leg_gazebo name="lh" load_force_sensors="$(arg load_force_sensors)"/>
+    <xacro:leg_transmission prefix="rf"/>
+    <xacro:leg_gazebo prefix="rf" robot_name="$(arg robot_name)" load_force_sensors="$(arg load_force_sensors)"/>
+    <xacro:leg_transmission prefix="lf"/>
+    <xacro:leg_gazebo prefix="lf" robot_name="$(arg robot_name)" load_force_sensors="$(arg load_force_sensors)"/>
+    <xacro:leg_transmission prefix="rh"/>
+    <xacro:leg_gazebo prefix="rh" robot_name="$(arg robot_name)" load_force_sensors="$(arg load_force_sensors)"/>
+    <xacro:leg_transmission prefix="lh"/>
+    <xacro:leg_gazebo prefix="lh" robot_name="$(arg robot_name)" load_force_sensors="$(arg load_force_sensors)"/>
 </robot>

File: descriptions/hyq_description/robots/hyq.urdf.xacro (robot description, xacro)
@@ -27,5 +27,5 @@
 	<!-- LF leg -->
 	<xacro:hyq_leg
-		name="lf"
+                prefix="lf"
 		parent="trunk"
 		reflect_hip="1"
@@ -38,5 +38,5 @@
 	<!-- RF leg -->
 	<xacro:hyq_leg
-		name="rf"
+                prefix="rf"
 		parent="trunk"
 		reflect_hip="-1"
@@ -49,5 +49,5 @@
 	<!-- LH leg -->
 	<xacro:hyq_leg
-		name="lh"
+                prefix="lh"
 		parent="trunk"
 		reflect_hip="-1"
@@ -60,5 +60,5 @@
 	<!-- RH leg -->
 	<xacro:hyq_leg
-		name="rh"
+                prefix="rh"
 		parent="trunk"
 		reflect_hip="1"

File: descriptions/hyq_description/urdfs/leg/leg.urdf.xacro (robot description, xacro)
@@ -3,11 +3,11 @@
 	<!-- ================================== Leg ================================== -->
 	<!-- The xacro macro xacro:hyq_leg contains: hip assembly, upper and lower leg -->
-	<xacro:macro name="hyq_leg" params="name parent *origin reflect_hip reflect_upper reflect_front knee_bent_backward load_force_sensors">
+        <xacro:macro name="hyq_leg" params="prefix parent *origin reflect_hip reflect_upper reflect_front knee_bent_backward load_force_sensors">
 		<!-- Joints -->
 		<!-- Hip assembly joint -->
-		<joint name="${name}_haa_joint" type="revolute">
+                <joint name="${prefix}_haa_joint" type="revolute">
 			<xacro:insert_block name="origin"/>
 			<parent link="${parent}"/>
-			<child  link="${name}_hipassembly"/>
+                        <child  link="${prefix}_hipassembly"/>
 			<axis xyz="0 0 1"/>
 			<limit effort="${haa_limit}" velocity="12.0" lower="${haa_min*PI/180}" upper="${haa_max*PI/180}" />
@@ -17,8 +17,8 @@
 		</joint>
 		<!-- Upper leg joint -->
-		<joint name="${name}_hfe_joint" type="revolute">
+                <joint name="${prefix}_hfe_joint" type="revolute">
 			<origin xyz="${hipassembly_length} 0 0" rpy="${reflect_upper*PI/2} 0 0"/>
-			<parent link="${name}_hipassembly"/>
-			<child  link="${name}_upperleg"/>
+                        <parent link="${prefix}_hipassembly"/>
+                        <child  link="${prefix}_upperleg"/>
 			<axis xyz="0 0 1"/>
 			<limit effort="${hfe_limit}" velocity="12.0"
@@ -31,8 +31,8 @@
 		</joint>
 		<!-- Lower leg joint -->
-		<joint name="${name}_kfe_joint" type="revolute">
+                <joint name="${prefix}_kfe_joint" type="revolute">
 			<origin xyz="${upperleg_length} 0 0" rpy="0 0 0"/>
-			<parent link="${name}_upperleg"/>
-			<child  link="${name}_lowerleg"/>
+                        <parent link="${prefix}_upperleg"/>
+                        <child  link="${prefix}_lowerleg"/>
 			<axis xyz="0 0 1"/>
 			<limit effort="${kfe_limit}" velocity="12.0"
@@ -45,12 +45,12 @@
 		<!-- Foot joint -->
 		</joint>
-		<joint name="${name}_foot_joint" type="fixed">
+                <joint name="${prefix}_foot_joint" type="fixed">
 			<origin xyz="${lowerleg_length} 0 0" rpy="${PI/2} 0 ${-PI/2}"/>
-			<parent link="${name}_lowerleg"/>
-			<child  link="${name}_foot"/>
+                        <parent link="${prefix}_lowerleg"/>
+                        <child  link="${prefix}_foot"/>
 		</joint>
 		<!-- Links -->
 		<!-- Hip assembly link -->
-		<link name="${name}_hipassembly">
+                <link name="${prefix}_hipassembly">
 			<inertial>
 				<origin xyz="${xcom_hipassembly}
@@ -75,5 +75,5 @@
 		</link>
 		<!-- Upper leg link -->
-		<link name="${name}_upperleg">
+                <link name="${prefix}_upperleg">
 			<inertial>
 				<origin xyz="${xcom_upperleg} ${-reflect_front*ycom_upperleg} ${zcom_upperleg}"/>
@@ -96,5 +96,5 @@
 		</link>
 		<!-- Lower leg link -->
-		<link name="${name}_lowerleg">
+                <link name="${prefix}_lowerleg">
 			<inertial>
 				<origin xyz="${xcom_lowerleg} ${reflect_front*ycom_lowerleg} ${reflect_front*zcom_lowerleg}"/>
@@ -117,5 +117,5 @@
 		</link>
 		<!-- Foot link -->
-		<link name="${name}_foot">
+                <link name="${prefix}_foot">
 			<collision>
 				<origin xyz="0 0 0" rpy="0 0 0"/>
@@ -132,6 +132,6 @@
 		</link>
 		<!-- Extensions -->
-		<xacro:leg_transmission name="${name}"/>
-		<xacro:leg_gazebo name="${name}" load_force_sensors="${load_force_sensors}"/>
+                <xacro:leg_transmission prefix="${prefix}"/>
+                <xacro:leg_gazebo prefix="${prefix}" robot_name="hyq" load_force_sensors="${load_force_sensors}"/>
 	</xacro:macro>
 </robot>

File: descriptions/minicheetah_description/robots/minicheetah.urdf.xacro (robot description, xacro)
@@ -718,11 +718,11 @@
   </joint>
   <!-- Extensions -->
-  <xacro:leg_transmission name="rf"/>
-  <xacro:leg_gazebo name="rf" load_force_sensors="$(arg load_force_sensors)"/>
-  <xacro:leg_transmission name="lf"/>
-  <xacro:leg_gazebo name="lf" load_force_sensors="$(arg load_force_sensors)"/>
-  <xacro:leg_transmission name="rh"/>
-  <xacro:leg_gazebo name="rh" load_force_sensors="$(arg load_force_sensors)"/>
-  <xacro:leg_transmission name="lh"/>
-  <xacro:leg_gazebo name="lh" load_force_sensors="$(arg load_force_sensors)"/>
+  <xacro:leg_transmission prefix="rf"/>
+  <xacro:leg_gazebo prefix="rf" robot_name="$(arg robot_name)" load_force_sensors="$(arg load_force_sensors)"/>
+  <xacro:leg_transmission prefix="lf"/>
+  <xacro:leg_gazebo prefix="lf" robot_name="$(arg robot_name)" load_force_sensors="$(arg load_force_sensors)"/>
+  <xacro:leg_transmission prefix="rh"/>
+  <xacro:leg_gazebo prefix="rh" robot_name="$(arg robot_name)" load_force_sensors="$(arg load_force_sensors)"/>
+  <xacro:leg_transmission prefix="lh"/>
+  <xacro:leg_gazebo prefix="lh" robot_name="$(arg robot_name)" load_force_sensors="$(arg load_force_sensors)"/>
 </robot>

File: descriptions/spot_description/robots/spot.urdf.xacro (robot description, xacro)
@@ -550,12 +550,12 @@
     <xacro:include filename="$(find spot_description)/urdfs/accessories.urdf.xacro" />
     <!-- Extensions -->
-    <xacro:leg_transmission name="rf"/>
-    <xacro:leg_gazebo name="rf" load_force_sensors="$(arg load_force_sensors)"/>
-    <xacro:leg_transmission name="lf"/>
-    <xacro:leg_gazebo name="lf" load_force_sensors="$(arg load_force_sensors)"/>
-    <xacro:leg_transmission name="rh"/>
-    <xacro:leg_gazebo name="rh" load_force_sensors="$(arg load_force_sensors)"/>
-    <xacro:leg_transmission name="lh"/>
-    <xacro:leg_gazebo name="lh" load_force_sensors="$(arg load_force_sensors)"/>
+    <xacro:leg_transmission prefix="rf"/>
+    <xacro:leg_gazebo prefix="rf" robot_name="$(arg robot_name)" load_force_sensors="$(arg load_force_sensors)"/>
+    <xacro:leg_transmission prefix="lf"/>
+    <xacro:leg_gazebo prefix="lf" robot_name="$(arg robot_name)" load_force_sensors="$(arg load_force_sensors)"/>
+    <xacro:leg_transmission prefix="rh"/>
+    <xacro:leg_gazebo prefix="rh" robot_name="$(arg robot_name)" load_force_sensors="$(arg load_force_sensors)"/>
+    <xacro:leg_transmission prefix="lh"/>
+    <xacro:leg_gazebo prefix="lh" robot_name="$(arg robot_name)" load_force_sensors="$(arg load_force_sensors)"/>
     <xacro:if value="$(arg arm_enabled)">
            <xacro:include filename="$(find spot_description)/urdfs/arm/$(arg arm_name)_adapter.urdf.xacro" /> -->

File: descriptions/wolf_description_utils/urdfs/leg.gazebo.xacro (robot description, xacro)
@@ -1,45 +1,45 @@
 <?xml version="1.0"?>
 <robot xmlns:xacro="http://ros.org/wiki/xacro">
-	<xacro:macro name="leg_gazebo" params="name load_force_sensors">
-		<gazebo reference="${name}_haa_joint">
+	<xacro:macro name="leg_gazebo" params="prefix robot_name load_force_sensors">
+		<gazebo reference="${prefix}_haa_joint">
 			<provideFeedback>true</provideFeedback>
 		</gazebo>
 		<xacro:if value="${load_force_sensors}">
 			<gazebo>
-				<plugin name="${name}_haa_sensor" filename="libgazebo_ros_ft_sensor.so">
-                                        <robotNamespace>/aliengo/internal_wrench/</robotNamespace>
+				<plugin name="${prefix}_haa_sensor" filename="libgazebo_ros_ft_sensor.so">
+                                        <robotNamespace>/${robot_name}/internal_wrench/</robotNamespace>
 					<updateRate>100.0</updateRate>
-					<topicName>${name}_haa_joint</topicName>
-					<jointName>${name}_haa_joint</jointName>
+					<topicName>${prefix}_haa_joint</topicName>
+					<jointName>${prefix}_haa_joint</jointName>
 				</plugin>
 			</gazebo>
 		</xacro:if>
-		<gazebo reference="${name}_kfe_joint">
+		<gazebo reference="${prefix}_kfe_joint">
 			<provideFeedback>true</provideFeedback>
 		</gazebo>
 		<xacro:if value="${load_force_sensors}">
 			<gazebo>
-				<plugin name="${name}_kfe_sensor" filename="libgazebo_ros_ft_sensor.so">
-                                        <robotNamespace>/aliengo/internal_wrench/</robotNamespace>
+				<plugin name="${prefix}_kfe_sensor" filename="libgazebo_ros_ft_sensor.so">
+                                        <robotNamespace>/${robot_name}/internal_wrench/</robotNamespace>
 					<updateRate>100.0</updateRate>
-					<topicName>${name}_kfe_joint</topicName>
-					<jointName>${name}_kfe_joint</jointName>
+					<topicName>${prefix}_kfe_joint</topicName>
+					<jointName>${prefix}_kfe_joint</jointName>
 				</plugin>
 			</gazebo>
 		</xacro:if>
-		<gazebo reference="${name}_hfe_joint">
+		<gazebo reference="${prefix}_hfe_joint">
 			<provideFeedback>true</provideFeedback>
 		</gazebo>
 		<xacro:if value="${load_force_sensors}">
 			<gazebo>
-				<plugin name="${name}_hfe_sensor" filename="libgazebo_ros_ft_sensor.so">
-                                        <robotNamespace>/aliengo/internal_wrench/</robotNamespace>
+				<plugin name="${prefix}_hfe_sensor" filename="libgazebo_ros_ft_sensor.so">
+                                        <robotNamespace>/${robot_name}/internal_wrench/</robotNamespace>
 					<updateRate>100.0</updateRate>
-					<topicName>${name}_hfe_joint</topicName>
-					<jointName>${name}_hfe_joint</jointName>
+					<topicName>${prefix}_hfe_joint</topicName>
+					<jointName>${prefix}_hfe_joint</jointName>
 				</plugin>
 			</gazebo>
 		</xacro:if>
-		<gazebo reference="${name}_upperleg">
+		<gazebo reference="${prefix}_upperleg">
 			<kp>1000000.0</kp>
 			<kd>100.0</kd>
@@ -50,5 +50,5 @@
 			<minDepth>0.00</minDepth>
 		</gazebo>
-		<gazebo reference="${name}_lowerleg">
+		<gazebo reference="${prefix}_lowerleg">
 			<kp>1000000.0</kp>
 			<kd>100.0</kd>
@@ -57,18 +57,18 @@
 			<maxVel>1.0</maxVel>
 			<maxContacts>1</maxContacts>
-			<sensor name="${name}_shin_contact_sensor" type="contact">
+			<sensor name="${prefix}_shin_contact_sensor" type="contact">
                 <always_on>true</always_on>
                 <update_rate>250.0</update_rate>
                 <contact>
-                  <collision>${name}_lowerleg_collision</collision>
+                  <collision>${prefix}_lowerleg_collision</collision>
                 </contact>
                 <!-- the sensor readings in terms of force torques are expressed in the lowerleg frame
                 because gazebo lumps the fake footframe with the real parent link, the normals are in the world frame-->
-                 <plugin name="${name}_shin_bumper" filename="libgazebo_ros_bumper.so">
-                  <bumperTopicName>/aliengo/${name}_shin_bumper</bumperTopicName>
+                 <plugin name="${prefix}_shin_bumper" filename="libgazebo_ros_bumper.so">
+                  <bumperTopicName>/${robot_name}/${prefix}_shin_bumper</bumperTopicName>
                 </plugin>
             </sensor>
 		</gazebo>
-		<gazebo reference="${name}_foot">
+		<gazebo reference="${prefix}_foot">
                         <kp>1000000.0</kp>
                         <kd>100.0</kd>
@@ -77,15 +77,15 @@
                         <maxVel>1.0</maxVel>
 			<maxContacts>1</maxContacts>
-			<sensor name="${name}_foot_contact_sensor" type="contact">
+			<sensor name="${prefix}_foot_contact_sensor" type="contact">
 				<always_on>true</always_on>
 				<update_rate>250.0</update_rate>
 				<contact>
-					<collision>${name}_lowerleg_fixed_joint_lump__${name}_foot_collision_1</collision>
+					<collision>${prefix}_lowerleg_fixed_joint_lump__${prefix}_foot_collision_1</collision>
 				</contact>
                                 <!-- the sensor readings in terms of force torques are expressed in the lowerleg frame
                                 because gazebo lumps the fake footframe with the real parent link, the normals are in the world frame-->
-				<plugin name="${name}_foot_bumper" filename="libgazebo_ros_bumper.so">
-                                        <bumperTopicName>/aliengo/${name}_foot_bumper</bumperTopicName>
-                                        <robotNamespace>aliengo</robotNamespace>
+				<plugin name="${prefix}_foot_bumper" filename="libgazebo_ros_bumper.so">
+                                        <bumperTopicName>/${robot_name}/${prefix}_foot_bumper</bumperTopicName>
+                                        <robotNamespace>${robot_name}</robotNamespace>
 				</plugin>
 			</sensor>

File: descriptions/wolf_description_utils/urdfs/leg.transmission.xacro (robot description, xacro)
@@ -1,12 +1,12 @@
 <?xml version="1.0"?>
 <robot xmlns:xacro="http://ros.org/wiki/xacro">
-	<xacro:macro name="leg_transmission" params="name">
+        <xacro:macro name="leg_transmission" params="prefix">
     	<!-- Hip assembly -->
-		<transmission name="${name}_haa_trans">
+                <transmission name="${prefix}_haa_trans">
 			<type>transmission_interface/SimpleTransmission</type>
-			<joint name="${name}_haa_joint">
+                        <joint name="${prefix}_haa_joint">
 				<hardwareInterface>EffortJointInterface</hardwareInterface>
 			</joint>
-			<actuator name="${name}_haa_motor">
+                        <actuator name="${prefix}_haa_motor">
 				<hardwareInterface>EffortJointInterface</hardwareInterface>
 				<mechanicalReduction>1</mechanicalReduction>
@@ -14,10 +14,10 @@
 		</transmission>
     	<!-- Upper leg -->
-		<transmission name="${name}_hfe_trans">
+                <transmission name="${prefix}_hfe_trans">
 			<type>transmission_interface/SimpleTransmission</type>
-			<joint name="${name}_hfe_joint">
+                        <joint name="${prefix}_hfe_joint">
 				<hardwareInterface>EffortJointInterface</hardwareInterface>
 			</joint>
-			<actuator name="${name}_hfe_motor">
+                        <actuator name="${prefix}_hfe_motor">
 				<hardwareInterface>EffortJointInterface</hardwareInterface>
 				<mechanicalReduction>1</mechanicalReduction>
@@ -25,10 +25,10 @@
 		</transmission>
     	<!-- Lower leg -->
-		<transmission name="${name}_kfe_trans">
+                <transmission name="${prefix}_kfe_trans">
 			<type>transmission_interface/SimpleTransmission</type>
-			<joint name="${name}_kfe_joint">
+                        <joint name="${prefix}_kfe_joint">
 				<hardwareInterface>EffortJointInterface</hardwareInterface>
 			</joint>
-			<actuator name="${name}_kfe_motor">
+                        <actuator name="${prefix}_kfe_motor">
 				<hardwareInterface>EffortJointInterface</hardwareInterface>
 				<mechanicalReduction>1</mechanicalReduction>
