Commit message: porting solo to 20.04

File: descriptions/solo_description/robots/solo.urdf.xacro (robot description, xacro)
@@ -6,4 +6,5 @@
   xmlns:xacro="http://playerstage.sourceforge.net/gazebo/xmlschema/#interface">
   <xacro:arg name="load_force_sensors" default="false"/>
+  <xacro:arg name="floating_base_link" default="true"/>
   <xacro:property name="color_name" value="grey" />
   <xacro:property name="color" value="0.8 0.8 0.8" />
@@ -13,10 +14,12 @@
         </xacro:include>
                 <!-- Floating-base Joint -->
-                <link name="world"/>
-                <joint name="floating_base_joint" type="floating">
-                    <origin rpy="0 0 0" xyz="0 0 0"/>
-                    <parent link="world"/>
-                    <child link="base_link"/>
-                </joint>
+                <xacro:if value="$(arg floating_base_link)">
+		        <link name="world"/>
+		        <joint name="floating_base_joint" type="floating">
+		            <origin rpy="0 0 0" xyz="0 0 0"/>
+		            <parent link="world"/>
+		            <child link="base_link"/>
+		        </joint>
+	        </xacro:if>
 		<link name="base_link" />
                 <joint name="floating_base" type="fixed">
