Commit message: Update solo

File: descriptions/solo_description/robots/solo.srdf.xacro (robot description, xacro)
@@ -2,18 +2,33 @@
 <robot name="solo" xmlns:xacro="http://ros.org/wiki/xacro">
 <xacro:arg name="arm" default="false"/>
-    <group name="base">
+    <group name="bases">
       <link name="base_link"/>
     </group>
     <group name="lf_leg">
-      <chain base_link="base_link" tip_link="lf_foot"/>
+        <joint name="lf_haa_joint" />
+        <joint name="lf_hfe_joint" />
+        <joint name="lf_kfe_joint" />
+        <chain base_link="base_link" tip_link="lf_foot" />
     </group>
+    <!-- right front leg -->
     <group name="rf_leg">
-      <chain base_link="base_link" tip_link="rf_foot"/>
+        <joint name="rf_haa_joint" />
+        <joint name="rf_hfe_joint" />
+        <joint name="rf_kfe_joint" />
+        <chain base_link="base_link" tip_link="rf_foot" />
     </group>
+    <!-- left hind leg -->
     <group name="lh_leg">
-      <chain base_link="base_link" tip_link="lh_foot"/>
+        <joint name="lh_haa_joint" />
+        <joint name="lh_hfe_joint" />
+        <joint name="lh_kfe_joint" />
+        <chain base_link="base_link" tip_link="lh_foot" />
     </group>
+    <!-- right hind leg -->
     <group name="rh_leg">
-      <chain base_link="base_link" tip_link="rh_foot"/>
+        <joint name="rh_haa_joint" />
+        <joint name="rh_hfe_joint" />
+        <joint name="rh_kfe_joint" />
+        <chain base_link="base_link" tip_link="rh_foot" />
     </group>
     <group name="lf_hip">
@@ -42,16 +57,16 @@
     </group>
   <group_state group="chains" name="home">
-    <joint name="lf_haa_joint" value="0.0"/>
-    <joint name="lf_hfe_joint" value="0.75"/>
-    <joint name="lf_kfe_joint" value="-1.0"/>
-    <joint name="rf_haa_joint" value="0.0"/>
-    <joint name="rf_hfe_joint" value="0.75"/>
-    <joint name="rf_kfe_joint" value="-1.0"/>
-    <joint name="lh_haa_joint" value="0.0"/>
-    <joint name="lh_hfe_joint" value="-0.75"/>
-    <joint name="lh_kfe_joint" value="1.0"/>
-    <joint name="rh_haa_joint" value="0.0"/>
-    <joint name="rh_hfe_joint" value="-0.75"/>
-    <joint name="rh_kfe_joint" value="1.0"/>
+    <joint name="lf_haa_joint" value="-0.2"       />
+    <joint name="lf_hfe_joint" value="0.78539816" />
+    <joint name="lf_kfe_joint" value="-1.57079633"/>
+    <joint name="rf_haa_joint" value="-0.2"       />
+    <joint name="rf_hfe_joint" value="0.78539816" />
+    <joint name="rf_kfe_joint" value="-1.57079633"/>
+    <joint name="lh_haa_joint" value="-0.2"       />
+    <joint name="lh_hfe_joint" value="-0.78539816"/>
+    <joint name="lh_kfe_joint" value="1.57079633" />
+    <joint name="rh_haa_joint" value="-0.2"       />
+    <joint name="rh_hfe_joint" value="-0.78539816"/>
+    <joint name="rh_kfe_joint" value="1.57079633" />
   </group_state>
 </robot>

File: descriptions/solo_description/robots/solo.urdf.xacro (robot description, xacro)
@@ -1,15 +1,11 @@
 <?xml version="1.0" ?>
-<robot name="solo"
-  xmlns:controller="http://playerstage.sourceforge.net/gazebo/xmlschema/#controller"
-  xmlns:interface="http://playerstage.sourceforge.net/gazebo/xmlschema/#interface"
-  xmlns:sensor="http://playerstage.sourceforge.net/gazebo/xmlschema/#sensor"
-  xmlns:xacro="http://playerstage.sourceforge.net/gazebo/xmlschema/#interface">
-  <xacro:arg name="load_force_sensors" default="false"/>
-  <xacro:property name="color_name" value="grey" />
-  <xacro:property name="color" value="0.8 0.8 0.8" />
-  <xacro:property name="opacity" value="1.0" />
-        <xacro:include filename="$(find solo_description)/gazebo/gazebo.urdf.xacro">
-             <xacro:arg name="task_period" value="$(arg task_period)"/>
-        </xacro:include>
+<robot name="solo" xmlns:xacro="http://ros.org/wiki/xacro">
+    <xacro:property name="color_name" value="grey" />
+    <xacro:property name="color" value="0.8 0.8 0.8" />
+    <xacro:property name="opacity" value="1.0" />
+    <xacro:arg name="load_force_sensors" default="false"/>
+    <xacro:include filename="$(find solo_description)/gazebo/gazebo.urdf.xacro">
+        <xacro:arg name="task_period" value="$(arg task_period)"/>
+    </xacro:include>
                 <!-- Floating-base Joint -->
                 <link name="world"/>
@@ -25,78 +21,78 @@
                     <child link="trunk"/>
                 </joint>
-		<link name="trunk">
-			<inertial>
-			    <origin xyz="0 0 0" rpy="0 0 0" />
-			    <mass value="1.63315091"/>
-			    <!-- The base is extremely symmetrical. -->
-			    <inertia ixx="0.00578574" ixy="0.0" ixz="0.0"
-				                      iyy="0.01938108" iyz="0.0"
-				                                       izz="0.02476124"/>
-			</inertial>
-			<visual>
-				<origin xyz="0 0 0" rpy="0 0 0" />
-				    <geometry>
-				      <mesh filename="package://solo_description/meshes/stl/with_foot/solo_body.stl"/>
-				    </geometry>
-				    <material name="${color_name}">
-				        <color rgba="${color} ${opacity}"/>
-				    </material>
-			</visual>
-			<collision>
-		            <origin xyz="0 0 0" rpy="0 0 0" />
-		            <geometry>
-		              <mesh filename="package://solo_description/meshes/stl/with_foot/solo_body.stl"/>
-		            </geometry>
-		            <material name="${color_name}">
-		                <color rgba="${color} ${opacity}"/>
-		            </material>
-               		 </collision>
-			<!-- Bullet specific paramters -->
-		        <contact>
-		          <lateral_friction value="1.0"/>
-		          <restitution value="0.5"/>
-		        </contact>
-		</link>
- 	 <!-- Include the legs -->
-  	<xacro:include filename="$(find solo_description)/urdfs/leg.xacro"/>
-  <!-- Include the front left leg -->
-  <xacro:leg
-      prefix="lf"
-      is_front="true"
-      is_right="false"
-      has_side_motion="true"
-      color_name="${color_name}"
-      color="${color}"
-      opacity="${opacity}"
-      load_force_sensors="$(arg load_force_sensors)"/>
-  <!-- Include the front right leg -->
-  <xacro:leg
-      prefix="rf"
-      is_front="true"
-      is_right="true"
-      has_side_motion="true"
-      color_name="${color_name}"
-      color="${color}"
-      opacity="${opacity}"
-      load_force_sensors="$(arg load_force_sensors)"/>
-  <!-- Include the hind left leg -->
-  <xacro:leg
-      prefix="lh"
-      is_front="false"
-      is_right="false"
-      has_side_motion="true"
-      color_name="${color_name}"
-      color="${color}"
-      opacity="${opacity}"
-      load_force_sensors="$(arg load_force_sensors)"/>
-  <!-- Include the hind right leg -->
-  <xacro:leg
-      prefix="rh"
-      is_front="false"
-      is_right="true"
-      has_side_motion="true"
-      color_name="${color_name}"
-      color="${color}"
-      opacity="${opacity}"
-      load_force_sensors="$(arg load_force_sensors)"/>
+    <link name="trunk">
+        <inertial>
+            <origin xyz="0 0 0" rpy="0 0 0" />
+            <mass value="1.16115091"/>
+            <!-- The base is extremely symmetrical. -->
+            <inertia ixx="0.00578574"   ixy="0.0"           ixz="0.0"
+                                        iyy="0.01938108"    iyz="0.0"
+                                                            izz="0.02476124"/>
+        </inertial>
+        <visual>
+            <origin xyz="0 0 0" rpy="0 0 0" />
+            <geometry>
+                <mesh filename="package://solo_description/meshes/stl/with_foot/solo_body.stl"/>
+            </geometry>
+                <material name="${color_name}">
+                <color rgba="${color} ${opacity}"/>
+            </material>
+        </visual>
+        <collision>
+            <origin xyz="0 0 0" rpy="0 0 0" />
+            <geometry>
+                <mesh filename="package://solo_description/meshes/stl/with_foot/solo_body.stl"/>
+            </geometry>
+            <material name="${color_name}">
+                <color rgba="${color} ${opacity}"/>
+            </material>
+        </collision>
+        <!-- Bullet specific paramters -->
+        <contact>
+            <lateral_friction value="1.0"/>
+            <restitution value="0.5"/>
+        </contact>
+    </link>
+    <!-- Include the legs -->
+    <xacro:include filename="$(find solo_description)/urdfs/leg.xacro"/>
+    <!-- LEFT FRONT LEG -->
+    <xacro:leg
+    prefix="lf"
+    is_front="true"
+    is_right="false"
+    has_side_motion="true"
+    color_name="${color_name}"
+    color="${color}"
+    opacity="${opacity}"
+    load_force_sensors="$(arg load_force_sensors)"/>
+    <!-- RIGHT FRONT LEG -->
+    <xacro:leg
+    prefix="rf"
+    is_front="true"
+    is_right="true"
+    has_side_motion="true"
+    color_name="${color_name}"
+    color="${color}"
+    opacity="${opacity}"
+    load_force_sensors="$(arg load_force_sensors)"/>
+    <!-- LEFT HIND LEG -->
+    <xacro:leg
+    prefix="lh"
+    is_front="false"
+    is_right="false"
+    has_side_motion="true"
+    color_name="${color_name}"
+    color="${color}"
+    opacity="${opacity}"
+    load_force_sensors="$(arg load_force_sensors)"/>
+    <!-- RIGHT HIND LEG -->
+    <xacro:leg
+    prefix="rh"
+    is_front="false"
+    is_right="true"
+    has_side_motion="true"
+    color_name="${color_name}"
+    color="${color}"
+    opacity="${opacity}"
+    load_force_sensors="$(arg load_force_sensors)"/>
 </robot>
