Commit message: playing with solo params...still not working

File: descriptions/solo_description/robots/solo.srdf.xacro (robot description, xacro)
@@ -47,16 +47,16 @@
     </group>
   <group_state group="chains" name="home">
-    <joint name="lf_haa_joint" value="0.2"       />
-    <joint name="lf_hfe_joint" value="0.75" />
-    <joint name="lf_kfe_joint" value="-1.5"/>
-    <joint name="rf_haa_joint" value="0.2"       />
-    <joint name="rf_hfe_joint" value="0.75" />
-    <joint name="rf_kfe_joint" value="-1.5"/>
-    <joint name="lh_haa_joint" value="-0.2"       />
-    <joint name="lh_hfe_joint" value="-0.75"/>
-    <joint name="lh_kfe_joint" value="1.5" />
-    <joint name="rh_haa_joint" value="-0.2"       />
-    <joint name="rh_hfe_joint" value="-0.75"/>
-    <joint name="rh_kfe_joint" value="1.5" />
+    <joint name="lf_haa_joint" value="0."       />
+    <joint name="lf_hfe_joint" value="0.78539816" />
+    <joint name="lf_kfe_joint" value="-1.57079633"/>
+    <joint name="rf_haa_joint" value="0."       />
+    <joint name="rf_hfe_joint" value="0.78539816" />
+    <joint name="rf_kfe_joint" value="-1.57079633"/>
+    <joint name="lh_haa_joint" value="0."       />
+    <joint name="lh_hfe_joint" value="-0.78539816"/>
+    <joint name="lh_kfe_joint" value="1.57079633" />
+    <joint name="rh_haa_joint" value="0."       />
+    <joint name="rh_hfe_joint" value="-0.78539816"/>
+    <joint name="rh_kfe_joint" value="1.57079633" />
   </group_state>
 </robot>

Commit message: Working version, still improvements to do

File: descriptions/solo_description/robots/solo.srdf.xacro (robot description, xacro)
@@ -29,14 +29,14 @@
     </group>
     <group name="lf_hip">
-      <chain base_link="base_link" tip_link="lf_hip_assembly"/>
+      <chain base_link="base_link" tip_link="lf_hipassembly"/>
     </group>
     <group name="rf_hip">
-      <chain base_link="base_link" tip_link="rf_hip_assembly"/>
+      <chain base_link="base_link" tip_link="rf_hipassembly"/>
     </group>
     <group name="lh_hip">
-      <chain base_link="base_link" tip_link="lh_hip_assembly"/>
+      <chain base_link="base_link" tip_link="lh_hipassembly"/>
     </group>
     <group name="rh_hip">
-      <chain base_link="base_link" tip_link="rh_hip_assembly"/>
+      <chain base_link="base_link" tip_link="rh_hipassembly"/>
     </group>
     <group name="chains">
@@ -47,16 +47,16 @@
     </group>
   <group_state group="chains" name="home">
-    <joint name="lf_haa_joint" value="0.2"       />
-    <joint name="lf_hfe_joint" value="0.75" />
-    <joint name="lf_kfe_joint" value="-1.5"/>
-    <joint name="rf_haa_joint" value="0.2"       />
-    <joint name="rf_hfe_joint" value="0.75" />
-    <joint name="rf_kfe_joint" value="-1.5"/>
-    <joint name="lh_haa_joint" value="-0.2"       />
-    <joint name="lh_hfe_joint" value="-0.75"/>
-    <joint name="lh_kfe_joint" value="1.5" />
-    <joint name="rh_haa_joint" value="-0.2"       />
-    <joint name="rh_hfe_joint" value="-0.75"/>
-    <joint name="rh_kfe_joint" value="1.5" />
+  <joint name="lf_haa_joint" value="0."       />
+  <joint name="lf_hfe_joint" value="0.78539816" />
+  <joint name="lf_kfe_joint" value="-1.57079633"/>
+  <joint name="rf_haa_joint" value="0."       />
+  <joint name="rf_hfe_joint" value="0.78539816" />
+  <joint name="rf_kfe_joint" value="-1.57079633"/>
+  <joint name="lh_haa_joint" value="0."       />
+  <joint name="lh_hfe_joint" value="-0.78539816"/>
+  <joint name="lh_kfe_joint" value="1.57079633" />
+  <joint name="rh_haa_joint" value="0."       />
+  <joint name="rh_hfe_joint" value="-0.78539816"/>
+  <joint name="rh_kfe_joint" value="1.57079633" />
   </group_state>
 </robot>

File: descriptions/solo_description/urdfs/leg.xacro (robot description, xacro)
@@ -22,5 +22,5 @@
             <joint name="${prefix}_haa_joint" type="revolute">
                 <parent link="trunk"/>
-                <child link="${prefix}_hip_assembly"/>
+                <child link="${prefix}_hipassembly"/>
                 <limit effort="1000" lower="-10" upper="10" velocity="1000"/>
                 <!-- joints rotates around the x-axis -->
@@ -51,6 +51,6 @@
             </joint>
             <!-- HIP ASSEMBLY -->
-            <link name="${prefix}_hip_assembly">
-            	<!-- create a dummy hip_assembly link to join the two joints -->
+            <link name="${prefix}_hipassembly">
+                <!-- create a dummy hipassembly link to join the two joints -->
             	<!-- HIP ASSEMBLY VISUAL-->
 	            <visual>
@@ -168,6 +168,6 @@
             <!--HFE JOINT-->
             <joint name="${prefix}_hfe_joint" type="revolute">
-                <parent link="${prefix}_hip_assembly"/>
-                <child link="${prefix}_upper_leg"/>
+                <parent link="${prefix}_hipassembly"/>
+                <child link="${prefix}_upperleg"/>
                 <limit effort="1000" lower="-10" upper="10" velocity="1000"/>
                 <!-- joints rotates around the y-axis -->
@@ -189,5 +189,5 @@
             <joint name="${prefix}_hfe_joint" type="revolute">
                 <parent link="trunk"/>
-                <child link="${prefix}_upper_leg"/>
+                <child link="${prefix}_upperleg"/>
                 <limit effort="1000" lower="-10" upper="10" velocity="1000"/>
                 <!-- joints rotates around the y-axis -->
@@ -215,5 +215,5 @@
         </xacro:unless>
         <!-- UPPER LEG LINK -->
-        <link name="${prefix}_upper_leg">
+        <link name="${prefix}_upperleg">
             <!-- UPPER LEG LINK INERTIAL -->
             <xacro:unless value="${is_right}">
@@ -275,6 +275,6 @@
         <!-- KFE JOINT: Joint between the upper leg and the lower leg -->
         <joint name="${prefix}_kfe_joint" type="revolute">
-            <parent link="${prefix}_upper_leg"/>
-            <child link="${prefix}_lower_leg"/>
+            <parent link="${prefix}_upperleg"/>
+            <child link="${prefix}_lowerleg"/>
             <limit effort="1000" lower="-10" upper="10" velocity="1000"/>
             <!-- joints rotates around the y-axis -->
@@ -301,5 +301,5 @@
         </joint>
         <!-- LOWERLEG -->
-        <link name="${prefix}_lower_leg">
+        <link name="${prefix}_lowerleg">
             <!-- LOWER LEG LINK INERTIAL -->
             <xacro:unless value="${is_right}">
@@ -361,5 +361,5 @@
         <!-- ANKLE: (Fixed) joint between the lower leg and the foot -->
         <joint name="${prefix}_ankle" type="fixed">
-            <parent link="${prefix}_lower_leg"/>
+            <parent link="${prefix}_lowerleg"/>
             <child link="${prefix}_foot"/>
             <!-- Joint placement -->
