Commit message: hyqarm -> gen3kinova

File: descriptions/gen3kinova_description/urdfs/arm.urdf.xacro (robot description, xacro)
@@ -1,4 +1,4 @@
 <?xml version="1.0"?>
-<robot name="hyqarm" xmlns:xacro="http://ros.org/wiki/xacro">
+<robot name="gen3kinova" xmlns:xacro="http://ros.org/wiki/xacro">
   <!-- Propagate last link name information because it is the gripper's parent link -->
   <xacro:property name="last_arm_link" value="end_effector_link"/>
@@ -18,14 +18,14 @@
         <origin xyz="0 0 0" rpy="0 0 0" />
         <geometry>
-          <mesh filename="package://hyqarm_description/meshes/base_link.dae" />
-        </geometry>
-        <material name="">
-          <color rgba="0.75294 0.75294 0.75294 1" />
-        </material>
-      </visual>
-      <collision>
-        <origin xyz="0 0 0" rpy="0 0 0" />
-        <geometry>
-          <mesh filename="package://hyqarm_description/meshes/base_link.dae" />
+          <mesh filename="package://gen3kinova_description/meshes/base_link.dae" />
+        </geometry>
+        <material name="">
+          <color rgba="0.75294 0.75294 0.75294 1" />
+        </material>
+      </visual>
+      <collision>
+        <origin xyz="0 0 0" rpy="0 0 0" />
+        <geometry>
+          <mesh filename="package://gen3kinova_description/meshes/base_link.dae" />
         </geometry>
       </collision>
@@ -40,14 +40,14 @@
         <origin xyz="0 0 0" rpy="0 0 0" />
         <geometry>
-          <mesh filename="package://hyqarm_description/meshes/shoulder_link.dae" />
-        </geometry>
-        <material name="">
-          <color rgba="0.75294 0.75294 0.75294 1" />
-        </material>
-      </visual>
-      <collision>
-        <origin xyz="0 0 0" rpy="0 0 0" />
-        <geometry>
-          <mesh filename="package://hyqarm_description/meshes/shoulder_link.dae" />
+          <mesh filename="package://gen3kinova_description/meshes/shoulder_link.dae" />
+        </geometry>
+        <material name="">
+          <color rgba="0.75294 0.75294 0.75294 1" />
+        </material>
+      </visual>
+      <collision>
+        <origin xyz="0 0 0" rpy="0 0 0" />
+        <geometry>
+          <mesh filename="package://gen3kinova_description/meshes/shoulder_link.dae" />
         </geometry>
       </collision>
@@ -69,14 +69,14 @@
         <origin xyz="0 0 0" rpy="0 0 0" />
         <geometry>
-          <mesh filename="package://hyqarm_description/meshes/bicep_link.dae" />
-        </geometry>
-        <material name="">
-          <color rgba="0.75294 0.75294 0.75294 1" />
-        </material>
-      </visual>
-      <collision>
-        <origin xyz="0 0 0" rpy="0 0 0" />
-        <geometry>
-          <mesh filename="package://hyqarm_description/meshes/bicep_link.dae" />
+          <mesh filename="package://gen3kinova_description/meshes/bicep_link.dae" />
+        </geometry>
+        <material name="">
+          <color rgba="0.75294 0.75294 0.75294 1" />
+        </material>
+      </visual>
+      <collision>
+        <origin xyz="0 0 0" rpy="0 0 0" />
+        <geometry>
+          <mesh filename="package://gen3kinova_description/meshes/bicep_link.dae" />
         </geometry>
       </collision>
@@ -98,14 +98,14 @@
         <origin xyz="0 0 0" rpy="0 0 0" />
         <geometry>
-          <mesh filename="package://hyqarm_description/meshes/forearm_link.dae" />
-        </geometry>
-        <material name="">
-          <color rgba="0.75294 0.75294 0.75294 1" />
-        </material>
-      </visual>
-      <collision>
-        <origin xyz="0 0 0" rpy="0 0 0" />
-        <geometry>
-          <mesh filename="package://hyqarm_description/meshes/forearm_link.dae" />
+          <mesh filename="package://gen3kinova_description/meshes/forearm_link.dae" />
+        </geometry>
+        <material name="">
+          <color rgba="0.75294 0.75294 0.75294 1" />
+        </material>
+      </visual>
+      <collision>
+        <origin xyz="0 0 0" rpy="0 0 0" />
+        <geometry>
+          <mesh filename="package://gen3kinova_description/meshes/forearm_link.dae" />
         </geometry>
       </collision>
@@ -127,14 +127,14 @@
         <origin xyz="0 0 0" rpy="0 0 0" />
         <geometry>
-          <mesh filename="package://hyqarm_description/meshes/spherical_wrist_1_link.dae" />
-        </geometry>
-        <material name="">
-          <color rgba="0.75294 0.75294 0.75294 1" />
-        </material>
-      </visual>
-      <collision>
-        <origin xyz="0 0 0" rpy="0 0 0" />
-        <geometry>
-          <mesh filename="package://hyqarm_description/meshes/spherical_wrist_1_link.dae" />
+          <mesh filename="package://gen3kinova_description/meshes/spherical_wrist_1_link.dae" />
+        </geometry>
+        <material name="">
+          <color rgba="0.75294 0.75294 0.75294 1" />
+        </material>
+      </visual>
+      <collision>
+        <origin xyz="0 0 0" rpy="0 0 0" />
+        <geometry>
+          <mesh filename="package://gen3kinova_description/meshes/spherical_wrist_1_link.dae" />
         </geometry>
       </collision>
@@ -156,14 +156,14 @@
         <origin xyz="0 0 0" rpy="0 0 0" />
         <geometry>
-          <mesh filename="package://hyqarm_description/meshes/spherical_wrist_2_link.dae" />
-        </geometry>
-        <material name="">
-          <color rgba="0.75294 0.75294 0.75294 1" />
-        </material>
-      </visual>
-      <collision>
-        <origin xyz="0 0 0" rpy="0 0 0" />
-        <geometry>
-          <mesh filename="package://hyqarm_description/meshes/spherical_wrist_2_link.dae" />
+          <mesh filename="package://gen3kinova_description/meshes/spherical_wrist_2_link.dae" />
+        </geometry>
+        <material name="">
+          <color rgba="0.75294 0.75294 0.75294 1" />
+        </material>
+      </visual>
+      <collision>
+        <origin xyz="0 0 0" rpy="0 0 0" />
+        <geometry>
+          <mesh filename="package://gen3kinova_description/meshes/spherical_wrist_2_link.dae" />
         </geometry>
       </collision>
@@ -185,14 +185,14 @@
         <origin xyz="0 0 0" rpy="0 0 0" />
         <geometry>
-          <mesh filename="package://hyqarm_description/meshes/bracelet_no_vision_link.dae" />
-        </geometry>
-        <material name="">
-          <color rgba="0.75294 0.75294 0.75294 1" />
-        </material>
-      </visual>
-      <collision>
-        <origin xyz="0 0 0" rpy="0 0 0" />
-        <geometry>
-          <mesh filename="package://hyqarm_description/meshes/bracelet_no_vision_link.dae" />
+          <mesh filename="package://gen3kinova_description/meshes/bracelet_no_vision_link.dae" />
+        </geometry>
+        <material name="">
+          <color rgba="0.75294 0.75294 0.75294 1" />
+        </material>
+      </visual>
+      <collision>
+        <origin xyz="0 0 0" rpy="0 0 0" />
+        <geometry>
+          <mesh filename="package://gen3kinova_description/meshes/bracelet_no_vision_link.dae" />
         </geometry>
       </collision>

File: descriptions/hyq_description/robots/hyq_gen3kinova.srdf.xacro (robot description, xacro)
@@ -1,5 +1,5 @@
 <?xml version="1.0" ?>
 <robot name="hyq" xmlns:xacro="http://ros.org/wiki/xacro">
-  <group name="hyqarm_arm">
+  <group name="gen3kinova_arm">
     <chain base_link="base_arm" tip_link="end_effector_link"/>
     <joint name="z_joint_1"/>
@@ -51,5 +51,5 @@
     <group name="lh_leg"/>
     <group name="rh_leg"/>
-    <group name="hyqarm_arm"/>
+    <group name="gen3kinova_arm"/>
   </group>
   <group_state group="chains" name="home">

File: descriptions/hyq_description/urdfs/arm/gen3kinova_adapter.urdf.xacro (robot description, xacro)
@@ -6,5 +6,5 @@
         <origin xyz="0.6 0 0.15" rpy="0 0.785398 0" />
  </joint>
-<xacro:include filename="$(find hyqarm_description)/urdfs/arm.urdf.xacro" />
+<xacro:include filename="$(find gen3kinova_description)/urdfs/arm.urdf.xacro" />
 <xacro:include filename="$(find hyq_description)/urdfs/arm/arm.transmission.xacro"/>
 <xacro:arm_transmission name="z_joint_1"/>
