Commit message: Add anymalc and move the launch file to controller

File: descriptions/anymalc_description/urdfs/leg.transmission.xacro (robot description, xacro)
@@ -1,12 +1,12 @@
 <?xml version="1.0"?>
 <robot xmlns:xacro="http://ros.org/wiki/xacro">
-        <xacro:macro name="leg_transmission" params="name">
+	<xacro:macro name="leg_transmission" params="name">
     	<!-- Hip assembly -->
-                <transmission name="${name}_haa_trans">
+		<transmission name="${name}_haa_trans">
 			<type>transmission_interface/SimpleTransmission</type>
-                        <joint name="${name}_haa_joint">
+			<joint name="${name}_haa_joint">
 				<hardwareInterface>EffortJointInterface</hardwareInterface>
 			</joint>
-                        <actuator name="${name}_haa_motor">
+			<actuator name="${name}_haa_motor">
 				<hardwareInterface>EffortJointInterface</hardwareInterface>
 				<mechanicalReduction>1</mechanicalReduction>
@@ -14,10 +14,10 @@
 		</transmission>
     	<!-- Upper leg -->
-                <transmission name="${name}_hfe_trans">
+		<transmission name="${name}_hfe_trans">
 			<type>transmission_interface/SimpleTransmission</type>
-                        <joint name="${name}_hfe_joint">
+			<joint name="${name}_hfe_joint">
 				<hardwareInterface>EffortJointInterface</hardwareInterface>
 			</joint>
-                        <actuator name="${name}_hfe_motor">
+			<actuator name="${name}_hfe_motor">
 				<hardwareInterface>EffortJointInterface</hardwareInterface>
 				<mechanicalReduction>1</mechanicalReduction>
@@ -25,10 +25,10 @@
 		</transmission>
     	<!-- Lower leg -->
-                <transmission name="${name}_kfe_trans">
+		<transmission name="${name}_kfe_trans">
 			<type>transmission_interface/SimpleTransmission</type>
-                        <joint name="${name}_kfe_joint">
+			<joint name="${name}_kfe_joint">
 				<hardwareInterface>EffortJointInterface</hardwareInterface>
 			</joint>
-                        <actuator name="${name}_kfe_motor">
+			<actuator name="${name}_kfe_motor">
 				<hardwareInterface>EffortJointInterface</hardwareInterface>
 				<mechanicalReduction>1</mechanicalReduction>
