Commit message: Move spot foot joints to improve the contacts

File: descriptions/spot_description/robots/spot.urdf.xacro (robot description, xacro)
@@ -60,5 +60,7 @@
     <!-- foot -->
     <xacro:property name="foot_mass" value="0.06"/>
-    <xacro:property name="foot_radius" value="0.034"/>
+    <xacro:property name="foot_radius" value="0.03"/>
+    <xacro:property name="foot_x" value="-0.01"/>
+    <xacro:property name="foot_z" value="-0.35"/>
     <!-- Floating-base Joint -->
     <link name="world"/>
@@ -182,5 +184,5 @@
     </joint>
     <joint name="lf_foot_joint" type="fixed">
-        <origin xyz="0 0.0 -0.35" rpy="0 0 0" />
+        <origin xyz="${foot_x} 0.0 ${foot_z}" rpy="0 0 0" />
         <parent link="lf_lowerleg" />
         <child link="lf_foot" />
@@ -290,5 +292,5 @@
     </joint>
     <joint name="rf_foot_joint" type="fixed">
-        <origin xyz="0 0.0 -0.35" rpy="0 0 0" />
+        <origin xyz="${foot_x} 0.0 ${foot_z}" rpy="0 0 0" />
         <parent link="rf_lowerleg" />
         <child link="rf_foot" />
@@ -398,5 +400,5 @@
     </joint>
     <joint name="lh_foot_joint" type="fixed">
-        <origin xyz="0 0.0 -0.35" rpy="0 0 0" />
+        <origin xyz="${foot_x} 0.0 ${foot_z}" rpy="0 0 0" />
         <parent link="lh_lowerleg" />
         <child link="lh_foot" />
@@ -506,5 +508,5 @@
     </joint>
     <joint name="rh_foot_joint" type="fixed">
-        <origin xyz="0 0.0 -0.35" rpy="0 0 0" />
+        <origin xyz="${foot_x} 0.0 ${foot_z}" rpy="0 0 0" />
         <parent link="rh_lowerleg" />
         <child link="rh_foot" />

Commit message: ported spot to 20.04

File: descriptions/spot_description/robots/spot.urdf.xacro (robot description, xacro)
@@ -6,4 +6,5 @@
     <xacro:arg name="arm_enabled" default="false"/>
     <xacro:arg name="arm_name" default="kinova"/>
+    <xacro:arg name="floating_base_link" default="true"/>
     <!-- legs transmission -->
     <xacro:include filename="$(find spot_description)/urdfs/leg.transmission.xacro"/>
@@ -64,10 +65,12 @@
     <xacro:property name="foot_z" value="-0.35"/>
     <!-- Floating-base Joint -->
-    <link name="world"/>
-    <joint name="floating_base_joint" type="floating">
-      <origin rpy="0 0 0" xyz="0 0 0"/>
-      <parent link="world"/>
-      <child link="base_link"/>
-    </joint>
+    <xacro:if value="$(arg floating_base_link)">
+	    <link name="world"/>
+	    <joint name="floating_base_joint" type="floating">
+	      <origin rpy="0 0 0" xyz="0 0 0"/>
+	      <parent link="world"/>
+	      <child link="base_link"/>
+	    </joint>
+    </xacro:if>
     <link name="base_link">
         <visual>

Commit message: Add some torque limits to spot

File: descriptions/spot_description/robots/spot.urdf.xacro (robot description, xacro)
@@ -130,5 +130,5 @@
         <parent link="base_link" />
         <child link="lf_hip" />
-        <limit effort="1000" velocity="1000.00" lower="-0.78539816339744827899" upper="0.78539816339744827899" />
+        <limit effort="50" velocity="1000.00" lower="-0.78539816339744827899" upper="0.78539816339744827899" />
     </joint>
     <link name="lf_upperleg">
@@ -157,5 +157,5 @@
         <parent link="lf_hip" />
         <child link="lf_upperleg" />
-        <limit effort="1000" velocity="1000.00" lower="-0.89884456477707963539" upper="2.2951079663725435509" />
+        <limit effort="50" velocity="1000.00" lower="-0.89884456477707963539" upper="2.2951079663725435509" />
     </joint>
     <link name="lf_lowerleg">
@@ -184,5 +184,5 @@
         <parent link="lf_upperleg" />
         <child link="lf_lowerleg" />
-        <limit effort="1000" velocity="1000.00" lower="-2.7929" upper="-0.254801" />
+        <limit effort="50" velocity="1000.00" lower="-2.7929" upper="-0.254801" />
     </joint>
     <joint name="lf_foot_joint" type="fixed">
@@ -238,5 +238,5 @@
         <parent link="base_link" />
         <child link="rf_hip" />
-        <limit effort="1000" velocity="1000.00" lower="-0.78539816339744827899" upper="0.78539816339744827899" />
+        <limit effort="50" velocity="1000.00" lower="-0.78539816339744827899" upper="0.78539816339744827899" />
     </joint>
     <link name="rf_upperleg">
@@ -265,5 +265,5 @@
         <parent link="rf_hip" />
         <child link="rf_upperleg" />
-        <limit effort="1000" velocity="1000.00" lower="-0.89884456477707963539" upper="2.2951079663725435509" />
+        <limit effort="50" velocity="1000.00" lower="-0.89884456477707963539" upper="2.2951079663725435509" />
     </joint>
     <link name="rf_lowerleg">
@@ -292,5 +292,5 @@
         <parent link="rf_upperleg" />
         <child link="rf_lowerleg" />
-        <limit effort="1000" velocity="1000.00" lower="-2.7929" upper="-0.247563" />
+        <limit effort="50" velocity="1000.00" lower="-2.7929" upper="-0.247563" />
     </joint>
     <joint name="rf_foot_joint" type="fixed">
@@ -346,5 +346,5 @@
         <parent link="base_link" />
         <child link="lh_hip" />
-        <limit effort="1000" velocity="1000.00" lower="-0.78539816339744827899" upper="0.78539816339744827899" />
+        <limit effort="50" velocity="1000.00" lower="-0.78539816339744827899" upper="0.78539816339744827899" />
     </joint>
     <link name="lh_upperleg">
@@ -373,5 +373,5 @@
         <parent link="lh_hip" />
         <child link="lh_upperleg" />
-        <limit effort="1000" velocity="1000.00" lower="-0.89884456477707963539" upper="2.2951079663725435509" />
+        <limit effort="50" velocity="1000.00" lower="-0.89884456477707963539" upper="2.2951079663725435509" />
     </joint>
     <link name="lh_lowerleg">
@@ -400,5 +400,5 @@
         <parent link="lh_upperleg" />
         <child link="lh_lowerleg" />
-        <limit effort="1000" velocity="1000.00" lower="-2.7929" upper="-0.267153" />
+        <limit effort="50" velocity="1000.00" lower="-2.7929" upper="-0.267153" />
     </joint>
     <joint name="lh_foot_joint" type="fixed">
@@ -454,5 +454,5 @@
         <parent link="base_link" />
         <child link="rh_hip" />
-        <limit effort="1000" velocity="1000.00" lower="-0.78539816339744827899" upper="0.78539816339744827899" />
+        <limit effort="50" velocity="1000.00" lower="-0.78539816339744827899" upper="0.78539816339744827899" />
     </joint>
     <link name="rh_upperleg">
@@ -481,5 +481,5 @@
         <parent link="rh_hip" />
         <child link="rh_upperleg" />
-        <limit effort="1000" velocity="1000.00" lower="-0.89884456477707963539" upper="2.2951079663725435509" />
+        <limit effort="50" velocity="1000.00" lower="-0.89884456477707963539" upper="2.2951079663725435509" />
     </joint>
     <link name="rh_lowerleg">
@@ -508,5 +508,5 @@
         <parent link="rh_upperleg" />
         <child link="rh_lowerleg" />
-        <limit effort="1000" velocity="1000.00" lower="-2.7929" upper="-0.257725" />
+        <limit effort="50" velocity="1000.00" lower="-2.7929" upper="-0.257725" />
     </joint>
     <joint name="rh_foot_joint" type="fixed">

Commit message: Add material color

File: descriptions/spot_description/robots/spot.urdf.xacro (robot description, xacro)
@@ -62,6 +62,6 @@
     <xacro:property name="foot_mass" value="0.06"/>
     <xacro:property name="foot_radius" value="0.03"/>
-    <xacro:property name="foot_x" value="-0.01"/>
-    <xacro:property name="foot_z" value="-0.35"/>
+    <xacro:property name="foot_x" value="-0.005"/>
+    <xacro:property name="foot_z" value="-0.348"/>
     <!-- Floating-base Joint -->
     <xacro:if value="$(arg floating_base_link)">
@@ -197,5 +197,7 @@
             <sphere radius="${foot_radius-0.01}"/>
         </geometry>
-        <material name="green"/>
+        <material name="green">
+          <color rgba="0.0 0.8 0.0 1.0"/>
+        </material>
     </visual>
     <collision>
@@ -305,5 +307,7 @@
             <sphere radius="${foot_radius-0.01}"/>
         </geometry>
-        <material name="green"/>
+        <material name="green">
+          <color rgba="0.0 0.8 0.0 1.0"/>
+        </material>
     </visual>
     <collision>
@@ -413,5 +417,7 @@
             <sphere radius="${foot_radius-0.01}"/>
         </geometry>
-        <material name="green"/>
+        <material name="green">
+          <color rgba="0.0 0.8 0.0 1.0"/>
+        </material>
     </visual>
     <collision>
@@ -521,5 +527,7 @@
             <sphere radius="${foot_radius-0.01}"/>
         </geometry>
-        <material name="green"/>
+        <material name="green">
+          <color rgba="0.0 0.8 0.0 1.0"/>
+        </material>
     </visual>
     <collision>
