Commit message: Fix spot standdown

File: descriptions/spot_description/robots/spot.srdf.xacro (robot description, xacro)
@@ -61,16 +61,16 @@
     </group_state>
     <group_state group="chains" name="standdown">
-        <joint name="lf_haa_joint" value="0.5"/>
-        <joint name="lf_hfe_joint" value="1.75"/>
-        <joint name="lf_kfe_joint" value="-2.79"/>
-        <joint name="rf_haa_joint" value="0.5"/>
-        <joint name="rf_hfe_joint" value="1.75"/>
-        <joint name="rf_kfe_joint" value="-2.79"/>
-        <joint name="lh_haa_joint" value="-0.75"/>
-        <joint name="lh_hfe_joint" value="1.60"/>
-        <joint name="lh_kfe_joint" value="-2.6"/>
-        <joint name="rh_haa_joint" value="-0.75"/>
-        <joint name="rh_hfe_joint" value="1.60"/>
-        <joint name="rh_kfe_joint" value="-2.6"/>
+        <joint name="lf_haa_joint" value="0.6"/>
+        <joint name="lf_hfe_joint" value="1.35"/>
+        <joint name="lf_kfe_joint" value="-2.7"/>
+        <joint name="rf_haa_joint" value="-0.6"/>
+        <joint name="rf_hfe_joint" value="1.35"/>
+        <joint name="rf_kfe_joint" value="-2.7"/>
+        <joint name="lh_haa_joint" value="0.6"/>
+        <joint name="lh_hfe_joint" value="1.35"/>
+        <joint name="lh_kfe_joint" value="-2.7"/>
+        <joint name="rh_haa_joint" value="-0.6"/>
+        <joint name="rh_hfe_joint" value="1.35"/>
+        <joint name="rh_kfe_joint" value="-2.7"/>
     </group_state>
 </robot>
