Commit message: Updated params for spot kinova

File: descriptions/spot_description/robots/spot_kinova.srdf.xacro (robot description, xacro)
@@ -78,7 +78,7 @@
       <joint name="rh_kfe_joint"  value="-1.35"/>
       <joint name="kinova_joint_1" value="0.0"/>
-      <joint name="kinova_joint_2" value="2.30"/>
-      <joint name="kinova_joint_3" value="1.0"/>
-      <joint name="kinova_joint_4" value="3.0"/>
+      <joint name="kinova_joint_2" value="4.0"/>
+      <joint name="kinova_joint_3" value="5.6"/>
+      <joint name="kinova_joint_4" value="3.14"/>
     </group_state>
 </robot>

File: descriptions/spot_description/urdfs/arm/kinova_adapter.urdf.xacro (robot description, xacro)
@@ -5,5 +5,5 @@
        <parent link="base_link"/>
        <child link="kinova_adapter_link"/>
-       <origin xyz="0.0 0.0 0.0" rpy="0 0 0"/>
+       <origin xyz="0.35 0.0 -0.08" rpy="0 0 0"/>
 </joint>
 <xacro:include filename="$(find kinova_description)/urdf/m1n4s200.xacro"/>

Commit message: Add base to spot with kinova

File: descriptions/spot_description/robots/spot_kinova.srdf.xacro (robot description, xacro)
@@ -1,4 +1,7 @@
 <?xml version="1.0" ?>
 <robot name="spot" xmlns:xacro="http://ros.org/wiki/xacro">
+    <group name="base">
+      <link name="base_link"/>
+    </group>
     <group name="kinova_arm">
       <chain base_link="kinova_link_base" tip_link="kinova_end_effector"/>

Commit message: Add standdown and standup for spot with kinova

File: descriptions/spot_description/robots/spot_kinova.srdf.xacro (robot description, xacro)
@@ -54,17 +54,17 @@
       <group name="kinova_arm"/>
     </group>
-    <group_state group="chains" name="home">
+    <group_state group="chains" name="standup">
       <joint name="lf_haa_joint" value="0.20"/>
       <joint name="lf_hfe_joint" value="0.70"/>
-      <joint name="lf_kfe_joint"  value="-1.35"/>
+      <joint name="lf_kfe_joint" value="-1.35"/>
       <joint name="rf_haa_joint" value="-0.20"/>
       <joint name="rf_hfe_joint" value="0.70"/>
-      <joint name="rf_kfe_joint"  value="-1.35"/>
+      <joint name="rf_kfe_joint" value="-1.35"/>
       <joint name="lh_haa_joint" value="0.20"/>
       <joint name="lh_hfe_joint" value="0.70"/>
-      <joint name="lh_kfe_joint"  value="-1.35"/>
+      <joint name="lh_kfe_joint" value="-1.35"/>
       <joint name="rh_haa_joint" value="-0.20"/>
       <joint name="rh_hfe_joint" value="0.70"/>
-      <joint name="rh_kfe_joint"  value="-1.35"/>
+      <joint name="rh_kfe_joint" value="-1.35"/>
       <joint name="kinova_joint_1" value="0.0"/>
       <joint name="kinova_joint_2" value="4.0"/>
@@ -72,3 +72,21 @@
       <joint name="kinova_joint_4" value="3.14"/>
     </group_state>
+    <group_state group="chains" name="standdown">
+      <joint name="lf_haa_joint" value="0.6"/>
+      <joint name="lf_hfe_joint" value="1.35"/>
+      <joint name="lf_kfe_joint" value="-2.7"/>
+      <joint name="rf_haa_joint" value="-0.6"/>
+      <joint name="rf_hfe_joint" value="1.35"/>
+      <joint name="rf_kfe_joint" value="-2.7"/>
+      <joint name="lh_haa_joint" value="0.6"/>
+      <joint name="lh_hfe_joint" value="1.35"/>
+      <joint name="lh_kfe_joint" value="-2.7"/>
+      <joint name="rh_haa_joint" value="-0.6"/>
+      <joint name="rh_hfe_joint" value="1.35"/>
+      <joint name="rh_kfe_joint" value="-2.7"/>
+      <joint name="kinova_joint_1" value="0.0"/>
+      <joint name="kinova_joint_2" value="4.9"/>
+      <joint name="kinova_joint_3" value="5.6"/>
+      <joint name="kinova_joint_4" value="0.0"/>
+    </group_state>
 </robot>
