Commit message: Clean up the robot descriptions, use wolf_description_utils for the common xacro files

File: descriptions/anymalc_description/robots/anymalc.urdf.xacro (robot description, xacro)
@@ -8,11 +8,14 @@
    <xacro:arg name="load_force_sensors" default="false"/>
    <xacro:arg name="task_period" default="0.004"/>
+   <xacro:arg name="floating_base_link" default="true"/>
+   <xacro:arg name="robot_name"  default="anymalc"/>
+   <xacro:arg name="base_name"   default="base"/>
+   <!-- load generic materials -->
+   <xacro:include filename="$(find wolf_description_utils)/urdfs/materials.xacro"/>
    <!-- generic simulator_gazebo plugins for starting mechanism control, ros time -->
-   <xacro:include filename="$(find anymalc_description)/gazebo/gazebo.urdf.xacro">
-        <xacro:arg name="task_period" value="$(arg task_period)"/>
-   </xacro:include> -->
-    legs transmission -->
-   <xacro:include filename="$(find anymalc_description)/urdfs/leg.transmission.xacro"/>
-   <xacro:include filename="$(find anymalc_description)/urdfs/leg.gazebo.xacro"/>
+   <xacro:include filename="$(find wolf_description_utils)/urdfs/gazebo.urdf.xacro"/>
+   <!-- legs transmission and gazebo plugins -->
+   <xacro:include filename="$(find wolf_description_utils)/urdfs/leg.transmission.xacro"/>
+   <xacro:include filename="$(find wolf_description_utils)/urdfs/leg.gazebo.xacro"/>
     <!-- Base link -->
     <link name="base">
@@ -62,10 +65,12 @@
     </link>
     <!-- Floating-base Joint -->
-    <link name="world"/>
-    <joint name="floating_base_joint" type="floating">
-      <origin rpy="0 0 0" xyz="0 0 0"/>
-      <parent link="world"/>
-      <child link="base"/>
-    </joint>
+    <xacro:if value="$(arg floating_base_link)">
+            <link name="world"/>
+            <joint name="floating_base_joint" type="floating">
+              <origin rpy="0 0 0" xyz="0 0 0"/>
+              <parent link="world"/>
+              <child link="base"/>
+            </joint>
+    </xacro:if>
     <!-- Fixed joint to add dummy inertia link -->
     <joint name="base_to_base_inertia" type="fixed">
@@ -572,5 +577,5 @@
     <!-- Camera color optical link -->
     <link name="depth_camera_right_color_optical_frame"/>
-    <!-- parent to cage joint, located between mounting plate on trunk and the cage -->
+    <!-- parent to cage joint, located between mounting plate on base and the cage -->
     <joint name="base_to_lidar_cage" type="fixed">
         <parent link="base"/>

File: descriptions/hyq_description/robots/hyq.urdf.xacro (robot description, xacro)
@@ -3,8 +3,16 @@
 	<xacro:arg name="task_period" default="0.004"/>
         <xacro:arg name="arm_enabled" default="false"/>
-        <xacro:arg name="arm_name" default="teleop"/>
-	<!-- This argument allows us to load joint sensors that measure the internal wrenches -->
+        <xacro:arg name="arm_name" default="kinova"/>
 	<xacro:arg name="load_force_sensors" default="false"/>
 	<xacro:arg name="floating_base_link" default="true"/>
+        <xacro:arg name="robot_name"  default="hyq"/>
+        <xacro:arg name="base_name"   default="base_link"/>
+        <!-- load generic materials -->
+        <xacro:include filename="$(find wolf_description_utils)/urdfs/materials.xacro"/>
+        <!-- generic simulator_gazebo plugins for starting mechanism control, ros time -->
+        <xacro:include filename="$(find wolf_description_utils)/urdfs/gazebo.urdf.xacro"/>
+        <!-- legs transmission and gazebo plugins -->
+        <xacro:include filename="$(find wolf_description_utils)/urdfs/leg.transmission.xacro"/>
+        <xacro:include filename="$(find wolf_description_utils)/urdfs/leg.gazebo.xacro"/>
 	<!-- The following included files set up definitions of parts of the robot body -->
 	<xacro:include filename="$(find hyq_description)/urdfs/common.xacro"/>
@@ -13,17 +21,4 @@
 	<!-- HyQ legs -->
 	<xacro:include filename="$(find hyq_description)/urdfs/leg/leg.urdf.xacro"/>
-	<!-- generic simulator_gazebo plugins for starting mechanism control, ros time -->
-        <xacro:include filename="$(find hyq_description)/gazebo/gazebo.urdf.xacro">
-             <xacro:arg name="task_period" value="$(arg task_period)"/>
-        </xacro:include>
-	<!-- Now we can start using the macros included above to define the actual HyQ -->
-	<!-- The first use of a macro. This one was defined in trunk.urdf.xacro above.
-A macro like this will expand to a set of link and joint definitions, and to additional
-Gazebo-related extensions (sensor plugins, etc). The macro takes an argument, name,
-that equals "base", and uses it to generate names for its component links and joints
-(e.g., base_link). The included origin block is also an argument to the macro. By convention,
-the origin block defines where the component is w.r.t its parent (in this case the parent
-is the world frame). For more, see http://ros.org/wiki/xacro -->
-	<!-- body -->
 	<!-- trunk -->
 	<xacro:hyq_trunk name="base" floating_base_link="$(arg floating_base_link)">

File: descriptions/hyq_description/urdfs/leg/leg.urdf.xacro (robot description, xacro)
@@ -1,7 +1,4 @@
 <?xml version="1.0"?>
 <robot xmlns:xacro="http://ros.org/wiki/xacro">
-	<!-- Things that are needed only for Gazebo (not the physical robot). These include sensor and controller plugin specifications -->
-	<xacro:include filename="$(find hyq_description)/urdfs/leg/leg.transmission.xacro"/>
-	<xacro:include filename="$(find hyq_description)/urdfs/leg/leg.gazebo.xacro"/>
 	<!-- ================================== Leg ================================== -->
 	<!-- The xacro macro xacro:hyq_leg contains: hip assembly, upper and lower leg -->

File: descriptions/minicheetah_description/robots/minicheetah.urdf.xacro (robot description, xacro)
@@ -23,11 +23,12 @@
   <xacro:arg name="load_force_sensors" default="false"/>
   <xacro:arg name="task_period" default="0.004"/>
+  <xacro:arg name="floating_base_link" default="true"/>
+  <xacro:arg name="robot_name"  default="minicheetah"/>
+  <xacro:arg name="base_name"   default="trunk"/>
   <!-- generic simulator_gazebo plugins for starting mechanism control, ros time -->
-  <xacro:include filename="$(find minicheetah_description)/gazebo/gazebo.urdf.xacro">
-       <xacro:arg name="task_period" value="$(arg task_period)"/>
-  </xacro:include>
-  <!-- legs transmission -->
-  <xacro:include filename="$(find minicheetah_description)/urdfs/leg.transmission.xacro"/>
-  <xacro:include filename="$(find minicheetah_description)/urdfs/leg.gazebo.xacro"/>
+  <xacro:include filename="$(find wolf_description_utils)/urdfs/gazebo.urdf.xacro"/>
+  <!-- legs transmission and gazebo plugins -->
+  <xacro:include filename="$(find wolf_description_utils)/urdfs/leg.transmission.xacro"/>
+  <xacro:include filename="$(find wolf_description_utils)/urdfs/leg.gazebo.xacro"/>
   <material name="black">
     <color rgba="0.0 0.0 0.0 1.0"/>
@@ -136,11 +137,13 @@
         </collision>
     </link> -->
-   <!-- Floating-base Joint -->
-   <link name="world"/>
-   <joint name="floating_base_joint" type="floating">
-     <origin rpy="0 0 0" xyz="0 0 0"/>
-     <parent link="world"/>
-     <child link="trunk"/>
-   </joint>
+  <!-- Floating-base Joint -->
+  <xacro:if value="$(arg floating_base_link)">
+          <link name="world"/>
+          <joint name="floating_base_joint" type="floating">
+            <origin rpy="0 0 0" xyz="0 0 0"/>
+            <parent link="world"/>
+            <child link="trunk"/>
+          </joint>
+  </xacro:if>
   <!-- //////////////////////haa//////////////////// -->
   <joint name="lh_haa_joint" type="revolute">

File: descriptions/solo_description/robots/solo.urdf.xacro (robot description, xacro)
@@ -5,23 +5,28 @@
     <xacro:property name="opacity" value="1.0" />
     <xacro:arg name="load_force_sensors" default="false"/>
+    <xacro:arg name="task_period" default="0.004"/>
     <xacro:arg name="floating_base_link" default="true"/>
-    <xacro:include filename="$(find solo_description)/gazebo/gazebo.urdf.xacro">
-        <xacro:arg name="task_period" value="$(arg task_period)"/>
-    </xacro:include>
-                <!-- Floating-base Joint -->
-		<xacro:if value="$(arg floating_base_link)">
-		        <link name="world"/>
-		        <joint name="floating_base_joint" type="floating">
-		            <origin rpy="0 0 0" xyz="0 0 0"/>
-		            <parent link="world"/>
-		            <child link="base_link"/>
-		        </joint>
-		</xacro:if>
-		<link name="base_link" />
-                <joint name="floating_base" type="fixed">
-                    <origin rpy="0 0 0" xyz="0 0 0"/>
-                    <parent link="base_link"/>
-                    <child link="trunk"/>
-                </joint>
+    <xacro:arg name="robot_name"  default="solo"/>
+    <xacro:arg name="base_name"   default="base_link"/>
+    <!-- generic simulator_gazebo plugins for starting mechanism control, ros time -->
+    <xacro:include filename="$(find wolf_description_utils)/urdfs/gazebo.urdf.xacro"/>
+    <!-- legs transmission and gazebo plugins -->
+    <xacro:include filename="$(find wolf_description_utils)/urdfs/leg.transmission.xacro"/>
+    <xacro:include filename="$(find wolf_description_utils)/urdfs/leg.gazebo.xacro"/>
+    <!-- Floating-base Joint -->
+    <xacro:if value="$(arg floating_base_link)">
+            <link name="world"/>
+            <joint name="floating_base_joint" type="floating">
+                <origin rpy="0 0 0" xyz="0 0 0"/>
+                <parent link="world"/>
+                <child link="base_link"/>
+            </joint>
+    </xacro:if>
+    <link name="base_link" />
+    <joint name="floating_base" type="fixed">
+        <origin rpy="0 0 0" xyz="0 0 0"/>
+        <parent link="base_link"/>
+        <child link="trunk"/>
+    </joint>
     <link name="trunk">
         <inertial>

File: descriptions/solo_description/urdfs/leg.xacro (robot description, xacro)
@@ -1,7 +1,4 @@
 <?xml version="1.0"?>
 <robot xmlns:xacro="http://ros.org/wiki/xacro" name="solo">
-    <!-- Things that are needed only for Gazebo (not the physical robot). These include sensor and controller plugin specifications -->
-    <xacro:include filename="$(find solo_description)/urdfs/leg.transmission.xacro"/>
-    <xacro:include filename="$(find solo_description)/urdfs/leg.gazebo.xacro"/>
     <!-- These are absoulte distance value, the sign are decided below -->
     <xacro:property name="base_2_HAA_x" value="${194.60 * 0.001}" />

File: descriptions/spot_description/robots/spot.urdf.xacro (robot description, xacro)
@@ -7,11 +7,13 @@
     <xacro:arg name="arm_name" default="kinova"/>
     <xacro:arg name="floating_base_link" default="true"/>
-    <!-- legs transmission -->
-    <xacro:include filename="$(find spot_description)/urdfs/leg.transmission.xacro"/>
-    <xacro:include filename="$(find spot_description)/urdfs/leg.gazebo.xacro"/>
+    <xacro:arg name="robot_name"  default="spot"/>
+    <xacro:arg name="base_name"   default="base_link"/>
+    <!-- load generic materials -->
+    <xacro:include filename="$(find wolf_description_utils)/urdfs/materials.xacro"/>
     <!-- generic simulator_gazebo plugins for starting mechanism control, ros time -->
-    <xacro:include filename="$(find spot_description)/gazebo/gazebo.urdf.xacro">
-         <xacro:arg name="task_period" value="$(arg task_period)"/>
-    </xacro:include>
+    <xacro:include filename="$(find wolf_description_utils)/urdfs/gazebo.urdf.xacro"/>
+    <!-- legs transmission and gazebo plugins -->
+    <xacro:include filename="$(find wolf_description_utils)/urdfs/leg.transmission.xacro"/>
+    <xacro:include filename="$(find wolf_description_utils)/urdfs/leg.gazebo.xacro"/>
     <!-- dynamics inertial value -->
     <!-- body -->
